File: Circuit/boneIO - relay board rev0.2/boneIO - relay board.kicad_pcb (KiCad board)
At the start: 2 copper layers, 169 x 108 mm, 47 parts, among them J1 Screw_Terminal_01x04, J10 Screw_Terminal_01x04, J11 Screw_Terminal_01x04, J12 Conn_02x13_Odd_Even, J2 Screw_Terminal_01x04, J3 Screw_Terminal_01x04, J4 Screw_Terminal_01x04, J5 Screw_Terminal_01x04, J6 Screw_Terminal_01x04, J7 POWER RELAY, J8 Screw_Terminal_01x04, J9 Screw_Terminal_01x04, K1 RM85-2011-35-1005, K10 RM85-2011-35-1005, K11 RM85-2011-35-1005, K12 RM85-2011-35-1005, K13 RM85-2011-35-1005, K14 RM85-2011-35-1005, K15 RM85-2011-35-1005, K16 RM85-2011-35-1005, K17 RM85-2011-35-1005, K18 RM85-2011-35-1005, K19 RM85-2011-35-1005, K2 RM85-2011-35-1005, K20 RM85-2011-35-1005, K3 RM85-2011-35-1005, K4 RM85-2011-35-1005, K5 RM85-2011-35-1005, K6 RM85-2011-35-1005, K7 RM85-2011-35-1005, K8 RM85-2011-35-1005, K9 RM85-2011-35-1005, U1 ULN2803A, U2 ULN2803A, U3 ULN2803A, U4 MCP9808_MSOP

Commit message: Zmniejszone pcb
Routing:
- net SDA: track 56.8 -> 61.1 mm
- net K6: track 75.2 -> 77.3 mm
- net K5: track 73.9 -> 75.9 mm
- net K4: track 72.9 -> 74.9 mm
- net K3: track 71.5 -> 73.5 mm
- net K2: track 70.4 -> 72.3 mm
- net SCL: track 58.2 -> 60.2 mm
- net K1: track 69.2 -> 71.1 mm
- net K9: track 25.6 -> 27.2 mm
- net +5V: track 136.6 -> 138.1 mm
- net +3V3: track 68.5 -> 69.9 mm
- net K7: track 35.0 -> 33.8 mm
- net GND: vias 4 -> 48
Other:
- board size 169 x 108 mm -> 169 x 102 mm
