File: Circuit/boneIO - relay board rev0.2/boneIO - relay board.sch (KiCad schematic (older format))
At the start: 93 parts, among them J1 Screw_Terminal_01x04, J10 Screw_Terminal_01x04, J11 Screw_Terminal_01x04, J2 Screw_Terminal_01x04, J3 Screw_Terminal_01x04, J4 Screw_Terminal_01x04, J5 Screw_Terminal_01x04, J6 Conn_02x11_Odd_Even, J7 Screw_Terminal_01x04, J8 Screw_Terminal_01x04, J9 Screw_Terminal_01x04, K1 RM85-2011-35-1005, K10 RM85-2011-35-1005, K11 RM85-2011-35-1005, K12 RM85-2011-35-1005, K13 RM85-2011-35-1005, K14 RM85-2011-35-1005, K15 RM85-2011-35-1005, K16 RM85-2011-35-1005, K17 RM85-2011-35-1005, K18 RM85-2011-35-1005, K19 RM85-2011-35-1005, K2 RM85-2011-35-1005, K20 RM85-2011-35-1005, K3 RM85-2011-35-1005, K4 RM85-2011-35-1005, K5 RM85-2011-35-1005, K6 RM85-2011-35-1005, K7 RM85-2011-35-1005, K8 RM85-2011-35-1005, K9 RM85-2011-35-1005, Q1 BC817, Q10 BC817, Q11 BC817, Q12 BC817, Q13 BC817, Q14 BC817, Q15 BC817, Q16 BC817, Q17 BC817, Q18 BC817, Q19 BC817, Q2 BC817, Q20 BC817, Q3 BC817, Q4 BC817, Q5 BC817, Q6 BC817, Q7 BC817, Q8 BC817, Q9 BC817

Commit message: Zmiana gniazd, driverów i dodanie czujnika temp
Parts:
- removed D1, D10, D11, D12, D13, D14, D15, D16, D17, D18, D19, D2, D20, D3, D4, D5, D6, D7, D8, D9: 1N4148, Diode_SMD:D_1206_3216Metric, symbol Diode:1N4148
- removed J6: Conn_02x11_Odd_Even, Connector_PinHeader_2.54mm:PinHeader_2x11_P2.54mm_Vertical, symbol Connector_Generic:Conn_02x11_Odd_Even
- removed J7: Screw_Terminal_01x04, TerminalBlock_MetzConnect:TerminalBlock_MetzConnect_Type171_RT13704HBWC_1x04_P7.50mm_Horizontal, symbol Connector:Screw_Terminal_01x04
- removed Q1, Q10, Q11, Q12, Q13, Q14, Q15, Q16, Q17, Q18, Q19, Q2, Q20, Q3, Q4, Q5, Q6, Q7, Q8, Q9: BC817, Package_TO_SOT_SMD:SOT-23, symbol Transistor_BJT:BC817
- removed R10, R11, R12, R13, R14, R15, R16, R17, R18, R19, R20: 670, Resistor_SMD:R_1206_3216Metric, symbol Device:R
- added J12: Conn_02x13_Odd_Even, Connector_PinHeader_2.54mm:PinHeader_2x13_P2.54mm_Vertical, symbol Connector_Generic:Conn_02x13_Odd_Even
- added J6: Screw_Terminal_01x04, Connector_Phoenix_GMSTB:PhoenixContact_GMSTBA_2,5_4-G_1x04_P7.50mm_Horizontal, symbol Connector:Screw_Terminal_01x04
- added J7: POWER RELAY, Connector_PinHeader_2.54mm:PinHeader_1x03_P2.54mm_Vertical, symbol Connector:Screw_Terminal_01x03
- added U1, U2, U3: ULN2803A, Package_SO:SOIC-18W_7.5x11.6mm_P1.27mm, symbol Transistor_Array:ULN2803A
- added U4: MCP9808_MSOP, Package_SO:MSOP-8_3x3mm_P0.65mm, symbol boneIO---relay-board-rescue:MCP9808_MSOP-Sensor_Temperature
- J1, J10, J11, J2, J3, J4, J5, J8, J9: footprint TerminalBlock_MetzConnect:TerminalBlock_MetzConnect_Type171_RT13704HBWC_1x04_P7.50mm_Horizontal -> Connector_Phoenix_GMSTB:PhoenixContact_GMSTBA_2,5_4-G_1x04_P7.50mm_Horizontal
- R1, R2, R3, R4, R5, R6: value 670 -> 0k; footprint Resistor_SMD:R_1206_3216Metric -> Resistor_SMD:R_0603_1608Metric
- R7, R8, R9: value 670 -> 4.7k; footprint Resistor_SMD:R_1206_3216Metric -> Resistor_SMD:R_0603_1608Metric
- renumbered H2 to H1, H1 to H2
Connections:
- net labels added: +24V, +3V3, K1, K10, K11, K12, K13, K14, K15, K16, K17, K18, K19, K2, K20, K3, K4, K5, K6, K7, K8, K9, RELAY1, RELAY10, RELAY11, RELAY12, RELAY13, RELAY14, RELAY15, RELAY16, RELAY17, RELAY18, RELAY19, RELAY2, RELAY20, RELAY3, RELAY4, RELAY5, RELAY6, RELAY7, RELAY8, RELAY9, SCL, SDA, VCC
- wire segments 440 -> 339
Other:
- note added: "MCP9808\n\n"
- note added: "PINOUT"
- note added: "POWER JUMPER\n\n"
- note added: "RELAY"
- note added: "ULN2803A"
- moved on the sheet: H1, H2

Commit message: Zmniejszone pcb
Parts:
- K1, K10, K11, K12, K13, K14, K15, K16, K17, K18, K19, K2, K20, K3, K4, K5, K6, K7, K8, K9: symbol boneIO---relay-board-rescue:RM85-2011-35-1005-MK -> boneIO---relay-board-rescue:RM85-2011-35-1005-MK-boneIO---relay-board-rescue
- U4: symbol boneIO---relay-board-rescue:MCP9808_MSOP-Sensor_Temperature -> boneIO---relay-board-rescue:MCP9808_MSOP-Sensor_Temperature-boneIO---relay-board-rescue
Changed lines of the file:
@@
 NoConn ~ 19450 10200
 $Comp
-L boneIO---relay-board-rescue:RM85-2011-35-1005-MK K18
+L boneIO---relay-board-rescue:RM85-2011-35-1005-MK-boneIO---relay-board-rescue K18
 U 1 1 656F8EFF
 P 19750 10200
@@
 NoConn ~ 19450 8450
 $Comp
-L boneIO---relay-board-rescue:RM85-2011-35-1005-MK K17
+L boneIO---relay-board-rescue:RM85-2011-35-1005-MK-boneIO---relay-board-rescue K17
 U 1 1 656F8F21
 P 19750 8450
@@
 NoConn ~ 19450 13750
 $Comp
-L boneIO---relay-board-rescue:RM85-2011-35-1005-MK K20
+L boneIO---relay-board-rescue:RM85-2011-35-1005-MK-boneIO---relay-board-rescue K20
 U 1 1 656F8F47
 P 19750 13750
@@
 NoConn ~ 19450 12000
 $Comp
-L boneIO---relay-board-rescue:RM85-2011-35-1005-MK K19
+L boneIO---relay-board-rescue:RM85-2011-35-1005-MK-boneIO---relay-board-rescue K19
 U 1 1 656F8F69
 P 19750 12000
@@
 NoConn ~ 15300 10200
 $Comp
-L boneIO---relay-board-rescue:RM85-2011-35-1005-MK K15
+L boneIO---relay-board-rescue:RM85-2011-35-1005-MK-boneIO---relay-board-rescue K15
 U 1 1 6557F0EC
 P 15000 10200
@@
 NoConn ~ 15300 8450
 $Comp
-L boneIO---relay-board-rescue:RM85-2011-35-1005-MK K16
+L boneIO---relay-board-rescue:RM85-2011-35-1005-MK-boneIO---relay-board-rescue K16
 U 1 1 6557F0CB
 P 15000 8450
@@
 NoConn ~ 15300 13750
 $Comp
-L boneIO---relay-board-rescue:RM85-2011-35-1005-MK K13
+L boneIO---relay-board-rescue:RM85-2011-35-1005-MK-boneIO---relay-board-rescue K13
 U 1 1 6557F0A7
 P 15000 13750
@@
 NoConn ~ 15300 12000
 $Comp
-L boneIO---relay-board-rescue:RM85-2011-35-1005-MK K14
+L boneIO---relay-board-rescue:RM85-2011-35-1005-MK-boneIO---relay-board-rescue K14
 U 1 1 6557F085
 P 15000 12000
@@
 	12500 13850 12500 13750
 $Comp
-L boneIO---relay-board-rescue:RM85-2011-35-1005-MK K11
+L boneIO---relay-board-rescue:RM85-2011-35-1005-MK-boneIO---relay-board-rescue K11
 U 1 1 6557F056
 P 12500 12000
@@
 	12200 10700 12200 10550
 $Comp
-L boneIO---relay-board-rescue:RM85-2011-35-1005-MK K12
+L boneIO---relay-board-rescue:RM85-2011-35-1005-MK-boneIO---relay-board-rescue K12
 U 1 1 6557F034
 P 12500 13750
@@
 	12500 10300 12500 10200
 $Comp
-L boneIO---relay-board-rescue:RM85-2011-35-1005-MK K9
+L boneIO---relay-board-rescue:RM85-2011-35-1005-MK-boneIO---relay-board-rescue K9
 U 1 1 6557F00E
 P 12500 8450
@@
 	12200 7150 12200 7000
 $Comp
-L boneIO---relay-board-rescue:RM85-2011-35-1005-MK K10
+L boneIO---relay-board-rescue:RM85-2011-35-1005-MK-boneIO---relay-board-rescue K10
 U 1 1 6557EFEC
 P 12500 10200
@@
 NoConn ~ 8100 10200
 $Comp
-L boneIO---relay-board-rescue:RM85-2011-35-1005-MK K6
+L boneIO---relay-board-rescue:RM85-2011-35-1005-MK-boneIO---relay-board-rescue K6
 U 1 1 650CB5D8
 P 7800 10200
@@
 NoConn ~ 8100 8450
 $Comp
-L boneIO---relay-board-rescue:RM85-2011-35-1005-MK K5
+L boneIO---relay-board-rescue:RM85-2011-35-1005-MK-boneIO---relay-board-rescue K5
 U 1 1 650CB5FA
 P 7800 8450
@@
 NoConn ~ 8100 13750
 $Comp
-L boneIO---relay-board-rescue:RM85-2011-35-1005-MK K8
+L boneIO---relay-board-rescue:RM85-2011-35-1005-MK-boneIO---relay-board-rescue K8
 U 1 1 650CB61E
 P 7800 13750
@@
 NoConn ~ 8100 12000
 $Comp
-L boneIO---relay-board-rescue:RM85-2011-35-1005-MK K7
+L boneIO---relay-board-rescue:RM85-2011-35-1005-MK-boneIO---relay-board-rescue K7
 U 1 1 650CB640
 P 7800 12000
@@
 	5300 13850 5300 13750
 $Comp
-L boneIO---relay-board-rescue:RM85-2011-35-1005-MK K3
+L boneIO---relay-board-rescue:RM85-2011-35-1005-MK-boneIO---relay-board-rescue K3
 U 1 1 64E84F3A
 P 5300 12000
@@
 	5000 10700 5000 10550
 $Comp
-L boneIO---relay-board-rescue:RM85-2011-35-1005-MK K4
+L boneIO---relay-board-rescue:RM85-2011-35-1005-MK-boneIO---relay-board-rescue K4
 U 1 1 64E84F18
 P 5300 13750
@@
 	5300 10300 5300 10200
 $Comp
-L boneIO---relay-board-rescue:RM85-2011-35-1005-MK K1
+L boneIO---relay-board-rescue:RM85-2011-35-1005-MK-boneIO---relay-board-rescue K1
 U 1 1 6266FFCC
 P 5300 8450
@@
 	5000 7150 5000 7000
 $Comp
-L boneIO---relay-board-rescue:RM85-2011-35-1005-MK K2
+L boneIO---relay-board-rescue:RM85-2011-35-1005-MK-boneIO---relay-board-rescue K2
 U 1 1 6266FFF0
 P 5300 10200
@@
 	4550 4450 4550 4150
 $Comp
-L boneIO---relay-board-rescue:MCP9808_MSOP-Sensor_Temperature U4
+L boneIO---relay-board-rescue:MCP9808_MSOP-Sensor_Temperature-boneIO---relay-board-rescue U4
 U 1 1 61B8C06C
 P 8750 4200
