File: Circuit/boneIO - input board/boneIO - input board.sch (KiCad schematic (older format))
At the start: 18 parts, among them J1 Screw_Terminal_01x03, J11 Conn_02x11_Odd_Even, J2 Screw_Terminal_01x08, J3 Screw_Terminal_01x08, J4 Screw_Terminal_01x08, J5 Screw_Terminal_01x08, J6 Screw_Terminal_01x08, J7 Screw_Terminal_01x08, P8 BeagleBone_Black_Header, P9 BeagleBone_Black_Header, SW1 SW_Push, SW2 SW_Push

Commit message: Circuit Repo Cleanup
Parts:
- AN1: symbol Connector:Screw_Terminal_01x07 -> boneIO---input-board-rescue:Screw_Terminal_01x07-Connector
- ANVDD1, VDD1: symbol Connector:Screw_Terminal_01x02 -> boneIO---input-board-rescue:Screw_Terminal_01x02-Connector
- H1, H2: symbol Mechanical:MountingHole -> boneIO---input-board-rescue:MountingHole-Mechanical
- I2C1: symbol Connector_Generic:Conn_01x04 -> boneIO---input-board-rescue:Conn_01x04-Connector_Generic
- J1: symbol Connector:Screw_Terminal_01x03 -> boneIO---input-board-rescue:Screw_Terminal_01x03-Connector
- J11: symbol Connector_Generic:Conn_02x11_Odd_Even -> boneIO---input-board-rescue:Conn_02x11_Odd_Even-Connector_Generic
- J2, J3, J4, J5, J6, J7: symbol Connector:Screw_Terminal_01x08 -> boneIO---input-board-rescue:Screw_Terminal_01x08-Connector
- P8, P9: symbol Connector_Generic:Conn_02x23_Odd_Even -> boneIO---input-board-rescue:Conn_02x23_Odd_Even-Connector_Generic
- SW1, SW2: symbol Switch:SW_Push -> boneIO---input-board-rescue:SW_Push-Switch
Changed lines of the file:
@@
 $EndDescr
 $Comp
-L Connector_Generic:Conn_02x23_Odd_Even P9
+L boneIO---input-board-rescue:Conn_02x23_Odd_Even-Connector_Generic P9
 U 1 1 55DF7DBA
 P 9300 3650
@@
 $EndComp
 $Comp
-L power:GND #PWR0101
+L boneIO---input-board-rescue:GND-power #PWR0101
 U 1 1 5FB90262
 P 9250 2200
@@
 $EndComp
 $Comp
-L power:GND #PWR0104
+L boneIO---input-board-rescue:GND-power #PWR0104
 U 1 1 5FB92372
 P 9650 3400
@@
 $EndComp
 $Comp
-L Connector_Generic:Conn_02x11_Odd_Even J11
+L boneIO---input-board-rescue:Conn_02x11_Odd_Even-Connector_Generic J11
 U 1 1 5FB93898
 P 6500 3650
@@
 $EndComp
 $Comp
-L power:+5V #PWR0107
+L boneIO---input-board-rescue:+5V-power #PWR0107
 U 1 1 5FBAF40F
 P 6000 4050
@@
 $EndComp
 $Comp
-L power:+5V #PWR0108
+L boneIO---input-board-rescue:+5V-power #PWR0108
 U 1 1 5FBB3985
 P 9700 4300
@@
 $EndComp
 $Comp
-L power:GND #PWR0109
+L boneIO---input-board-rescue:GND-power #PWR0109
 U 1 1 5FBB4249
 P 10500 2250
@@
 $EndComp
 $Comp
-L Connector:Screw_Terminal_01x08 J7
+L boneIO---input-board-rescue:Screw_Terminal_01x08-Connector J7
 U 1 1 5FBC0ABF
 P 2550 1600
@@
 $EndComp
 $Comp
-L Connector:Screw_Terminal_01x08 J6
+L boneIO---input-board-rescue:Screw_Terminal_01x08-Connector J6
 U 1 1 5FBC27EC
 P 3500 1600
@@
 $EndComp
 $Comp
-L Connector:Screw_Terminal_01x08 J5
+L boneIO---input-board-rescue:Screw_Terminal_01x08-Connector J5
 U 1 1 5FBC4BBE
 P 4450 1600
@@
 $EndComp
 $Comp
-L Connector:Screw_Terminal_01x08 J2
+L boneIO---input-board-rescue:Screw_Terminal_01x08-Connector J2
 U 1 1 5FBC66CA
 P 3150 5600
@@
 $EndComp
 $Comp
-L power:GND #PWR0113
+L boneIO---input-board-rescue:GND-power #PWR0113
 U 1 1 5FBCF9DC
 P 1500 5050
@@
 $EndComp
 $Comp
-L power:GND #PWR0114
+L boneIO---input-board-rescue:GND-power #PWR0114
 U 1 1 5FBCFD71
 P 6000 3150
@@
 $EndComp
 $Comp
-L Connector:Screw_Terminal_01x08 J3
+L boneIO---input-board-rescue:Screw_Terminal_01x08-Connector J3
 U 1 1 5FCC407F
 P 4200 5600
@@
 $EndComp
 $Comp
-L Connector:Screw_Terminal_01x08 J4
+L boneIO---input-board-rescue:Screw_Terminal_01x08-Connector J4
 U 1 1 5FCC570E
 P 5150 5600
@@
 $EndComp
 $Comp
-L Connector:Screw_Terminal_01x03 J1
+L boneIO---input-board-rescue:Screw_Terminal_01x03-Connector J1
 U 1 1 5FD7EAE8
 P 2300 5600
@@
 $EndComp
 $Comp
-L Connector:Screw_Terminal_01x02 VDD1
+L boneIO---input-board-rescue:Screw_Terminal_01x02-Connector VDD1
 U 1 1 5FDB330F
 P 5950 6950
@@
 $EndComp
 $Comp
-L power:GND #PWR0118
+L boneIO---input-board-rescue:GND-power #PWR0118
 U 1 1 5FDB3CFF
 P 5600 7350
@@
 $EndComp
 $Comp
-L power:+5V #PWR0119
+L boneIO---input-board-rescue:+5V-power #PWR0119
 U 1 1 5FDB44B3
 P 5550 6650
@@
 	5600 7050 5600 7350
 $Comp
-L power:+3.3V #PWR0121
+L boneIO---input-board-rescue:+3.3V-power #PWR0121
 U 1 1 5FDDE18D
 P 9850 4650
@@
 $EndComp
 $Comp
-L Connector_Generic:Conn_01x04 I2C1
+L boneIO---input-board-rescue:Conn_01x04-Connector_Generic I2C1
 U 1 1 5FDF9F1B
 P 9900 3750
@@
 $EndComp
 $Comp
-L power:+3.3V #PWR0122
+L boneIO---input-board-rescue:+3.3V-power #PWR0122
 U 1 1 5FDFA9B6
 P 9900 3400
@@
 $EndComp
 $Comp
-L power:GND #PWR0123
+L boneIO---input-board-rescue:GND-power #PWR0123
 U 1 1 5FDFB41B
 P 8200 4800
@@
 $EndComp
 $Comp
-L Connector:Screw_Terminal_01x02 ANVDD1
+L boneIO---input-board-rescue:Screw_Terminal_01x02-Connector ANVDD1
 U 1 1 5FE784F5
 P 8700 2200
@@
 $EndComp
 $Comp
-L Connector:Screw_Terminal_01x07 AN1
+L boneIO---input-board-rescue:Screw_Terminal_01x07-Connector AN1
 U 1 1 5FE99E8D
 P 7750 5450
@@
 $EndComp
 $Comp
-L Connector_Generic:Conn_02x23_Odd_Even P8
+L boneIO---input-board-rescue:Conn_02x23_Odd_Even-Connector_Generic P8
 U 1 1 55DF7DE1
 P 1550 3600
@@
 NoConn ~ 9000 4450
 $Comp
-L Switch:SW_Push SW1
+L boneIO---input-board-rescue:SW_Push-Switch SW1
 U 1 1 60E68B6D
 P 10750 2550
@@
 	10500 2350 10750 2350
 $Comp
-L Switch:SW_Push SW2
+L boneIO---input-board-rescue:SW_Push-Switch SW2
 U 1 1 60E913E3
 P 8750 4600
@@
 $EndComp
 $Comp
-L Mechanical:MountingHole H1
+L boneIO---input-board-rescue:MountingHole-Mechanical H1
 U 1 1 6082D678
 P 2850 6550
@@
 $EndComp
 $Comp
-L Mechanical:MountingHole H2
+L boneIO---input-board-rescue:MountingHole-Mechanical H2
 U 1 1 6082DBB5
 P 4350 6600
@@
 	2350 2450 2350 1800
 $Comp
-L power:GND #PWR0102
+L boneIO---input-board-rescue:GND-power #PWR0102
 U 1 1 60F14745
 P 2400 5150
@@
 $EndComp
 $Comp
-L power:GND #PWR0103
+L boneIO---input-board-rescue:GND-power #PWR0103
 U 1 1 60F15484
 P 3450 5150
@@
 $EndComp
 $Comp
-L power:GND #PWR0105
+L boneIO---input-board-rescue:GND-power #PWR0105
 U 1 1 60F159E6
 P 4500 5150
@@
 $EndComp
 $Comp
-L power:GND #PWR0106
+L boneIO---input-board-rescue:GND-power #PWR0106
 U 1 1 60F15BC0
 P 5450 5150
@@
 	5450 5150 5450 5400
 $Comp
-L power:GND #PWR0110
+L boneIO---input-board-rescue:GND-power #PWR0110
 U 1 1 60F7ECAD
 P 4150 2000
@@
 $EndComp
 $Comp
-L power:GND #PWR0111
+L boneIO---input-board-rescue:GND-power #PWR0111
 U 1 1 60F7FFFD
 P 3200 2000
@@
 $EndComp
 $Comp
-L power:GND #PWR0112
+L boneIO---input-board-rescue:GND-power #PWR0112
 U 1 1 60F80392
 P 2250 2000
