File: Circuit/boneIO - input board/boneIO_input board_v0.2.sch (KiCad schematic (older format))
At the start: 175 parts, among them J1 I2C_OUT, J2 Screw_Terminal_01x08, J3 Screw_Terminal_01x08, J4 Screw_Terminal_01x08, J5 Screw_Terminal_01x08, J6 Screw_Terminal_01x08, J7 Screw_Terminal_01x08, J9 Conn_02x13_Odd_Even, P3 BeagleBone_Black_Header, P4 BeagleBone_Black_Header, SW1 SW_Push, U1 LM2596S-ADJ, U10 PC847, U11 PC847, U12 PC847, U13 DS1307Z+, U2 PC847, U3 PC847, U4 PC847, U5 PC847, U6 PC847, U7 PC847, U8 PC847, U9 PC847, Y1 32,788 MHz

Commit message: Zmiany 27-10-2021
nowa PCB
Parts:
- removed AN1: Screw_Terminal_01x07, Connector_Phoenix_MSTB:PhoenixContact_MSTBA_2,5_7-G_1x07_P5.00mm_Horizontal, symbol Connector:Screw_Terminal_01x07
- removed C10, C17, C18, C9: 100n, Capacitor_SMD:C_0603_1608Metric, symbol Device:C
- removed J1: I2C_OUT, Connector:Phoenix_1x04_P5.00mm_Horizontal, symbol Connector:Screw_Terminal_01x04
- removed R15, R16, R17, R30, R36, R37, R42, R51, R52, R53, R54, R55, R56, R57, R58, R59, R60, R61, R62, R63, R64, R65, R66, R67, R68, R69, R70, R71, R72, R73, R74, R75, R76, R77, R78, R79, R80, R81, R82, R83, R84, R85, R86, R87, R88, R89, R90, R91: 10k, Resistor_SMD:R_0603_1608Metric, symbol Device:R
- removed U10, U11, U12, U2, U3, U4, U5, U6, U7, U8, U9: PC847, Package_SO:SOP-16_4.55x10.3mm_P1.27mm, symbol Isolator:PC847
- added C31, C39, C43, C44: 100n, Capacitor_SMD:C_0603_1608Metric, symbol Device:C
- added J7, J9: Screw_Terminal_01x08, Connector:8pin, symbol Connector:Screw_Terminal_01x08
- added PS1: B2424S-1WR2, CONV_B0505S-1WR2, symbol Power_Management:B2424S-1WR2
- added R39, R45, R46, R47, R48, R49: 10k, Resistor_SMD:R_0603_1608Metric, symbol Device:R
- added U1, U10, U11, U12, U13, U14, U15, U16, U17, U18, U19, U2, U20, U21, U22, U23, U24, U25, U26, U27, U29, U3, U30, U31, U32, U34, U35, U36, U37, U38, U39, U4, U40, U41, U42, U43, U44, U45, U5, U6, U7, U8: EL357N-G, Package_SO:OPTO_EL357N-G, symbol Isolator:PC817
- added U28: RS485, Module:RS485_moduleTTL, symbol RF_Module:RS485
- BT1: footprint Battery:BatteryHolder_Keystone_103_1x20mm -> Battery:Battery_Panasonic_CR1220-VCN_Vertical_CircularHoles
- SW1: footprint Button_Switch_THT:SW_PUSH_6mm_H8mm -> Button_Switch_THT:SW_PUSH_6mm_H13mm
- Y1: footprint Crystal:Crystal_C38-LF_D3.0mm_L8.0mm_Horizontal_1EP_style1 -> Crystal:Crystal_C26-LF_D2.1mm_L6.5mm_Horizontal
- renumbered C44 to C10, C47 to C17, C48 to C18, C43 to C9, D2 to D1, D3 to D2, D4 to D3, J3 to J1, J5 to J2, J4 to J3, J6 to J4, J2 to J5, J7 to J6, J9 to J8, L2 to L1, L1 to L2, P4 to P1, P3 to P2, R47 to R15, R48 to R16, R49 to R17, R45 to R30, R46 to R31, R94 to R36, R95 to R37, R96 to R42, U13 to U33, U1 to U9
Connections:
- net labels added: +24VA, A+, B-, GNDD, GND_ADC, P8.03_OUT, P8.04_OUT, P8.05_OUT, P8.06_OUT, P8.07_OUT, P8.08_OUT, P8.09_OUT, P8.10_OUT, P8.11_OUT, P8.12_OUT, P8.14_OUT, P8.15_OUT, P8.16_OUT, P8.17_OUT, P8.18_OUT, P8.20_OUT, P8.21_OUT, P8.22_OUT, P8.23_OUT, P8.24_OUT, P8.25_OUT, P8.26_OUT, P8.27_OUT, P8.28_OUT, P8.29_OUT, P8.30_OUT, P8.31_OUT, P8.32_OUT, P8.33_OUT, P8.34_OUT, P8.35_OUT, P8.36_OUT, P8.37_OUT, P8.38_OUT, P8.39_OUT, P8.40_OUT, P8.41_OUT, P8.42_OUT, P8.43_OUT, P8.44_OUT, P8.45_OUT, P8.46_OUT, VDD_ADC
- net labels removed: P9.24, P9.26, P9.32, P9.34
- wire segments 829 -> 625
Other:
- note removed: "Pull_Up\n"
- moved on the sheet: ANVDD1, BT1, C10, C17, C18, C9, D1, D2, D3, F1, I2C1, J1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

Commit message: Aktualizacja 28_10_2021
Parts:
- C1, C10, C11, C12, C13, C14, C15, C16, C19, C2, C20, C21, C22, C23, C24, C25, C26, C27, C28, C29, C3, C30, C31, C32, C33, C34, C35, C36, C37, C38, C39, C4, C40, C41, C42, C43, C44, C45, C46, C5, C6, C7, C8: JLCPCB (none) -> C14663
- C17: JLCPCB (none) -> C107149
- C18: JLCPCB (none) -> C311611
- C9: value 100u/50V -> 100uF/50V; JLCPCB (none) -> C72480
- D1: JLCPCB (none) -> C64982
- D2: value 1N5825 -> SS34; JLCPCB (none) -> C8678
- D3: value LED_GREEN -> LED_RED; JLCPCB (none) -> C84256
- F1: JLCPCB (none) -> C136367
- L1: value 4,7uH -> 4.7uH; JLCPCB (none) -> C338848
- L2: JLCPCB (none) -> C85840
- PS1: JLCPCB (none) -> C91799
- R1, R10, R11, R12, R13, R14, R18, R19, R2, R20, R21, R22, R23, R24, R25, R26, R27, R28, R29, R3, R32, R33, R34, R35, R36, R37, R38, R39, R4, R40, R41, R42, R43, R44, R45, R46, R47, R48, R49, R5, R50, R6, R7, R8, R9: JLCPCB (none) -> C238881
- R15: JLCPCB (none) -> C126358
- R16, R17: JLCPCB (none) -> C269704
- R30, R31: JLCPCB (none) -> C101062
- RV1: JLCPCB (none) -> C317745
- U1, U10, U11, U12, U13, U14, U15, U16, U17, U18, U19, U2, U20, U21, U22, U23, U24, U25, U26, U27, U29, U3, U30, U31, U32, U34, U35, U36, U37, U38, U39, U4, U40, U41, U42, U43, U44, U45, U5, U6, U7, U8: JLCPCB (none) -> C6649
- U33: JLCPCB (none) -> C26858

Commit message: Zmiany 28.10.2021_2
Parts:
- removed P1, P2: BeagleBone_Black_Header, Connector_PinHeader_2.54mm:PinHeader_2x23_P2.54mm_Vertical, symbol Connector_Generic:Conn_02x23_Odd_Even
- added C47: 100n, Capacitor_SMD:C_0603_1608Metric, symbol Device:C
- added D4: BAT54A, Package_TO_SOT_SMD:SOT-23, symbol Diode:BAT54A
- added J10, J11: BeagleBone_Black_Header, Connector_PinHeader_2.54mm:PinHeader_2x23_P2.54mm_Vertical, symbol Connector_Generic:BeagleBone_Black_Header
- added R51, R52: 680R, Resistor_SMD:R_0603_1608Metric, symbol Device:R
- added U46: P82B96, Package_SO:SO-8_3.9x4.9mm_P1.27mm, symbol Interface_Expansion:P82B96
Connections:
- net +3V3: now also C47.1, J10.3 (Pin_3), J10.4 (Pin_4), R51.1, R52.1, U46.8 (VCC)
- net +5V: now also J10.5 (Pin_5), J10.6 (Pin_6)
- net GND: now also C47.2, D4.3, J10.1 (Pin_1), J10.2 (Pin_2), J10.43 (Pin_43), J10.44 (Pin_44), J10.45 (Pin_45), J10.46 (Pin_46), J11.1 (Pin_1), J11.2 (Pin_2), U46.4 (GND)
- net GND_ADC: now also J10.34 (Pin_34)
- net P8.03: now also J11.3 (Pin_3)
- net P8.04: now also J11.4 (Pin_4)
- net P8.05: now also J11.5 (Pin_5)
- net P8.06: now also J11.6 (Pin_6)
- net P8.07: now also J11.7 (Pin_7)
- net P8.08: now also J11.8 (Pin_8)
- net P8.09: now also J11.9 (Pin_9)
- net P8.10: now also J11.10 (Pin_10)
- net P8.11: now also J11.11 (Pin_11)
- net P8.12: now also J11.12 (Pin_12)
- net P8.13: now also J11.13 (Pin_13)
- net P8.14: now also J11.14 (Pin_14)
- net P8.15: now also J11.15 (Pin_15)
- net P8.16: now also J11.16 (Pin_16)
- net P8.17: now also J11.17 (Pin_17)
- net P8.18: now also J11.18 (Pin_18)
- net P8.19: now also J11.19 (Pin_19)
- net P8.20: now also J11.20 (Pin_20)
- net P8.21: now also J11.21 (Pin_21)
- net P8.22: now also J11.22 (Pin_22)
- net P8.23: now also J11.23 (Pin_23)
- net P8.24: now also J11.24 (Pin_24)
- net P8.25: now also J11.25 (Pin_25)
- net P8.26: now also J11.26 (Pin_26)
- net P8.26_OUT: now also J3.8 (Pin_8); no longer J5.8 (Pin_8)
- net P8.27: now also J11.27 (Pin_27)
- net P8.27_OUT: now also J3.7 (Pin_7); no longer J5.7 (Pin_7)
- net P8.28: now also J11.28 (Pin_28)
- net P8.28_OUT: now also J3.6 (Pin_6); no longer J5.6 (Pin_6)
- net P8.29: now also J11.29 (Pin_29)
- net P8.29_OUT: now also J3.5 (Pin_5); no longer J5.5 (Pin_5)
- net P8.30: now also J11.30 (Pin_30)
- net P8.30_OUT: now also J3.4 (Pin_4); no longer J5.4 (Pin_4)
- net P8.31: now also J11.31 (Pin_31)
- net P8.31_OUT: now also J3.3 (Pin_3); no longer J5.3 (Pin_3)
- net P8.32: now also J11.32 (Pin_32)
- net P8.32_OUT: now also J3.2 (Pin_2); no longer J5.2 (Pin_2)
- net P8.33: now also J11.33 (Pin_33)
- net P8.33_OUT: now also J1.8 (Pin_8); no longer J3.8 (Pin_8)
- net P8.34: now also J11.34 (Pin_34)
- net P8.34_OUT: now also J1.7 (Pin_7); no longer J3.7 (Pin_7)
- net P8.35: now also J11.35 (Pin_35)
- net P8.35_OUT: now also J1.6 (Pin_6); no longer J3.6 (Pin_6)
- net P8.36: now also J11.36 (Pin_36)
- net P8.36_OUT: now also J1.5 (Pin_5); no longer J3.5 (Pin_5)
- net P8.37: now also J11.37 (Pin_37)
- net P8.37_OUT: now also J1.4 (Pin_4); no longer J3.4 (Pin_4)
- net P8.38: now also J11.38 (Pin_38)
- net P8.38_OUT: now also J1.3 (Pin_3); no longer J3.3 (Pin_3)
- net P8.39: now also J11.39 (Pin_39)
- net P8.39_OUT: now also J1.2 (Pin_2); no longer J3.2 (Pin_2)
- net P8.40: now also J11.40 (Pin_40)
- net P8.40_OUT: now also J5.8 (Pin_8); no longer J1.8 (Pin_8)
- net P8.41: now also J11.41 (Pin_41)
- net P8.41_OUT: now also J5.7 (Pin_7); no longer J1.7 (Pin_7)
- net P8.42: now also J11.42 (Pin_42)
- net P8.42_OUT: now also J5.6 (Pin_6); no longer J1.6 (Pin_6)
- net P8.43: now also J11.43 (Pin_43)
- net P8.43_OUT: now also J5.5 (Pin_5); no longer J1.5 (Pin_5)
- net P8.44: now also J11.44 (Pin_44)
- net P8.44_OUT: now also J5.4 (Pin_4); no longer J1.4 (Pin_4)
- net P8.45: now also J11.45 (Pin_45)
- net P8.45_OUT: now also J5.3 (Pin_3); no longer J1.3 (Pin_3)
- net P8.46: now also J11.46 (Pin_46)
- net P8.46_OUT: now also J5.2 (Pin_2); no longer J1.2 (Pin_2)
- net P9.11: now also J10.11 (Pin_11)
- net P9.12: now also J10.12 (Pin_12)
- net P9.13: now also J10.13 (Pin_13)
- net P9.14: now also J10.14 (Pin_14)
- net P9.15: now also J10.15 (Pin_15)
- net P9.16: now also J10.16 (Pin_16)
- net P9.17: now also J10.17 (Pin_17)
- net P9.18: now also J10.18 (Pin_18)
- net P9.21: now also J10.21 (Pin_21)
- net P9.22: now also J10.22 (Pin_22)
- net P9.23: now also J10.23 (Pin_23)
- net P9.25: now also J10.25 (Pin_25)
- net P9.27: now also J10.27 (Pin_27)
- net P9.28: now also J10.28 (Pin_28)
- net P9.29: now also J10.29 (Pin_29)
- net P9.30: now also J10.30 (Pin_30)
- net P9.31: now also J10.31 (Pin_31)
- net P9.33: now also J10.33 (Pin_33)
- net P9.35: now also J10.35 (Pin_35)
- net P9.36: now also J10.36 (Pin_36)
- net P9.37: now also J10.37 (Pin_37)
- net P9.38: now also J10.38 (Pin_38)
- net P9.39: now also J10.39 (Pin_39)
- net P9.40: now also J10.40 (Pin_40)
- net P9.41: now also J10.41 (Pin_41)
- net P9.42: now also J10.42 (Pin_42)
- net RX: now also J10.26 (Pin_26)
- net SCL: now also J10.19 (Pin_19), U46.7 (SCL); no longer J9.4 (Pin_4)
- net SDA: now also J10.20 (Pin_20), U46.1 (SDA); no longer J9.5 (Pin_5)
- net TX: now also J10.24 (Pin_24)
- net VDD_ADC: now also J10.32 (Pin_32)
- new net SCL_OUT: D4.1, J9.5 (Pin_5), R51.2, U46.5 (TXD-SCL), U46.6 (RXD-SCL)
- new net SDA_OUT: D4.2, J9.4 (Pin_4), R52.2, U46.2 (RXD-SDA), U46.3 (TXD-SDA)
- no-connect marks 4 -> 1
