File: Circuit/boneIO - input board/boneIO_input board_v0.2.sch (KiCad schematic (older format))
At the start: 171 parts, among them J1 Screw_Terminal_01x08, J10 BeagleBone_Black_Header, J11 BeagleBone_Black_Header, J2 Screw_Terminal_01x08, J3 Screw_Terminal_01x08, J4 Screw_Terminal_01x08, J5 Screw_Terminal_01x08, J6 Screw_Terminal_01x08, J7 Screw_Terminal_01x08, J8 Conn_02x13_Odd_Even, J9 Screw_Terminal_01x08, SW1 SW_Push, U1 EL357N-G, U10 EL357N-G, U11 EL357N-G, U12 EL357N-G, U13 EL357N-G, U14 EL357N-G, U15 EL357N-G, U16 EL357N-G, U17 EL357N-G, U18 EL357N-G, U19 EL357N-G, U2 EL357N-G, U20 EL357N-G, U21 EL357N-G, U22 EL357N-G, U23 EL357N-G, U24 EL357N-G, U25 EL357N-G, U26 EL357N-G, U27 EL357N-G, U28 RS485, U29 EL357N-G, U3 EL357N-G, U30 EL357N-G, U31 EL357N-G, U32 EL357N-G, U33 DS1307Z+, U34 EL357N-G, U35 EL357N-G, U36 EL357N-G, U37 EL357N-G, U38 EL357N-G, U39 EL357N-G, U4 EL357N-G, U40 EL357N-G, U41 EL357N-G, U42 EL357N-G, U43 EL357N-G, U44 EL357N-G, U45 EL357N-G, U46 P82B96, U5 EL357N-G, U6 EL357N-G, U7 EL357N-G, U8 EL357N-G, U9 LM2596S-ADJ, Y1 32,788 MHz

Commit message: Input Board_v0.2_F
PCB ukończone do sprawdzenia.
Parts:
- added C48: 100n, Capacitor_SMD:C_0603_1608Metric, symbol Device:C
- added D5: 1N4148, Diode_SMD:D_MiniMELF, symbol Device:D
- added R53: 330R, Resistor_SMD:R_0603_1608Metric, symbol Device:R
- added R54: 4.7k, Resistor_SMD:R_0603_1608Metric, symbol Device:R
Connections:
- wire segments 630 -> 638
Other:
- moved on the sheet: SW1
Changed lines of the file:
@@
 	10450 12500 10600 12500
 Wire Wire Line
-	8700 1800 8700 1900
+	8650 1800 8650 1900
 Wire Wire Line
-	8950 1800 8700 1800
-Wire Wire Line
-	8700 2300 8700 2500
-Text Notes 8400 1750 0    157  ~ 31
+	8650 2600 8650 2800
+Text Notes 8500 1400 0    157  ~ 31
 Switch\n\n
 Text Notes 15900 13150 0    157  ~ 31
@@
 Text GLabel 13700 13200 0    50   Input ~ 0
 P9.33
-Text GLabel 8950 1800 2    50   Input ~ 0
+Text GLabel 9550 1800 2    50   Input ~ 0
 P9.41
 Wire Wire Line
@@
 Text GLabel 16950 14200 2    50   Input ~ 0
 P9.27
-Text GLabel 16950 14400 2    50   Input ~ 0
+Text GLabel 16950 14300 2    50   Input ~ 0
 P9.25
-Text GLabel 16950 14600 2    50   Input ~ 0
+Text GLabel 16950 14400 2    50   Input ~ 0
 P9.23
 Text GLabel 11400 2100 0    50   Input ~ 0
@@
 Text GLabel 16450 14200 0    50   Input ~ 0
 P9.16
-Text GLabel 16450 14300 0    50   Input ~ 0
+Text GLabel 16450 14500 0    50   Input ~ 0
 P9.17
-Text GLabel 16450 14400 0    50   Input ~ 0
+Text GLabel 16450 14600 0    50   Input ~ 0
 P9.18
-Text GLabel 16450 14500 0    50   Input ~ 0
+Text GLabel 16950 14600 2    50   Input ~ 0
 P9.21
-Text GLabel 16450 14600 0    50   Input ~ 0
+Text GLabel 16950 14500 2    50   Input ~ 0
 P9.22
 Text GLabel 5200 12850 2    50   Input ~ 0
@@
 L Switch:SW_Push SW1
 U 1 1 618FEB23
-P 8700 2100
-F 0 "SW1" V 8654 2248 50  0000 L CNN
-F 1 "SW_Push" V 8745 2248 50  0000 L CNN
-F 2 "Button_Switch_THT:SW_PUSH_6mm_H13mm" H 8700 2300 50  0001 C CNN
-F 3 "~" H 8700 2300 50  0001 C CNN
-	1    8700 2100
+P 8650 2100
+F 0 "SW1" V 8604 2248 50  0000 L CNN
+F 1 "SW_Push" V 8695 2248 50  0000 L CNN
+F 2 "Button_Switch_THT:SW_PUSH_6mm_H13mm" H 8650 2300 50  0001 C CNN
+F 3 "~" H 8650 2300 50  0001 C CNN
+	1    8650 2100
 	0    -1   -1   0
 $EndComp
@@
 L power:GND #PWR035
 U 1 1 618FEB0F
-P 8700 2500
-F 0 "#PWR035" H 8700 2250 50  0001 C CNN
-F 1 "GND" H 8705 2327 50  0000 C CNN
-F 2 "" H 8700 2500 50  0001 C CNN
-F 3 "" H 8700 2500 50  0001 C CNN
-	1    8700 2500
+P 8650 2800
+F 0 "#PWR035" H 8650 2550 50  0001 C CNN
+F 1 "GND" H 8655 2627 50  0000 C CNN
+F 2 "" H 8650 2800 50  0001 C CNN
+F 3 "" H 8650 2800 50  0001 C CNN
+	1    8650 2800
 	1    0    0    -1
 $EndComp
@@
 Wire Wire Line
 	20400 13600 20400 13700
-Text GLabel 16950 14300 2    50   Input ~ 0
+Text GLabel 16450 14400 0    50   Input ~ 0
 P8.19
-Text GLabel 16950 14500 2    50   Input ~ 0
+Text GLabel 16450 14300 0    50   Input ~ 0
 P8.13
 Text GLabel 13700 14800 3    50   Input ~ 0
@@
 	21650 3800 21500 3800
 NoConn ~ 13700 13300
+$Comp
+L Device:R R53
+U 1 1 62D25CAC
+P 8650 2450
+F 0 "R53" H 8720 2496 50  0000 L CNN
+F 1 "330R" H 8720 2405 50  0000 L CNN
+F 2 "Resistor_SMD:R_0603_1608Metric" V 8580 2450 50  0001 C CNN
+F 3 "~" H 8650 2450 50  0001 C CNN
+F 4 "C101062" H 8650 2450 50  0001 C CNN "JLCPCB"
+	1    8650 2450
+	1    0    0    -1
+$EndComp
+$Comp
+L Device:C C48
+U 1 1 62FDF461
+P 9050 2450
+F 0 "C48" H 9165 2496 50  0000 L CNN
+F 1 "100n" H 9165 2405 50  0000 L CNN
+F 2 "Capacitor_SMD:C_0603_1608Metric" H 9088 2300 50  0001 C CNN
+F 3 "~" H 9050 2450 50  0001 C CNN
+F 4 "C14663" H 9050 2450 50  0001 C CNN "JLCPCB"
+	1    9050 2450
+	1    0    0    -1
+$EndComp
+Wire Wire Line
+	9050 1800 9050 2300
+Wire Wire Line
+	8650 1800 9050 1800
+Wire Wire Line
+	9050 2600 9050 2800
+$Comp
+L power:GND #PWR0106
+U 1 1 630C9F71
+P 9050 2800
+F 0 "#PWR0106" H 9050 2550 50  0001 C CNN
+F 1 "GND" H 9055 2627 50  0000 C CNN
+F 2 "" H 9050 2800 50  0001 C CNN
+F 3 "" H 9050 2800 50  0001 C CNN
+	1    9050 2800
+	1    0    0    -1
+$EndComp
+$Comp
+L Device:R R54
+U 1 1 631B3AD2
+P 9050 1600
+F 0 "R54" H 9120 1646 50  0000 L CNN
+F 1 "4.7k" H 9120 1555 50  0000 L CNN
+F 2 "Resistor_SMD:R_0603_1608Metric" V 8980 1600 50  0001 C CNN
+F 3 "~" H 9050 1600 50  0001 C CNN
+F 4 "C101062" H 9050 1600 50  0001 C CNN "JLCPCB"
+	1    9050 1600
+	1    0    0    -1
+$EndComp
+Wire Wire Line
+	9050 1800 9050 1750
+Connection ~ 9050 1800
+$Comp
+L power:+3.3V #PWR0107
+U 1 1 634008CE
+P 9050 1400
+F 0 "#PWR0107" H 9050 1250 50  0001 C CNN
+F 1 "+3.3V" H 9065 1573 50  0000 C CNN
+F 2 "" H 9050 1400 50  0001 C CNN
+F 3 "" H 9050 1400 50  0001 C CNN
+	1    9050 1400
+	1    0    0    -1
+$EndComp
+Wire Wire Line
+	9050 1450 9050 1400
+$Comp
+L Device:D D5
+U 1 1 635D8BC6
+P 9350 1600
+F 0 "D5" V 9304 1680 50  0000 L CNN
+F 1 "1N4148" V 9395 1680 50  0000 L CNN
+F 2 "Diode_SMD:D_MiniMELF" H 9350 1600 50  0001 C CNN
+F 3 "~" H 9350 1600 50  0001 C CNN
+	1    9350 1600
+	0    1    1    0
+$EndComp
+Wire Wire Line
+	9050 1800 9350 1800
+Wire Wire Line
+	9350 1800 9350 1750
+Connection ~ 9350 1800
+Wire Wire Line
+	9350 1800 9550 1800
+$Comp
+L power:+3.3V #PWR0108
+U 1 1 637421AB
+P 9350 1400
+F 0 "#PWR0108" H 9350 1250 50  0001 C CNN
+F 1 "+3.3V" H 9365 1573 50  0000 C CNN
+F 2 "" H 9350 1400 50  0001 C CNN
+F 3 "" H 9350 1400 50  0001 C CNN
+	1    9350 1400
+	1    0    0    -1
+$EndComp
+Wire Wire Line
+	9350 1450 9350 1400
 $EndSCHEMATC

Commit message: aktualizacja
Parts:
- removed J8: Conn_02x13_Odd_Even, Connector_PinSocket_2.54mm:PinSocket_2x13_P2.54mm_Vertical, symbol Connector_Generic:Conn_02x13_Odd_Even
- added J12: Conn_02x04_Odd_Even, Connector_PinHeader_2.54mm:PinHeader_2x04_P2.54mm_Vertical, symbol Connector_Generic:Conn_02x04_Odd_Even
Connections:
- wire segments 638 -> 642
Changed lines of the file:
@@
 Text Notes 8500 1400 0    157  ~ 31
 Switch\n\n
-Text Notes 15900 13150 0    157  ~ 31
-Pin_Down_PCB\n\n
-Text GLabel 16950 14700 2    50   Input ~ 0
-SDA
-Text GLabel 16450 14700 0    50   Input ~ 0
-SCL
 Text GLabel 13700 12600 0    50   Input ~ 0
 P9.39
@@
 Text GLabel 9550 1800 2    50   Input ~ 0
 P9.41
-Wire Wire Line
-	15750 14800 15750 13450
-Wire Wire Line
-	16450 14800 15750 14800
-$Comp
-L power:+3.3V #PWR065
-U 1 1 653C1BB9
-P 15750 13450
-F 0 "#PWR065" H 15750 13300 50  0001 C CNN
-F 1 "+3.3V" H 15765 13623 50  0000 C CNN
-F 2 "" H 15750 13450 50  0001 C CNN
-F 3 "" H 15750 13450 50  0001 C CNN
-	1    15750 13450
-	1    0    0    -1
-$EndComp
-$Comp
-L power:+24V #PWR067
-U 1 1 653A44CA
-P 16050 13450
-F 0 "#PWR067" H 16050 13300 50  0001 C CNN
-F 1 "+24V" H 16065 13623 50  0000 C CNN
-F 2 "" H 16050 13450 50  0001 C CNN
-F 3 "" H 16050 13450 50  0001 C CNN
-	1    16050 13450
-	1    0    0    -1
-$EndComp
-Connection ~ 17400 14800
-Wire Wire Line
-	16950 13600 17400 13600
-Wire Wire Line
-	17400 13600 17400 14800
-Wire Wire Line
-	17400 14800 17400 14850
-Wire Wire Line
-	16950 14800 17400 14800
-$Comp
-L power:GND #PWR074
-U 1 1 6534CE80
-P 17400 14850
-F 0 "#PWR074" H 17400 14600 50  0001 C CNN
-F 1 "GND" H 17405 14677 50  0000 C CNN
-F 2 "" H 17400 14850 50  0001 C CNN
-F 3 "" H 17400 14850 50  0001 C CNN
-	1    17400 14850
-	1    0    0    -1
-$EndComp
-Wire Wire Line
-	16050 13600 16050 13450
-Wire Wire Line
-	16450 13600 16050 13600
-Text GLabel 16950 13700 2    50   Input ~ 0
-P9.42
-Text GLabel 16950 13800 2    50   Input ~ 0
-P9.31
-Text GLabel 16950 13900 2    50   Input ~ 0
-P9.30
-Text GLabel 16950 14000 2    50   Input ~ 0
-P9.29
-Text GLabel 16950 14100 2    50   Input ~ 0
-P9.28
-Text GLabel 16950 14200 2    50   Input ~ 0
-P9.27
-Text GLabel 16950 14300 2    50   Input ~ 0
-P9.25
-Text GLabel 16950 14400 2    50   Input ~ 0
-P9.23
 Text GLabel 11400 2100 0    50   Input ~ 0
 SCL
@@
 Wire Wire Line
 	12300 1900 12150 1900
-Text GLabel 16450 13700 0    50   Input ~ 0
-P9.11
-Text GLabel 16450 13800 0    50   Input ~ 0
-P9.12
-Text GLabel 16450 13900 0    50   Input ~ 0
-P9.13
-Text GLabel 16450 14000 0    50   Input ~ 0
-P9.14
-Text GLabel 16450 14100 0    50   Input ~ 0
-P9.15
-Text GLabel 16450 14200 0    50   Input ~ 0
-P9.16
-Text GLabel 16450 14500 0    50   Input ~ 0
-P9.17
-Text GLabel 16450 14600 0    50   Input ~ 0
-P9.18
-Text GLabel 16950 14600 2    50   Input ~ 0
-P9.21
-Text GLabel 16950 14500 2    50   Input ~ 0
-P9.22
 Text GLabel 5200 12850 2    50   Input ~ 0
 P8.03
@@
 $EndComp
 $Comp
-L Connector_Generic:Conn_02x13_Odd_Even J8
-U 1 1 61AC45D9
-P 16650 14200
-F 0 "J8" H 16700 15017 50  0000 C CNN
-F 1 "Conn_02x13_Odd_Even" H 16700 14926 50  0000 C CNN
-F 2 "Connector_PinSocket_2.54mm:PinSocket_2x13_P2.54mm_Vertical" H 16650 14200 50  0001 C CNN
-F 3 "~" H 16650 14200 50  0001 C CNN
-	1    16650 14200
-	1    0    0    -1
-$EndComp
-$Comp
 L Switch:SW_Push SW1
 U 1 1 618FEB23
@@
 Wire Wire Line
 	20400 13600 20400 13700
-Text GLabel 16450 14400 0    50   Input ~ 0
-P8.19
-Text GLabel 16450 14300 0    50   Input ~ 0
-P8.13
 Text GLabel 13700 14800 3    50   Input ~ 0
 GND_ADC
@@
 Wire Wire Line
 	9350 1450 9350 1400
+$Comp
+L Connector_Generic:Conn_02x04_Odd_Even J12
+U 1 1 61855C49
+P 18750 13950
+F 0 "J12" H 18800 14267 50  0000 C CNN
+F 1 "Conn_02x04_Odd_Even" H 18800 14176 50  0000 C CNN
+F 2 "Connector_PinHeader_2.54mm:PinHeader_2x04_P2.54mm_Vertical" H 18750 13950 50  0001 C CNN
+F 3 "~" H 18750 13950 50  0001 C CNN
+	1    18750 13950
+	1    0    0    -1
+$EndComp
+$Comp
+L power:+24V #PWR0109
+U 1 1 61857D08
+P 19350 13600
+F 0 "#PWR0109" H 19350 13450 50  0001 C CNN
+F 1 "+24V" H 19365 13773 50  0000 C CNN
+F 2 "" H 19350 13600 50  0001 C CNN
+F 3 "" H 19350 13600 50  0001 C CNN
+	1    19350 13600
+	-1   0    0    -1
+$EndComp
+$Comp
+L power:+5V #PWR0110
+U 1 1 61859D3B
+P 19550 13600
+F 0 "#PWR0110" H 19550 13450 50  0001 C CNN
+F 1 "+5V" H 19565 13773 50  0000 C CNN
+F 2 "" H 19550 13600 50  0001 C CNN
+F 3 "" H 19550 13600 50  0001 C CNN
+	1    19550 13600
+	-1   0    0    -1
+$EndComp
+$Comp
+L power:+3.3V #PWR0111
+U 1 1 6185BCCA
+P 19750 13600
+F 0 "#PWR0111" H 19750 13450 50  0001 C CNN
+F 1 "+3.3V" H 19765 13773 50  0000 C CNN
+F 2 "" H 19750 13600 50  0001 C CNN
+F 3 "" H 19750 13600 50  0001 C CNN
+	1    19750 13600
+	-1   0    0    -1
+$EndComp
+Wire Wire Line
+	19050 13850 19350 13850
+Wire Wire Line
+	19350 13850 19350 13600
+Wire Wire Line
+	19050 13950 19550 13950
+Wire Wire Line
+	19550 13950 19550 13600
+Wire Wire Line
+	19050 14150 19750 14150
+Wire Wire Line
+	19750 14150 19750 13600
+$Comp
+L power:GND #PWR0112
+U 1 1 61C1E0E6
+P 18200 14400
+F 0 "#PWR0112" H 18200 14150 50  0001 C CNN
+F 1 "GND" H 18205 14227 50  0000 C CNN
+F 2 "" H 18200 14400 50  0001 C CNN
+F 3 "" H 18200 14400 50  0001 C CNN
+	1    18200 14400
+	-1   0    0    -1
+$EndComp
+Wire Wire Line
+	18550 14150 18200 14150
+Wire Wire Line
+	18200 14150 18200 14400
+Wire Wire Line
+	18550 13850 18200 13850
+Wire Wire Line
+	18200 13850 18200 13950
+Connection ~ 18200 14150
+Wire Wire Line
+	18550 13950 18200 13950
+Connection ~ 18200 13950
+Wire Wire Line
+	18200 13950 18200 14150
+Text GLabel 18550 14050 0    50   Input ~ 0
+SDA
+Text GLabel 19050 14050 2    50   Input ~ 0
+SCL
+Text Notes 18050 13450 0    157  ~ 31
+Pin_Down_PCB\n\n
 $EndSCHEMATC

Commit message: 01.11.2021
Parts:
- added C49, C50, C51, C52, C53, C54, C55, C56, C57, C58: 100n, Capacitor_SMD:C_0603_1608Metric, symbol Device:C
- added J13: Screw_Terminal_01x04, Connector:Phoenix_1x04_P5.00mm_Horizontal, symbol Connector:Screw_Terminal_01x04
- added J8: Screw_Terminal_01x08, Connector:8pin, symbol Connector:Screw_Terminal_01x08
- added R55, R56, R57, R58, R59, R60, R61, R62, R63, R64: 10k, Resistor_SMD:R_0603_1608Metric, symbol Device:R
- added U47, U48, U49, U50, U51, U52, U53, U54, U55, U56: EL357N-G, Package_SO:OPTO_EL357N-G, symbol Isolator:PC817
Connections:
- net labels added: P9.11_OUT, P9.12_OUT, P9.13_OUT, P9.14_OUT, P9.15_OUT, P9.16_OUT, P9.17_OUT, P9.18_OUT, P9.21_OUT, P9.22_OUT, P9.23_OUT, P9.24, P9.24_OUT, P9.25_OUT, P9.26, P9.26_OUT, P9.27_OUT, P9.28_OUT, P9.29_OUT, P9.30_OUT, P9.31_OUT, P9.42_OUT
- net labels removed: P8.03_OUT, P8.04_OUT, P8.05_OUT, P8.06_OUT, P8.20_OUT, P8.21_OUT, P8.22_OUT, P8.23_OUT, P8.24_OUT, P8.25_OUT
- wire segments 642 -> 746
Other:
- moved on the sheet: BT1, C10, C12, C15, C18, C19, C21, C25, C26, C29, C3, C30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
