File: Circuit/boneIO - input board/boneIO_input board_v0.2.sch (KiCad schematic (older format))
At the start: 184 parts, among them J1 I2C_OUT, J2 Screw_Terminal_01x08, J3 Screw_Terminal_01x08, J4 Screw_Terminal_01x08, J5 Screw_Terminal_01x08, J6 Screw_Terminal_01x08, J7 Screw_Terminal_01x08, J8 Screw_Terminal_01x03, J9 Conn_02x13_Odd_Even, P3 BeagleBone_Black_Header, P4 BeagleBone_Black_Header, SW1 SW_Push, U1 LM2596S-ADJ, U10 PC847, U11 PC847, U12 PC847, U13 DS1307Z+, U2 PC847, U3 PC847, U4 PC847, U5 PC847, U6 PC847, U7 PC847, U8 PC847, U9 PC847, Y1 32,788 MHz

Commit message: Update boneIO_input board_v0.2.sch
aktualizacja pcb
Parts:
- removed D1: B340A-13F, Diode_SMD:D_SMA, symbol Device:D_ALT
- removed J8: Screw_Terminal_01x03, Connector:3pin_5.0, symbol Connector:Screw_Terminal_01x03
- removed PS1: B2424S-1W, Module:CONV_B0505S-1WR2, symbol boneIO_input-board_v0.2-rescue:B0505S-1WR2-power-RelayCH8-rescue
- removed R92, R93: 10k, Resistor_SMD:R_0603_1608Metric, symbol Device:R
Connections:
- net labels added: RX, TX
- net labels removed: +24VA
- wire segments 855 -> 841
Other:
- moved on the sheet: ANVDD1

Commit message: Zmiany TEST
TEST
Parts:
- removed C31, C39: 100n, Capacitor_SMD:C_0603_1608Metric, symbol Device:C
- removed R31, R39: 10k, Resistor_SMD:R_0603_1608Metric, symbol Device:R
Connections:
- wire segments 841 -> 829
Other:
- moved on the sheet: C37, R37
Changed lines of the file:
@@
 Connection ~ 3400 18500
 $Comp
-L Device:C C39
-U 1 1 66A062C9
-P 3850 18750
-F 0 "C39" H 3965 18796 50  0000 L CNN
-F 1 "100n" H 3965 18705 50  0000 L CNN
-F 2 "Capacitor_SMD:C_0603_1608Metric" H 3888 18600 50  0001 C CNN
-F 3 "~" H 3850 18750 50  0001 C CNN
-	1    3850 18750
-	1    0    0    -1
-$EndComp
-$Comp
-L Device:R R39
-U 1 1 66A062CF
-P 3850 18250
-F 0 "R39" H 3920 18296 50  0000 L CNN
-F 1 "10k" H 3920 18205 50  0000 L CNN
-F 2 "Resistor_SMD:R_0603_1608Metric" V 3780 18250 50  0001 C CNN
-F 3 "~" H 3850 18250 50  0001 C CNN
-	1    3850 18250
-	1    0    0    -1
-$EndComp
-Wire Wire Line
-	3850 18100 3850 18000
-$Comp
-L power:GND #PWR087
-U 1 1 66A062D6
-P 3850 19000
-F 0 "#PWR087" H 3850 18750 50  0001 C CNN
-F 1 "GND" H 3855 18827 50  0000 C CNN
-F 2 "" H 3850 19000 50  0001 C CNN
-F 3 "" H 3850 19000 50  0001 C CNN
-	1    3850 19000
-	1    0    0    -1
-$EndComp
-Wire Wire Line
-	3850 18900 3850 19000
-Wire Wire Line
-	3850 18500 4150 18500
-Wire Wire Line
-	4150 18500 4150 18350
-Wire Wire Line
-	3850 18500 3850 18600
-Wire Wire Line
-	3850 18400 3850 18500
-Connection ~ 3850 18500
-$Comp
 L Device:C C6
 U 1 1 66FF185D
@@
 Text GLabel 3700 18350 1    50   Input ~ 0
 P8.20
-Text GLabel 4150 18350 1    50   Input ~ 0
-P8.19
 $Comp
 L Device:C C45
@@
 Connection ~ 2900 20050
 $Comp
-L Device:C C31
-U 1 1 673882F4
+L Device:C C37
+U 1 1 6738830D
 P 3350 20300
-F 0 "C31" H 3465 20346 50  0000 L CNN
+F 0 "C37" H 3465 20346 50  0000 L CNN
 F 1 "100n" H 3465 20255 50  0000 L CNN
 F 2 "Capacitor_SMD:C_0603_1608Metric" H 3388 20150 50  0001 C CNN
@@
 $EndComp
 $Comp
-L Device:R R31
-U 1 1 673882FA
+L Device:R R37
+U 1 1 67388313
 P 3350 19800
-F 0 "R31" H 3420 19846 50  0000 L CNN
+F 0 "R37" H 3420 19846 50  0000 L CNN
 F 1 "10k" H 3420 19755 50  0000 L CNN
 F 2 "Resistor_SMD:R_0603_1608Metric" V 3280 19800 50  0001 C CNN
@@
 	3350 19650 3350 19550
 $Comp
-L power:GND #PWR070
-U 1 1 67388301
+L power:GND #PWR083
+U 1 1 6738831A
 P 3350 20550
-F 0 "#PWR070" H 3350 20300 50  0001 C CNN
+F 0 "#PWR083" H 3350 20300 50  0001 C CNN
 F 1 "GND" H 3355 20377 50  0000 C CNN
 F 2 "" H 3350 20550 50  0001 C CNN
@@
 	3350 19950 3350 20050
 Connection ~ 3350 20050
-$Comp
-L Device:C C37
-U 1 1 6738830D
-P 3800 20300
-F 0 "C37" H 3915 20346 50  0000 L CNN
-F 1 "100n" H 3915 20255 50  0000 L CNN
-F 2 "Capacitor_SMD:C_0603_1608Metric" H 3838 20150 50  0001 C CNN
-F 3 "~" H 3800 20300 50  0001 C CNN
-	1    3800 20300
-	1    0    0    -1
-$EndComp
-$Comp
-L Device:R R37
-U 1 1 67388313
-P 3800 19800
-F 0 "R37" H 3870 19846 50  0000 L CNN
-F 1 "10k" H 3870 19755 50  0000 L CNN
-F 2 "Resistor_SMD:R_0603_1608Metric" V 3730 19800 50  0001 C CNN
-F 3 "~" H 3800 19800 50  0001 C CNN
-	1    3800 19800
-	1    0    0    -1
-$EndComp
-Wire Wire Line
-	3800 19650 3800 19550
-$Comp
-L power:GND #PWR083
-U 1 1 6738831A
-P 3800 20550
-F 0 "#PWR083" H 3800 20300 50  0001 C CNN
-F 1 "GND" H 3805 20377 50  0000 C CNN
-F 2 "" H 3800 20550 50  0001 C CNN
-F 3 "" H 3800 20550 50  0001 C CNN
-	1    3800 20550
-	1    0    0    -1
-$EndComp
-Wire Wire Line
-	3800 20450 3800 20550
-Wire Wire Line
-	3800 20050 4100 20050
-Wire Wire Line
-	4100 20050 4100 19900
-Wire Wire Line
-	3800 20050 3800 20150
-Wire Wire Line
-	3800 19950 3800 20050
-Connection ~ 3800 20050
 Text GLabel 1400 19900 1    50   Input ~ 0
 P8.18
@@
 P8.14
 Text GLabel 3650 19900 1    50   Input ~ 0
-P8.13
-Text GLabel 4100 19900 1    50   Input ~ 0
 P8.12
 $Comp
@@
 $EndComp
 $Comp
-L power:+3.3V #PWR0161
-U 1 1 6381C163
-P 3850 18000
-F 0 "#PWR0161" H 3850 17850 50  0001 C CNN
-F 1 "+3.3V" H 3865 18173 50  0000 C CNN
-F 2 "" H 3850 18000 50  0001 C CNN
-F 3 "" H 3850 18000 50  0001 C CNN
-	1    3850 18000
-	1    0    0    -1
-$EndComp
-$Comp
 L power:+3.3V #PWR0162
 U 1 1 638D1315
@@
 $EndComp
 $Comp
-L power:+3.3V #PWR0167
-U 1 1 63C5A8AF
+L power:+3.3V #PWR0168
+U 1 1 63D0F91C
 P 3350 19550
-F 0 "#PWR0167" H 3350 19400 50  0001 C CNN
+F 0 "#PWR0168" H 3350 19400 50  0001 C CNN
 F 1 "+3.3V" H 3365 19723 50  0000 C CNN
 F 2 "" H 3350 19550 50  0001 C CNN
@@
 	1    0    0    -1
 $EndComp
-$Comp
-L power:+3.3V #PWR0168
-U 1 1 63D0F91C
-P 3800 19550
-F 0 "#PWR0168" H 3800 19400 50  0001 C CNN
-F 1 "+3.3V" H 3815 19723 50  0000 C CNN
-F 2 "" H 3800 19550 50  0001 C CNN
-F 3 "" H 3800 19550 50  0001 C CNN
-	1    3800 19550
-	1    0    0    -1
-$EndComp

Commit message: test
Parts:
- removed AN1: Screw_Terminal_01x07, Connector_Phoenix_MSTB:PhoenixContact_MSTBA_2,5_7-G_1x07_P5.00mm_Horizontal, symbol Connector:Screw_Terminal_01x07
- removed C10, C18, C9: 100n, Capacitor_SMD:C_0603_1608Metric, symbol Device:C
- removed C43: 100u/50V, Capacitor_SMD:CP_Elec_8x10, symbol Device:CP
- removed D2: B340A-13F, Diode_SMD:D_SMA, symbol Device:D_ALT
- removed D3: 1N5825, Diode_SMD:D_SMA, symbol Device:D
- removed J1: I2C_OUT, Connector:Phoenix_1x04_P5.00mm_Horizontal, symbol Connector:Screw_Terminal_01x04
- removed J2: Screw_Terminal_01x08, Connector:8pin, symbol Connector:Screw_Terminal_01x08
- removed J9: Conn_02x13_Odd_Even, Connector_PinSocket_2.54mm:PinSocket_2x13_P2.54mm_Vertical, symbol Connector_Generic:Conn_02x13_Odd_Even
- removed L2: 4,7uH, Inductor_SMD:L_12x12mm_H6mm, symbol Device:L
- removed P3, P4: BeagleBone_Black_Header, Connector_PinHeader_2.54mm:PinHeader_2x23_P2.54mm_Vertical, symbol Connector_Generic:Conn_02x23_Odd_Even
- removed R15, R17, R42, R65, R66, R67, R68, R69, R70, R71, R72, R73, R74, R75, R76, R77, R78, R79, R80, R81, R82, R83, R84, R85, R86, R87, R88, R89, R90, R91, R94, R95: 10k, Resistor_SMD:R_0603_1608Metric, symbol Device:R
- removed U1: LM2596S-ADJ, Package_TO_SOT_SMD:TO-263-5_TabPin3, symbol Regulator_Switching:LM2596S-ADJ
- removed U10, U11, U12, U2, U3, U4, U5, U6, U7, U8, U9: PC847, Package_SO:SOP-16_4.55x10.3mm_P1.27mm, symbol Isolator:PC847
- added C31, C39, C43, C44, C48, C49, C50, C51, C52, C53, C54, C55, C56, C57, C58: 100n, Capacitor_SMD:C_0603_1608Metric, symbol Device:C
- added C9: 100uF/50V, Capacitor_SMD:CP_Elec_8x10, symbol Device:CP
- added D1: B340A-13F, Diode_SMD:D_SMA, symbol Device:D_ALT
- added D2: SS34, Diode_SMD:D_SMA, symbol Device:D
- added D4: BAT54A, Package_TO_SOT_SMD:SOT-23, symbol Diode:BAT54A
- added D5: 1N4148, Diode_SMD:D_MiniMELF, symbol Device:D
- added J10, J11: BeagleBone_Black_Header, Connector_PinHeader_2.54mm:PinHeader_2x23_P2.54mm_Vertical, symbol Connector_Generic:BeagleBone_Black_Header
- added J12: Conn_02x04_Odd_Even, Connector_PinHeader_2.54mm:PinHeader_2x04_P2.54mm_Vertical, symbol Connector_Generic:Conn_02x04_Odd_Even
- added J13: Screw_Terminal_01x04, Connector:Phoenix_1x04_P5.00mm_Horizontal, symbol Connector:Screw_Terminal_01x04
- added J5, J7, J8, J9: Screw_Terminal_01x08, Connector:8pin, symbol Connector:Screw_Terminal_01x08
- added L1: 4.7uH, Inductor_SMD:L_12x12mm_H6mm, symbol Device:L
- added PS1: B2424S-1WR2, CONV_B0505S-1WR2, symbol Power_Management:B2424S-1WR2
- added R31: 4.7k, Resistor_SMD:R_0603_1608Metric, symbol Device:R
- added R39, R47, R49: 10k, Resistor_SMD:R_0603_1608Metric, symbol Device:R
- added U1, U10, U11, U12, U13, U14, U15, U16, U17, U18, U19, U2, U20, U21, U22, U23, U24, U25, U26, U27, U29, U3, U30, U31, U32, U34, U35, U36, U37, U38, U39, U4, U40, U41, U42, U43, U44, U45, U47, U48, U49, U5, U50, U51, U52, U53, U54, U55, U56, U6, U7, U8: EL357N-G, Package_SO:OPTO_EL357N-G, symbol Isolator:PC817
- added U28: RS485, Module:RS485_moduleTTL, symbol RF_Module:RS485
- added U46: P82B96, Package_SO:SO-8_3.9x4.9mm_P1.27mm, symbol Interface_Expansion:P82B96
- added U9: LM2596S-ADJ, Package_TO_SOT_SMD:TO-263-5_TabPin3, symbol Regulator_Switching:LM2596S-ADJ
- BT1: footprint Battery:BatteryHolder_Keystone_103_1x20mm -> Battery:Battery_Panasonic_CR1220-VCN_Vertical_CircularHoles
- C1, C11, C12, C13, C14, C15, C16, C19, C2, C20, C21, C22, C23, C24, C25, C26, C27, C28, C29, C3, C30, C32, C33, C34, C35, C36, C37, C38, C4, C40, C41, C42, C45, C46, C5, C6, C7, C8: JLCPCB (none) -> C14663
- C10: renamed from C44; JLCPCB (none) -> C14663
- C17: value 100n -> 3n3; footprint Capacitor_SMD:C_0603_1608Metric -> Capacitor_SMD:C_0805_2012Metric; JLCPCB (none) -> C107149
- C18: renamed from C48; JLCPCB (none) -> C311611
- C47: value 3n3 -> 100n; footprint Capacitor_SMD:C_0805_2012Metric -> Capacitor_SMD:C_0603_1608Metric; JLCPCB (none) -> C14663
- D3: renamed from D4; value LED_GREEN -> LED_RED; JLCPCB (none) -> C84256
- F1: JLCPCB (none) -> C136367
- L2: renamed from L1; JLCPCB (none) -> C85840
- R1, R10, R11, R12, R13, R14, R18, R19, R2, R20, R21, R22, R23, R24, R25, R26, R27, R28, R29, R3, R32, R33, R34, R35, R36, R37, R38, R4, R40, R41, R43, R44, R5, R50, R55, R56, R57, R58, R59, R6, R60, R61, R62, R63, R64, R7, R8, R9: JLCPCB (none) -> C238881
- R15: renamed from R47; JLCPCB (none) -> C126358
- R16: value 10k -> 1k; JLCPCB (none) -> C269704
- R17: renamed from R49; JLCPCB (none) -> C269704
- R30, R54: value 10k -> 4.7k; JLCPCB (none) -> C101062
- R42: renamed from R96; JLCPCB (none) -> C238881
- R45, R46: value 4.7k -> 10k; JLCPCB (none) -> C238881
- R48: value 1k -> 10k; JLCPCB (none) -> C238881
- R51, R52: value 10k -> 680R; JLCPCB (none) -> C269704
- R53: value 10k -> 330R; JLCPCB (none) -> C101062
- RV1: JLCPCB (none) -> C317745
- SW1: footprint Button_Switch_THT:SW_PUSH_6mm_H8mm -> Button_Switch_THT:SW_PUSH_6mm_H13mm
- U33: renamed from U13; JLCPCB (none) -> C26858
- Y1: footprint Crystal:Crystal_C38-LF_D3.0mm_L8.0mm_Horizontal_1EP_style1 -> Crystal:Crystal_C26-LF_D2.1mm_L6.5mm_Horizontal
- renumbered J3 to J1, J5 to J2, J4 to J3, J6 to J4, J7 to J6
Connections:
- net labels added: +24VA, A+, B-, GNDD, GND_ADC, P8.07_OUT, P8.08_OUT, P8.09_OUT, P8.10_OUT, P8.11_OUT, P8.12_OUT, P8.14_OUT, P8.15_OUT, P8.16_OUT, P8.17_OUT, P8.18_OUT, P8.26_OUT, P8.27_OUT, P8.28_OUT, P8.29_OUT, P8.30_OUT, P8.31_OUT, P8.32_OUT, P8.33_OUT, P8.34_OUT, P8.35_OUT, P8.36_OUT, P8.37_OUT, P8.38_OUT, P8.39_OUT, P8.40_OUT, P8.41_OUT, P8.42_OUT, P8.43_OUT, P8.44_OUT, P8.45_OUT, P8.46_OUT, P9.11_OUT, P9.12_OUT, P9.13_OUT, P9.14_OUT, P9.15_OUT, P9.16_OUT, P9.17_OUT, P9.18_OUT, P9.21_OUT, P9.22_OUT, P9.23_OUT, P9.24_OUT, P9.25_OUT, P9.26_OUT, P9.27_OUT, P9.28_OUT, P9.29_OUT, P9.30_OUT, P9.31_OUT, P9.42_OUT, SCL_OUT, SDA_OUT, VDD_ADC
- net labels removed: P9.32, P9.34
- wire segments 829 -> 746
- no-connect marks 4 -> 1
Other:
- note removed: "Pull_Up\n"
- moved on the sheet: BT1, C10, C18, D3, J1, J2, J3, J4, J6, L2, R15, R17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

Commit message: 03.11.2021
Parts:
- removed PS1: B2424S-1WR2, CONV_B0505S-1WR2, symbol Power_Management:B2424S-1WR2
- removed U1, U10, U11, U12, U13, U14, U15, U16, U17, U18, U19, U2, U20, U21, U22, U23, U24, U25, U26, U27, U29, U3, U30, U31, U32, U34, U35, U36, U37, U38, U39, U4, U40, U41, U42, U43, U44, U45, U47, U48, U49, U5, U50, U51, U52, U53, U54, U55, U56, U6, U7, U8: EL357N-G, Package_SO:OPTO_EL357N-G, symbol Isolator:PC817
- added J14: ZW_VCC, Connector_PinHeader_2.54mm:PinHeader_1x03_P2.54mm_Vertical, symbol Connector:Screw_Terminal_01x03
- added J15: ZW_GND, Connector_PinHeader_2.54mm:PinHeader_1x03_P2.54mm_Vertical, symbol Connector:Screw_Terminal_01x03
- added J16: INNY ZASILACZ, Connector:Phoenix_1x02_P5.00mm_Horizontal, symbol Connector:Screw_Terminal_01x02
- added R100, R101, R102, R103, R104, R105, R106, R107, R108, R113, R114, R115, R116, R65, R66, R67, R68, R69, R70, R71, R72, R73, R74, R75, R76, R93, R94, R95, R96, R97, R98, R99: 10k, Resistor_SMD:R_0603_1608Metric, symbol Device:R
- added R109, R110, R111, R112, R77, R78, R79, R80, R81, R82, R83, R84, R85, R86, R87, R88, R89, R90, R91, R92: 4,7k, Resistor_SMD:R_0603_1608Metric, symbol Device:R
- added U1, U10, U11, U12, U13, U14, U2, U3, U4, U5, U6, U7, U8: TLP290-4, Package_SO:SOP-16_4.55x10.3mm_P1.27mm, symbol Isolator:TLP290-4
- R1, R10, R11, R12, R13, R14, R18, R19, R20, R21, R22, R40, R41, R43, R44, R45, R46, R47, R48, R49, R5, R50, R55, R56, R57, R58, R59, R6, R60, R7, R8, R9: value 10k -> 4,7k
Connections:
- net +24V: now also J14.1 (Pin_1)
- net +3V3: now also R2.2, R23.2, R24.2, R25.2, R26.2, R27.2, R28.2, R29.2, R3.2, R32.2, R33.2, R34.2, R35.2, R38.2, R39.2, R4.2, R61.2, R62.2, R63.2, R64.2, R100.2, R101.2, R102.2, R103.2, R104.2, R105.2, R106.2, R107.2, R108.2, R113.2, R114.2, R115.2, R116.2, R65.2, R66.2, R67.2, R68.2, R69.2, R70.2, R71.2, R72.2, R73.2, R74.2, R75.2, R76.2, R93.2, R94.2, R95.2, R96.2, R97.2, R98.2, R99.2
- net GND: now also C1.2, C11.2, C12.2, C13.2, C14.2, C15.2, C16.2, C19.2, C2.2, C20.2, C21.2, C22.2, C23.2, C24.2, C25.2, C26.2, C27.2, C28.2, C29.2, C3.2, C30.2, C31.2, C32.2, C33.2, C34.2, C35.2, C36.2, C37.2, C38.2, C39.2, C4.2, C40.2, C41.2, C42.2, C43.2, C44.2, C45.2, C46.2, C49.2, C5.2, C50.2, C51.2, C52.2, C53.2, C54.2, C55.2, C56.2, C57.2, C58.2, C6.2, C7.2, C8.2, J15.1 (Pin_1), U1.11, U1.13, U1.15, U1.9, U10.11, U10.13, U10.15, U10.9, U11.11, U11.13, U11.15, U11.9, U12.11, U12.13, U12.15, U12.9, U13.11, U13.13, U13.15, U13.9, U14.11, U14.13, U14.15, U14.9, U2.11, U2.13, U2.15, U2.9, U3.11, U3.13, U3.15, U3.9, U4.11, U4.13, U4.15, U4.9, U5.11, U5.13, U5.15, U5.9, U6.11, U6.13, U6.15, U6.9, U7.11, U7.13, U7.15, U7.9, U8.11, U8.13, U8.15, U8.9; no longer J13.1 (Pin_1), J8.1 (Pin_1)
- net GNDA: now also R1.2, R10.2, R11.2, R12.2, R13.2, R14.2, R18.2, R19.2, R20.2, R21.2, R22.2, R40.2, R41.2, R43.2, R44.2, R45.2, R46.2, R47.2, R48.2, R49.2, R5.2, R50.2, R55.2, R56.2, R57.2, R58.2, R59.2, R6.2, R60.2, R7.2, R8.2, R9.2, J15.2 (Pin_2), R109.2, R110.2, R111.2, R112.2, R77.2, R78.2, R79.2, R80.2, R81.2, R82.2, R83.2, R84.2, R85.2, R86.2, R87.2, R88.2, R89.2, R90.2, R91.2, R92.2; no longer J1.1 (Pin_1), J2.1 (Pin_1), J3.1 (Pin_1), J4.1 (Pin_1), J5.1 (Pin_1), J6.1 (Pin_1)
- net GNDD: now also J15.3 (Pin_3), J16.1 (Pin_1)
- net P8.07: now also C36.1, R76.1, U8.10
- net P8.07_OUT: now also U8.7; no longer C6.2
- net P8.08: now also C32.1, R72.1, U8.12
- net P8.08_OUT: now also U8.5; no longer C5.2
- net P8.09: now also C28.1, R68.1, U8.14
- net P8.09_OUT: now also U8.3; no longer C46.2
- net P8.10: now also C24.1, R64.1, U8.16
- net P8.10_OUT: now also U8.1; no longer C45.2
- net P8.11: now also C35.1, R75.1, U7.10
- net P8.11_OUT: now also U7.7; no longer C44.2
- net P8.12: now also C31.1, R71.1, U7.12
- net P8.12_OUT: now also U7.5; no longer C43.2
- net P8.14: now also C27.1, R67.1, U7.14
- net P8.14_OUT: now also U7.3; no longer C42.2
- net P8.15: now also C23.1, R63.1, U7.16
- net P8.15_OUT: now also U7.1; no longer C41.2
- net P8.16: now also C34.1, R74.1, U6.10
- net P8.16_OUT: now also U6.7; no longer C40.2
- net P8.17: now also C30.1, R70.1, U6.12
- net P8.17_OUT: now also U6.5; no longer C39.2
- net P8.18: now also C26.1, R66.1, U6.14
- net P8.18_OUT: now also U6.3; no longer C38.2
- net P8.26: now also C22.1, R62.1, U6.16
- net P8.26_OUT: now also U6.1; no longer C31.2
- net P8.27: now also C33.1, R73.1, U5.10
- net P8.27_OUT: now also U5.7; no longer C30.2
- net P8.28: now also C29.1, R69.1, U5.12
- net P8.28_OUT: now also U5.5; no longer C29.2
- net P8.29: now also C25.1, R65.1, U5.14
- net P8.29_OUT: now also U5.3; no longer C28.2
- net P8.30: now also C21.1, R61.1, U5.16
- net P8.30_OUT: now also U5.1; no longer C27.2
- net P8.31: now also C20.1, R39.1, U4.10
- net P8.31_OUT: now also U4.7; no longer C26.2
- net P8.32: now also C15.1, R33.1, U4.12
- net P8.32_OUT: now also U4.5; no longer C25.2
- net P8.33: now also C12.1, R28.1, U4.14
- net P8.33_OUT: now also U4.3; no longer C24.2
- net P8.34: now also C7.1, R25.1, U4.16
- net P8.34_OUT: now also U4.1; no longer C23.2
- net P8.35: now also C19.1, R38.1, U3.10
- net P8.35_OUT: now also U3.7; no longer C22.2
- net P8.36: now also C14.1, R32.1, U3.12
- net P8.36_OUT: now also U3.5; no longer C21.2
- net P8.37: now also C11.1, R27.1, U3.14
- net P8.37_OUT: now also U3.3; no longer C20.2
- net P8.38: now also C6.1, R24.1, U3.16
- net P8.38_OUT: now also U3.1; no longer C19.2
- net P8.39: now also C16.1, R35.1, U2.10
- net P8.39_OUT: now also U2.7; no longer C14.2
- net P8.40: now also C13.1, R29.1, U2.12
- net P8.40_OUT: now also U2.5; no longer C13.2
- net P8.41: now also C8.1, R26.1, U2.14
- net P8.41_OUT: now also U2.3; no longer C12.2
- net P8.42: now also C5.1, R23.1, U2.16
- net P8.42_OUT: now also U2.1; no longer C11.2
- net P8.43: now also C3.1, R34.1, U1.10
- net P8.43_OUT: now also U1.1; no longer C4.2
- net P8.44: now also C4.1, R4.1, U1.12
- net P8.44_OUT: now also U1.3; no longer C3.2
- net P8.45: now also C2.1, R3.1, U1.14
- net P8.45_OUT: now also U1.5; no longer C2.2
- net P8.46: now also C1.1, R2.1, U1.16
- net P8.46_OUT: now also U1.7; no longer C1.2
- net P9.11: now also C37.1, R93.1, U10.16
- net P9.11_OUT: now also U10.1; no longer C35.2
- net P9.12: now also C41.1, R97.1, U10.14
- net P9.12_OUT: now also U10.3; no longer C36.2
- net P9.13: now also C45.1, R101.1, U10.12
- net P9.13_OUT: now also U10.5; no longer C37.2
- net P9.14: now also C51.1, R105.1, U10.10
- net P9.14_OUT: now also U10.7; no longer C7.2
- net P9.15: now also C38.1, R94.1, U11.16
- net P9.15_OUT: now also U11.1; no longer C8.2
- net P9.16: now also C42.1, R98.1, U11.14
- net P9.16_OUT: now also U11.3; no longer C32.2
- net P9.17: now also C46.1, R102.1, U11.12
- net P9.17_OUT: now also U11.5; no longer C33.2
- net P9.18: now also C52.1, R106.1, U11.10
- net P9.18_OUT: now also U11.7; no longer C34.2
- net P9.21: now also C39.1, R95.1, U12.16
- net P9.21_OUT: now also U12.1; no longer C15.2
- net P9.22: now also C43.1, R99.1, U12.14
- net P9.22_OUT: now also U12.3; no longer C16.2
- net P9.23: now also C49.1, R103.1, U12.12
- net P9.23_OUT: now also U12.5; no longer C53.2
- net P9.24: now also C53.1, R107.1, U12.10
- net P9.24_OUT: now also U12.7; no longer C52.2
- net P9.25: now also C40.1, R96.1, U13.16
- net P9.25_OUT: now also U13.1; no longer C51.2
- net P9.26: now also C44.1, R100.1, U13.14
- net P9.26_OUT: now also U13.3; no longer C50.2
- net P9.27: now also C50.1, R104.1, U13.12
- net P9.27_OUT: now also U13.5; no longer C49.2
- net P9.28: now also C54.1, R108.1, U13.10
- net P9.28_OUT: now also U13.7; no longer C58.2
- net P9.29: now also C55.1, R113.1, U14.16
- net P9.29_OUT: now also U14.1; no longer C57.2
- net P9.30: now also C56.1, R114.1, U14.14
- net P9.30_OUT: now also U14.3; no longer C56.2
- net P9.31: now also C57.1, R115.1, U14.12
- net P9.31_OUT: now also U14.5; no longer C55.2
- net P9.42: now also C58.1, R116.1, U14.10
- net P9.42_OUT: now also U14.7; no longer C54.2
- net at R1.1: now also U1.2; no longer C1.1
- net at R9.1: now also U2.4; no longer C11.1
- net at R11.1: now also U2.8; no longer C13.1
- net at R12.1: now also U3.2; no longer C14.1
- net at R18.1: now also U3.8; no longer C19.1
- net at R19.1: now also U4.2; no longer C20.1
- net at R21.1: now also U4.6; no longer C22.1
- net at R22.1: now also U4.8; no longer C23.1
- net at R40.1: now also U5.2; no longer C37.1
- net at R41.1: now also U5.4; no longer C38.1
- net at R43.1: now also U5.6; no longer C39.1
- net at R44.1: now also U5.8; no longer C40.1
- net at R45.1: now also U6.2; no longer C41.1
- net at R46.1: now also U6.4; no longer C42.1
- net at R47.1: now also U6.6; no longer C43.1
- net at R48.1: now also U6.8; no longer C44.1
- net at R49.1: now also U7.2; no longer C45.1
- net at R5.1: now also U1.4; no longer C5.1
- net at R6.1: now also U1.6; no longer C6.1
- net at R7.1: now also U1.8; no longer C7.1
- net at R8.1: now also U2.2; no longer C8.1
- net at R13.1: now also U3.4; no longer C15.1
- net at R14.1: now also U3.6; no longer C16.1
- net at R10.1: now also U2.6; no longer C12.1
- net at R20.1: now also U4.4; no longer C21.1
- net at R60.1: now also U8.8; no longer C54.1
- net at R57.1: now also U8.2; no longer C51.1
- net at R56.1: now also U7.8; no longer C50.1
- net at R55.1: now also U7.6; no longer C49.1
- net at R58.1: now also U8.4; no longer C52.1
- net at R59.1: now also U8.6; no longer C53.1
- net at R50.1: now also U7.4; no longer C46.1
- removed net +24VA: R1.2, R10.2, R11.2, R12.2, R13.2, R14.2, R18.2, R19.2, R2.2, R20.2, R21.2, R22.2, R23.2, R24.2, R25.2, R26.2, R27.2, R28.2, R29.2, R3.2, R32.2, R33.2, R34.2, R35.2, R38.2, R39.2, R4.2, R40.2, R41.2, R43.2, R44.2, R45.2, R46.2, R47.2, R48.2, R49.2, R5.2, R50.2, R55.2, R56.2, R57.2, R58.2, R59.2, R6.2, R60.2, R61.2, R62.2, R63.2, R64.2, R7.2, R8.2, R9.2
- new net: R77.1, U10.2
- new net: R78.1, U10.4
- new net: R79.1, U10.6
- new net: R80.1, U10.8
- new net: R81.1, U11.2
- new net: R82.1, U11.4
- new net: R83.1, U11.6
- new net: R84.1, U11.8
- new net: R85.1, U12.2
- new net: R86.1, U12.4
- new net: R87.1, U12.6
- new net: R88.1, U12.8
- new net: R89.1, U13.2
- new net: R90.1, U13.4
- new net: R91.1, U13.6
- new net: R92.1, U13.8
- new net: R109.1, U14.2
- new net: R110.1, U14.4
- new net: R111.1, U14.6
- new net: R112.1, U14.8
- new net +48V: J14.3 (Pin_3), J16.2 (Pin_2)
- new net VDD: J1.1 (Pin_1), J13.1 (Pin_1), J14.2 (Pin_2), J2.1 (Pin_1), J3.1 (Pin_1), J4.1 (Pin_1), J5.1 (Pin_1), J6.1 (Pin_1), J8.1 (Pin_1)
Other:
- note removed: "Pin_Out\n"
- moved on the sheet: ANVDD1, BT1, C1, C2, C3, C4, C47, C48, D4, D5, I2C1, J1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

Commit message: 04.11.2021
Connections:
- net GNDD: no longer J15.3 (Pin_3), J16.1 (Pin_1)
- net P8.07: now also C55.1, R113.1, U14.16; no longer C36.1, R76.1, U8.10
- net P8.07_OUT: now also U14.1; no longer U8.7
- net P8.08: now also C36.1, R76.1, U8.10; no longer C32.1, R72.1, U8.12
- net P8.08_OUT: now also U8.7; no longer U8.5
- net P8.09: now also C32.1, R72.1, U8.12; no longer C28.1, R68.1, U8.14
- net P8.09_OUT: now also U8.5; no longer U8.3
- net P8.10: now also C28.1, R68.1, U8.14; no longer C24.1, R64.1, U8.16
- net P8.10_OUT: now also U8.3; no longer U8.1
- net P8.11: now also C24.1, R64.1, U8.16; no longer C35.1, R75.1, U7.10
- net P8.11_OUT: now also U8.1; no longer U7.7
- net P8.12: now also C35.1, R75.1, U7.10; no longer C31.1, R71.1, U7.12
- net P8.12_OUT: now also U7.7; no longer U7.5
- net P8.14: now also C31.1, R71.1, U7.12; no longer C27.1, R67.1, U7.14
- net P8.14_OUT: now also U7.5; no longer U7.3
- net P8.15: now also C27.1, R67.1, U7.14; no longer C23.1, R63.1, U7.16
- net P8.15_OUT: now also U7.3; no longer U7.1
- net P8.16: now also C23.1, R63.1, U7.16; no longer C34.1, R74.1, U6.10
- net P8.16_OUT: now also U7.1; no longer U6.7
- net P8.17: now also C34.1, R74.1, U6.10; no longer C30.1, R70.1, U6.12
- net P8.17_OUT: now also U6.7; no longer U6.5
- net P8.18: now also C30.1, R70.1, U6.12; no longer C26.1, R66.1, U6.14
- net P8.18_OUT: now also U6.5; no longer U6.3
- net P8.26: now also C33.1, R73.1, U5.10; no longer C22.1, R62.1, U6.16
- net P8.26_OUT: now also U5.7; no longer U6.1
- net P8.27: now also C29.1, R69.1, U5.12; no longer C33.1, R73.1, U5.10
- net P8.27_OUT: now also U5.5; no longer U5.7
- net P8.28: now also C25.1, R65.1, U5.14; no longer C29.1, R69.1, U5.12
- net P8.28_OUT: now also U5.3; no longer U5.5
- net P8.29: now also C21.1, R61.1, U5.16; no longer C25.1, R65.1, U5.14
- net P8.29_OUT: now also U5.1; no longer U5.3
- net P8.30: now also C20.1, R39.1, U4.10; no longer C21.1, R61.1, U5.16
- net P8.30_OUT: now also U4.7; no longer U5.1
- net P8.31: now also C15.1, R33.1, U4.12; no longer C20.1, R39.1, U4.10
- net P8.31_OUT: now also U4.5; no longer U4.7
- net P8.32: now also C12.1, R28.1, U4.14; no longer C15.1, R33.1, U4.12
- net P8.32_OUT: now also U4.3; no longer U4.5
- net P8.33: now also C7.1, R25.1, U4.16; no longer C12.1, R28.1, U4.14
- net P8.33_OUT: now also U4.1; no longer U4.3
- net P8.34: now also C19.1, R38.1, U3.10; no longer C7.1, R25.1, U4.16
- net P8.34_OUT: now also U3.7; no longer U4.1
- net P8.35: now also C14.1, R32.1, U3.12; no longer C19.1, R38.1, U3.10
- net P8.35_OUT: now also U3.5; no longer U3.7
- net P8.36: now also C11.1, R27.1, U3.14; no longer C14.1, R32.1, U3.12
- net P8.36_OUT: now also U3.3; no longer U3.5
- net P8.37: now also C6.1, R24.1, U3.16; no longer C11.1, R27.1, U3.14
- net P8.37_OUT: now also U3.1; no longer U3.3
- net P8.38: now also C16.1, R35.1, U2.10; no longer C6.1, R24.1, U3.16
- net P8.38_OUT: now also U2.7; no longer U3.1
- net P8.39: now also C13.1, R29.1, U2.12; no longer C16.1, R35.1, U2.10
- net P8.39_OUT: now also U2.5; no longer U2.7
- net P8.40: now also C8.1, R26.1, U2.14; no longer C13.1, R29.1, U2.12
- net P8.40_OUT: now also U2.3; no longer U2.5
- net P8.41: now also C5.1, R23.1, U2.16; no longer C8.1, R26.1, U2.14
- net P8.41_OUT: now also U2.1; no longer U2.3
- net P8.42: now also C3.1, R34.1, U1.10; no longer C5.1, R23.1, U2.16
- net P8.42_OUT: now also U1.7; no longer U2.1
- net P8.43: now also C4.1, R4.1, U1.12; no longer C3.1, R34.1, U1.10
- net P8.43_OUT: now also U1.5; no longer U1.1
- net P8.44: now also C2.1, R3.1, U1.14; no longer C4.1, R4.1, U1.12
- net P8.45: now also C1.1, R2.1, U1.16; no longer C2.1, R3.1, U1.14
- net P8.45_OUT: now also U1.1; no longer U1.5
- net P8.46: no longer C1.1, R2.1, U1.16
- net P8.46_OUT: now also U13.7; no longer U1.7
- net P9.11: now also C38.1, R94.1, U11.16; no longer C37.1, R93.1, U10.16
- net P9.11_OUT: now also U11.1; no longer U10.1
- net P9.12: now also C42.1, R98.1, U11.14; no longer C41.1, R97.1, U10.14
- net P9.12_OUT: now also U11.3; no longer U10.3
- net P9.13: now also C46.1, R102.1, U11.12; no longer C45.1, R101.1, U10.12
- net P9.13_OUT: now also U11.5; no longer U10.5
- net P9.14: now also C52.1, R106.1, U11.10; no longer C51.1, R105.1, U10.10
- net P9.14_OUT: now also U11.7; no longer U10.7
- net P9.15: now also C22.1, R62.1, U6.16; no longer C38.1, R94.1, U11.16
- net P9.15_OUT: now also U6.1; no longer U11.1
- net P9.16: now also C26.1, R66.1, U6.14; no longer C42.1, R98.1, U11.14
- net P9.16_OUT: now also U6.3; no longer U11.3
- net P9.17: now also C50.1, R104.1, U13.12; no longer C46.1, R102.1, U11.12
- net P9.17_OUT: now also U13.5; no longer U11.5
- net P9.18: now also C43.1, R99.1, U12.14; no longer C52.1, R106.1, U11.10
- net P9.18_OUT: now also U12.3; no longer U11.7
- net P9.21: now also C49.1, R103.1, U12.12; no longer C39.1, R95.1, U12.16
- net P9.21_OUT: now also U12.5; no longer U12.1
- net P9.22: now also C53.1, R107.1, U12.10; no longer C43.1, R99.1, U12.14
- net P9.22_OUT: now also U12.7; no longer U12.3
- net P9.23: now also C44.1, R100.1, U13.14; no longer C49.1, R103.1, U12.12
- net P9.23_OUT: now also U13.3; no longer U12.5
- net P9.24: now also C40.1, R96.1, U13.16; no longer C53.1, R107.1, U12.10
- net P9.24_OUT: now also U13.1; no longer U12.7
- net P9.25: now also C51.1, R105.1, U10.10; no longer C40.1, R96.1, U13.16
- net P9.25_OUT: now also U10.7; no longer U13.1
- net P9.26: now also C45.1, R101.1, U10.12; no longer C44.1, R100.1, U13.14
- net P9.26_OUT: now also U10.5; no longer U13.3
- net P9.27: now also C41.1, R97.1, U10.14; no longer C50.1, R104.1, U13.12
- net P9.27_OUT: now also U10.3; no longer U13.5
- net P9.28: now also C37.1, R93.1, U10.16; no longer C54.1, R108.1, U13.10
- net P9.28_OUT: now also U10.1; no longer U13.7
- net P9.29: now also C39.1, R95.1, U12.16; no longer C55.1, R113.1, U14.16
- net P9.29_OUT: now also U12.1; no longer U14.1
- net P9.30: now also C58.1, R116.1, U14.10; no longer C56.1, R114.1, U14.14
- net P9.30_OUT: now also U14.7; no longer U14.3
- net P9.42: now also C56.1, R114.1, U14.14; no longer C58.1, R116.1, U14.10
- net P9.42_OUT: now also U14.3; no longer U14.7
- new net GND1: J15.3 (Pin_3), J16.1 (Pin_1)
- new net P9.46: C54.1, R108.1, U13.10
Other:
- moved on the sheet: ANVDD1, J1, J13, J14, J15, J16, J2, J3, J4, J5, J6, J7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

Commit message: 06/11/21
Parts:
- renumbered C47 to C1, C11 to C10, C12 to C11, C4 to C12, C3 to C16, C16 to C17, C19 to C18, C20 to C19, C9 to C2, C17 to C20, C18 to C21, C21 to C22, C22 to C23, C23 to C24, C24 to C25, C25 to C26, C26 to C27, C27 to C28, C28 to C29, C10 to C3, C29 to C30, C30 to C31, C31 to C32, C32 to C33, C33 to C34, C34 to C35, C35 to C36, C36 to C37, C48 to C38, C37 to C39, C1 to C4, C38 to C40, C39 to C41, C40 to C42, C41 to C43, C42 to C44, C43 to C45, C44 to C46, C45 to C47, C46 to C48, C2 to C8, C8 to C9, D4 to D2, D2 to D3, D3 to D4, J12 to J1, J13 to J10, J7 to J11, J10 to J12, J14 to J13, J15 to J14, J11 to J15, J9 to J2, J1 to J3, J2 to J4, J3 to J5, J4 to J6, J5 to J7, J6 to J8, J8 to J9, R13 to R10, R103 to R100, R104 to R101, R105 to R102, R106 to R103, R107 to R104, R108 to R105, R36 to R106, R37 to R107, R109 to R108, R110 to R109, R14 to R11, R111 to R110, R112 to R111, R42 to R112, R18 to R12, R19 to R13, R20 to R14, R21 to R15, R22 to R16, R51 to R17, R2 to R18, R23 to R19, R5 to R2, R24 to R20, R25 to R21, R3 to R22, R26 to R23, R27 to R24, R28 to R25, R52 to R26, R4 to R27, R29 to R28, R32 to R29, R6 to R3, R33 to R30, R34 to R31, R35 to R32, R38 to R33, R39 to R34, R15 to R35, R16 to R36, R17 to R37, R40 to R38, R41 to R39, R7 to R4, R43 to R40, R44 to R41, R45 to R42, R46 to R43, R47 to R44, R48 to R45, R49 to R46, R50 to R47, R55 to R48, R56 to R49, R8 to R5, R57 to R50, R58 to R51, R59 to R52, R60 to R53, R61 to R54, R62 to R55, R63 to R56, R64 to R57, R65 to R58, R66 to R59, R9 to R6, R67 to R60, R68 to R61, R69 to R62, R70 to R63, R71 to R64, R72 to R65, R73 to R66, R74 to R67, R75 to R68, R76 to R69, R10 to R7, R53 to R70, R54 to R71, R77 to R72, R78 to R73, R79 to R74, R80 to R75, R81 to R76, R82 to R77, R83 to R78, R84 to R79, R11 to R8, R85 to R80, R86 to R81, R87 to R82, R88 to R83, R89 to R84, R90 to R85, R91 to R86, R92 to R87, R93 to R88, R94 to R89, R12 to R9, R95 to R90, R96 to R91, R30 to R92, R97 to R93, R98 to R94, R99 to R95, R100 to R96, R31 to R97, R101 to R98, R102 to R99, U46 to U1, U7 to U10, U8 to U11, U10 to U12, U11 to U13, U12 to U14, U13 to U15, U33 to U16, U14 to U17, U1 to U2, U2 to U3, U3 to U4, U4 to U5, U9 to U6, U28 to U7, U5 to U8, U6 to U9
