File: Circuit/boneIO - input board/boneIO_input board_v0.2.kicad_pcb (KiCad board)
At the start: 2 copper layers, 231 x 74 mm, 177 parts, among them J1 Screw_Terminal_01x08, J10 BeagleBone_Black_Header, J11 BeagleBone_Black_Header, J12 Conn_02x04_Odd_Even, J2 Screw_Terminal_01x08, J3 Screw_Terminal_01x08, J4 Screw_Terminal_01x08, J5 Screw_Terminal_01x08, J6 Screw_Terminal_01x08, J7 Screw_Terminal_01x08, J9 Screw_Terminal_01x08, SW1 SW_Push, U1 EL357N-G, U10 EL357N-G, U11 EL357N-G, U12 EL357N-G, U13 EL357N-G, U14 EL357N-G, U15 EL357N-G, U16 EL357N-G, U17 EL357N-G, U18 EL357N-G, U19 EL357N-G, U2 EL357N-G, U20 EL357N-G, U21 EL357N-G, U22 EL357N-G, U23 EL357N-G, U24 EL357N-G, U25 EL357N-G, U26 EL357N-G, U27 EL357N-G, U28 RS485, U29 EL357N-G, U3 EL357N-G, U30 EL357N-G, U31 EL357N-G, U32 EL357N-G, U33 DS1307Z+, U34 EL357N-G, U35 EL357N-G, U36 EL357N-G, U37 EL357N-G, U38 EL357N-G, U39 EL357N-G, U4 EL357N-G, U40 EL357N-G, U41 EL357N-G, U42 EL357N-G, U43 EL357N-G, U44 EL357N-G, U45 EL357N-G, U46 P82B96, U5 EL357N-G, U6 EL357N-G, U7 EL357N-G, U8 EL357N-G, U9 LM2596S-ADJ, Y1 32,788 MHz

Commit message: 01.11.2021
Parts:
- removed G***: LOGO, Symbol:boneIO_LOGO
- added C49: 100n, Capacitor_SMD:C_0603_1608Metric, F.Cu at (138.7, 16.0)
- added C50: 100n, Capacitor_SMD:C_0603_1608Metric, F.Cu at (116.9, 38.6)
- added C51: 100n, Capacitor_SMD:C_0603_1608Metric, F.Cu at (121.0, 34.1)
- added C52: 100n, Capacitor_SMD:C_0603_1608Metric, F.Cu at (134.0, 21.0)
- added C53: 100n, Capacitor_SMD:C_0603_1608Metric, F.Cu at (142.7, 13.5)
- added C54: 100n, Capacitor_SMD:C_0603_1608Metric, F.Cu at (108.9, 43.6)
- added C55: 100n, Capacitor_SMD:C_0603_1608Metric, F.Cu at (89.2, 42.9)
- added C56: 100n, Capacitor_SMD:C_0603_1608Metric, F.Cu at (144.9, -0.94)
- added C57: 100n, Capacitor_SMD:C_0603_1608Metric, F.Cu at (130.6, 14.1)
- added C58: 100n, Capacitor_SMD:C_0603_1608Metric, F.Cu at (119.8, 26.5)
- added D1: B340A-13F, Diode_SMD:D_SMA, F.Cu at (106.9, 35.1)
- added D2: SS34, Diode_SMD:D_SMA, F.Cu at (113.7, 27.5)
- added F1: Fuse_3A, Fuse:Fuse_2512_6332Metric, F.Cu at (124.3, 15.3)
- added J13: Screw_Terminal_01x04, Connector:Phoenix_1x04_P5.00mm_Horizontal, F.Cu at (153.9, 117.8)
- added J8: Screw_Terminal_01x08, Connector:8pin, F.Cu at (186.3, 60.5)
- added R16: 1k, Resistor_SMD:R_0603_1608Metric, F.Cu at (131.9, 11.0)
- added R55: 10k, Resistor_SMD:R_0603_1608Metric, F.Cu at (145.2, 1.57)
- added R56: 10k, Resistor_SMD:R_0603_1608Metric, F.Cu at (145.2, 4.08)
- added R57: 10k, Resistor_SMD:R_0603_1608Metric, F.Cu at (121.9, 21.5)
- added R58: 10k, Resistor_SMD:R_0603_1608Metric, F.Cu at (112.9, 36.1)
- added R59: 10k, Resistor_SMD:R_0603_1608Metric, F.Cu at (117.0, 33.5)
- added R60: 10k, Resistor_SMD:R_0603_1608Metric, F.Cu at (123.8, 26.6)
- added R61: 10k, Resistor_SMD:R_0603_1608Metric, F.Cu at (139.9, 11.0)
- added R62: 10k, Resistor_SMD:R_0603_1608Metric, F.Cu at (134.6, 16.0)
- added R63: 10k, Resistor_SMD:R_0603_1608Metric, F.Cu at (112.9, 38.6)
- added R64: 10k, Resistor_SMD:R_0603_1608Metric, F.Cu at (143.9, 7.86)
- added U27: EL357N-G, Package_SO:OPTO_EL357N-G, F.Cu at (88.2, 38.8)
- added U47: EL357N-G, Package_SO:OPTO_EL357N-G, F.Cu at (114.6, 5.46)
- added U48: EL357N-G, Package_SO:OPTO_EL357N-G, F.Cu at (85.1, 27.5)
- added U49: EL357N-G, Package_SO:OPTO_EL357N-G, F.Cu at (95.4, 13.0)
- added U50: EL357N-G, Package_SO:OPTO_EL357N-G, F.Cu at (85.1, 21.8)
- added U51: EL357N-G, Package_SO:OPTO_EL357N-G, F.Cu at (75.2, 33.4)
- added U52: EL357N-G, Package_SO:OPTO_EL357N-G, F.Cu at (118.3, -6.89)
- added U53: EL357N-G, Package_SO:OPTO_EL357N-G, F.Cu at (75.2, 27.7)
- added U54: EL357N-G, Package_SO:OPTO_EL357N-G, F.Cu at (125.2, 10.1)
- added U55: EL357N-G, Package_SO:OPTO_EL357N-G, F.Cu at (138.2, -6.89)
- added U56: EL357N-G, Package_SO:OPTO_EL357N-G, F.Cu at (98.2, 35.6)
- moved U35 129.7 mm to (128.2, -1.25), turned to 0 degrees
- moved R37 126.3 mm to (134.6, 13.5)
- moved C35 125.4 mm to (134.6, 18.5)
- moved R36 123.8 mm to (139.9, 8.48)
- moved U37 117.8 mm to (124.5, 4.41), turned to 0 degrees
- moved C16 115.4 mm to (144.9, -3.44)
- moved C44 113.0 mm to (143.9, 10.4)
- moved R31 111.7 mm to (130.6, 16.6), turned to 0 degrees
- moved R7 111.3 mm to (141.2, 5.34)
- moved R30 111.2 mm to (126.0, 21.5), turned to 0 degrees
- moved C36 107.2 mm to (123.8, 29.1)
- moved R13 105.8 mm to (135.9, 8.48)
- moved R33 104.9 mm to (108.9, 38.6)
- moved C22 103.7 mm to (144.9, -8.46), turned to 0 degrees
- moved R44 102.9 mm to (123.8, 24.0)
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Connections:
- C15 pad 2: P8.04_OUT -> P9.21_OUT
- C16 pad 2: P8.03_OUT -> P9.22_OUT
- C32 pad 2: P8.25_OUT -> P9.16_OUT
- C33 pad 2: P8.24_OUT -> P9.17_OUT
- C34 pad 2: P8.23_OUT -> P9.18_OUT
- C35 pad 2: P8.22_OUT -> P9.11_OUT
- C36 pad 2: P8.21_OUT -> P9.12_OUT
- C37 pad 2: P8.20_OUT -> P9.13_OUT
- C7 pad 2: P8.06_OUT -> P9.14_OUT
- C8 pad 2: P8.05_OUT -> P9.15_OUT
- J12 pad 5: SDA -> GND
- J12 pad 6: SCL -> +3V3
- J12 pad 7: GND -> SDA
- J12 pad 8: +3V3 -> SCL
- J2 pad 2: P8.25_OUT -> P9.11_OUT
- J2 pad 3: P8.24_OUT -> P9.12_OUT
- J2 pad 4: P8.23_OUT -> P9.13_OUT
- J2 pad 5: P8.22_OUT -> P9.14_OUT
- J2 pad 6: P8.21_OUT -> P9.15_OUT
- J2 pad 7: P8.20_OUT -> P9.16_OUT
- J6 pad 5: P8.06_OUT -> P9.42_OUT
- J6 pad 6: P8.05_OUT -> P9.31_OUT
- J6 pad 7: P8.04_OUT -> P9.30_OUT
- J6 pad 8: P8.03_OUT -> P9.29_OUT
- U14 pad 2: P8.04_OUT -> P9.21_OUT
- U14 pad 4: P8.04 -> P9.21
- U15 pad 2: P8.03_OUT -> P9.22_OUT
- U15 pad 4: P8.03 -> P9.22
- U30 pad 2: P8.25_OUT -> P9.16_OUT
- U30 pad 4: P8.25 -> P9.16
- U31 pad 2: P8.24_OUT -> P9.17_OUT
- U31 pad 4: P8.24 -> P9.17
- U32 pad 2: P8.23_OUT -> P9.18_OUT
- U32 pad 4: P8.23 -> P9.18
- U34 pad 2: P8.22_OUT -> P9.11_OUT
- U34 pad 4: P8.22 -> P9.11
- U35 pad 2: P8.21_OUT -> P9.12_OUT
- U35 pad 4: P8.21 -> P9.12
- U36 pad 2: P8.20_OUT -> P9.13_OUT
- U36 pad 4: P8.20 -> P9.13
- U7 pad 2: P8.06_OUT -> P9.14_OUT
- U7 pad 4: P8.06 -> P9.14
- U8 pad 2: P8.05_OUT -> P9.15_OUT
- U8 pad 4: P8.05 -> P9.15
Routing:
- net +24VA: track 360.3 -> 0.00 mm, vias 42 -> 0
- net +3V3: track 261.5 -> 0.00 mm, vias 6 -> 0
- net SCL: track 209.0 -> 0.00 mm, vias 2 -> 0
- net GND: track 207.2 -> 0.00 mm, vias 161 -> 0
- net P9.11: track 200.8 -> 0.00 mm, vias 1 -> 0
- net P9.15: track 197.6 -> 0.00 mm, vias 1 -> 0
- net P9.13: track 197.3 -> 0.00 mm, vias 1 -> 0
- net P9.12: track 195.4 -> 0.00 mm, vias 1 -> 0
- net P8.25: track 195.1 -> 0.00 mm, vias 1 -> 0
- net P9.14: track 194.8 -> 0.00 mm, vias 1 -> 0
- net P9.16: track 191.4 -> 0.00 mm, vias 1 -> 0
- net SDA: track 188.8 -> 0.00 mm, vias 3 -> 0
- net P8.24: track 186.7 -> 0.00 mm, vias 1 -> 0
- net P9.17: track 184.7 -> 0.00 mm, vias 1 -> 0
- net P8.23: track 184.5 -> 0.00 mm, vias 1 -> 0
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Other:
- board size 231 x 74 mm -> 256 x 74 mm
- board text removed: "AIN0"
- board text removed: "AIN1"
- board text removed: "AIN2"
- board text removed: "AIN3"
- board text removed: "AIN4"
- board text removed: "AIN5"
- board text removed: "AIN6"
