File: Circuit/boneIO - input board/boneIO_input board_v0.2.kicad_pcb (KiCad board)
At the start: 2 copper layers, 231 x 74 mm, 185 parts, among them J1 I2C_OUT, J2 Screw_Terminal_01x08, J3 Screw_Terminal_01x08, J4 Screw_Terminal_01x08, J5 Screw_Terminal_01x08, J6 Screw_Terminal_01x08, J7 Screw_Terminal_01x08, J8 Screw_Terminal_01x03, J9 Conn_02x13_Odd_Even, P3 BeagleBone_Black_Header, P4 BeagleBone_Black_Header, SW1 SW_Push, U1 LM2596S-ADJ, U10 PC847, U11 PC847, U12 PC847, U13 DS1307Z+, U2 PC847, U3 PC847, U4 PC847, U5 PC847, U6 PC847, U7 PC847, U8 PC847, U9 PC847, Y1 32,788 MHz

Commit message: Zmiany TEST
TEST
Parts:
- removed C31, C39: 100n, Capacitor_SMD:C_0603_1608Metric
- removed D1: B340A-13F, Diode_SMD:D_SMA
- removed J8: Screw_Terminal_01x03, Connector:3pin_5.0
- removed PS1: B2424S-1W, Module:CONV_B0505S-1WR2
- removed R31, R39, R92, R93: 10k, Resistor_SMD:R_0603_1608Metric
- removed REF**: StepDown_LM2596, Module:StepDown_LM2596
- moved D2 9.88 mm to (186.4, 92.5)
- moved D4 9.88 mm to (145.9, 99.6)
- moved RV1 9.88 mm to (187.4, 85.2)
- moved U1 9.88 mm to (168.6, 92.5)
- moved C43 9.88 mm to (179.8, 90.5)
- moved R47 9.88 mm to (152.3, 96.3)
- moved C44 9.88 mm to (175.5, 84.5)
- moved C47 9.88 mm to (156.8, 96.2)
- moved C48 9.88 mm to (144.6, 90.0)
- moved D3 9.88 mm to (171.2, 82.0)
- moved F1 9.88 mm to (191.8, 96.0)
- moved L1 9.88 mm to (192.1, 81.9)
- moved L2 9.88 mm to (155.6, 87.1)
- moved R48 9.88 mm to (154.2, 99.7)
- moved R49 9.88 mm to (147.0, 96.8)
Connections:
- J2 pad 1: +24VA -> GNDA
- J3 pad 1: +24VA -> GNDA
- J4 pad 1: +24VA -> GNDA
- J5 pad 1: +24VA -> GNDA
- J6 pad 1: +24VA -> GNDA
- J7 pad 1: +24VA -> GNDA
- P3 pad 23: P9.24 -> TX
- P3 pad 25: P9.26 -> RX
- R1 pad 1: +5V -> +3V3
- R10 pad 1: +5V -> +3V3
- R11 pad 1: +5V -> +3V3
- R12 pad 1: +5V -> +3V3
- R13 pad 1: +5V -> +3V3
- R14 pad 1: +5V -> +3V3
- R15 pad 1: +5V -> +3V3
- R16 pad 1: +5V -> +3V3
- R17 pad 1: +5V -> +3V3
- R18 pad 1: +5V -> +3V3
- R19 pad 1: +5V -> +3V3
- R2 pad 1: +5V -> +3V3
- R20 pad 1: +5V -> +3V3
- R21 pad 1: +5V -> +3V3
- R22 pad 1: +5V -> +3V3
- R23 pad 1: +5V -> +3V3
- R24 pad 1: +5V -> +3V3
- R25 pad 1: +5V -> +3V3
- R26 pad 1: +5V -> +3V3
- R27 pad 1: +5V -> +3V3
- R28 pad 1: +5V -> +3V3
- R29 pad 1: +5V -> +3V3
- R3 pad 1: +5V -> +3V3
- R30 pad 1: +5V -> +3V3
- R32 pad 1: +5V -> +3V3
- R33 pad 1: +5V -> +3V3
- R34 pad 1: +5V -> +3V3
- R35 pad 1: +5V -> +3V3
- R36 pad 1: +5V -> +3V3
- R37 pad 1: +5V -> +3V3
- R38 pad 1: +5V -> +3V3
- R4 pad 1: +5V -> +3V3
- R40 pad 1: +5V -> +3V3
- R41 pad 1: +5V -> +3V3
- R42 pad 1: +5V -> +3V3
- R43 pad 1: +5V -> +3V3
- R44 pad 1: +5V -> +3V3
- R5 pad 1: +5V -> +3V3
- R50 pad 1: Net-(J2-Pad2) -> +24V
- R51 pad 1: Net-(J2-Pad3) -> +24V
- R52 pad 1: Net-(J2-Pad4) -> +24V
- R53 pad 1: Net-(J2-Pad5) -> +24V
- R54 pad 1: Net-(J2-Pad6) -> +24V
- R55 pad 1: Net-(J2-Pad7) -> +24V
- R56 pad 1: Net-(J2-Pad8) -> +24V
- R57 pad 1: Net-(J3-Pad2) -> +24V
- R58 pad 1: Net-(J3-Pad3) -> +24V
- R59 pad 1: Net-(J3-Pad4) -> +24V
- R6 pad 1: +5V -> +3V3
- R60 pad 1: Net-(J3-Pad5) -> +24V
- R61 pad 1: Net-(J3-Pad6) -> +24V
- R62 pad 1: Net-(J3-Pad7) -> +24V
- R63 pad 1: Net-(J3-Pad8) -> +24V
- R64 pad 1: Net-(J4-Pad2) -> +24V
- R65 pad 1: Net-(J4-Pad3) -> +24V
- R66 pad 1: Net-(J4-Pad4) -> +24V
- R67 pad 1: Net-(J4-Pad5) -> +24V
- R68 pad 1: Net-(J4-Pad6) -> +24V
- R69 pad 1: Net-(J4-Pad7) -> +24V
- R7 pad 1: +5V -> +3V3
- R70 pad 1: Net-(J4-Pad8) -> +24V
- R71 pad 1: Net-(J5-Pad2) -> +24V
- R72 pad 1: Net-(J5-Pad3) -> +24V
- R73 pad 1: Net-(J5-Pad4) -> +24V
- R74 pad 1: Net-(J5-Pad5) -> +24V
- R75 pad 1: Net-(J5-Pad6) -> +24V
- R76 pad 1: Net-(J5-Pad7) -> +24V
- R77 pad 1: Net-(J5-Pad8) -> +24V
- R78 pad 1: Net-(J6-Pad2) -> +24V
- R79 pad 1: Net-(J6-Pad3) -> +24V
- R8 pad 1: +5V -> +3V3
- R80 pad 1: Net-(J6-Pad4) -> +24V
- R81 pad 1: Net-(J6-Pad5) -> +24V
- R82 pad 1: Net-(J6-Pad6) -> +24V
- R83 pad 1: Net-(J6-Pad7) -> +24V
- R84 pad 1: Net-(J6-Pad8) -> +24V
- R85 pad 1: Net-(J7-Pad2) -> +24V
- R86 pad 1: Net-(J7-Pad3) -> +24V
- R87 pad 1: Net-(J7-Pad4) -> +24V
- R88 pad 1: Net-(J7-Pad5) -> +24V
- R89 pad 1: Net-(J7-Pad6) -> +24V
- R9 pad 1: +5V -> +3V3
- R90 pad 1: Net-(J7-Pad7) -> +24V
- R91 pad 1: Net-(J7-Pad8) -> +24V
- R94 pad 1: +5V -> +3V3
- R95 pad 1: +5V -> +3V3
- R96 pad 1: +5V -> +3V3
- U10 pad 10: P8.11 -> P8.09
- U10 pad 12: P8.12 -> P8.10
- U10 pad 14: P8.13 -> P8.11
- U10 pad 16: P8.14 -> P8.12
- U10 pad 2: GNDA -> Net-(J6-Pad6)
- U10 pad 4: GNDA -> Net-(J6-Pad7)
- U10 pad 6: GNDA -> Net-(J6-Pad8)
- U10 pad 8: GNDA -> Net-(J7-Pad2)
- U11 pad 10: P8.07 -> P8.05
- U11 pad 12: P8.08 -> P8.06
- U11 pad 14: P8.09 -> P8.07
- U11 pad 16: P8.10 -> P8.08
- U11 pad 2: GNDA -> Net-(J7-Pad3)
- U11 pad 4: GNDA -> Net-(J7-Pad4)
- U11 pad 6: GNDA -> Net-(J7-Pad5)
- U11 pad 8: GNDA -> Net-(J7-Pad6)
- U12 pad 10: P8.03 -> Net-(U12-Pad10)
- U12 pad 11: GND -> Net-(U12-Pad11)
- U12 pad 12: P8.04 -> Net-(U12-Pad12)
- U12 pad 14: P8.05 -> P8.03
- U12 pad 16: P8.06 -> P8.04
- U12 pad 2: GNDA -> Net-(J7-Pad7)
- U12 pad 4: GNDA -> Net-(J7-Pad8)
- U12 pad 6: GNDA -> Net-(U12-Pad6)
- U12 pad 8: GNDA -> Net-(U12-Pad8)
- U12 pad 9: GND -> Net-(U12-Pad9)
- U13 pad 8: +5V -> +3V3
- U2 pad 2: GNDA -> Net-(J2-Pad2)
- U2 pad 4: GNDA -> Net-(J2-Pad3)
- U2 pad 6: GNDA -> Net-(J2-Pad4)
- U2 pad 8: GNDA -> Net-(J2-Pad5)
- U3 pad 2: GNDA -> Net-(J2-Pad6)
- U3 pad 4: GNDA -> Net-(J2-Pad7)
- U3 pad 6: GNDA -> Net-(J2-Pad8)
- U3 pad 8: GNDA -> Net-(J3-Pad2)
- U4 pad 2: GNDA -> Net-(J3-Pad3)
- U4 pad 4: GNDA -> Net-(J3-Pad4)
- U4 pad 6: GNDA -> Net-(J3-Pad5)
- U4 pad 8: GNDA -> Net-(J3-Pad6)
- U5 pad 2: GNDA -> Net-(J3-Pad7)
- U5 pad 4: GNDA -> Net-(J3-Pad8)
- U5 pad 6: GNDA -> Net-(J4-Pad2)
- U5 pad 8: GNDA -> Net-(J4-Pad3)
- U6 pad 2: GNDA -> Net-(J4-Pad4)
- U6 pad 4: GNDA -> Net-(J4-Pad5)
- U6 pad 6: GNDA -> Net-(J4-Pad6)
- U6 pad 8: GNDA -> Net-(J4-Pad7)
- U7 pad 2: GNDA -> Net-(J4-Pad8)
- U7 pad 4: GNDA -> Net-(J5-Pad2)
- U7 pad 6: GNDA -> Net-(J5-Pad3)
- U7 pad 8: GNDA -> Net-(J5-Pad4)
- U8 pad 10: P8.19 -> P8.18
- U8 pad 2: GNDA -> Net-(J5-Pad5)
- U8 pad 4: GNDA -> Net-(J5-Pad6)
- U8 pad 6: GNDA -> Net-(J5-Pad7)
- U8 pad 8: GNDA -> Net-(J5-Pad8)
- U9 pad 10: P8.15 -> P8.14
- U9 pad 12: P8.16 -> P8.15
- U9 pad 14: P8.17 -> P8.16
- U9 pad 16: P8.18 -> P8.17
- U9 pad 2: GNDA -> Net-(J6-Pad2)
- U9 pad 4: GNDA -> Net-(J6-Pad3)
- U9 pad 6: GNDA -> Net-(J6-Pad4)
- U9 pad 8: GNDA -> Net-(J6-Pad5)
Other:
- board text removed: "+5V"
- board text removed: "P8.03"
- board text removed: "P8.04"
- board text removed: "P9.11"
- board text removed: "P9.12"
- board text removed: "P9.13"
- board text removed: "P9.14"
- board text removed: "P9.15"
- board text removed: "P9.16"
- board text removed: "P9.17"
- board text removed: "P9.18"
- board text removed: "P9.21"
- board text removed: "P9.22"
- board text removed: "P9.23"
- board text removed: "P9.24"
- board text removed: "P9.25"
- board text removed: "P9.26"
- board text removed: "P9.27"
- board text removed: "P9.28"
- board text removed: "P9.29"
- board text removed: "P9.30"
- board text removed: "P9.31"
- board text removed: "P9.42"

Commit message: test
Parts:
- removed AN1: Screw_Terminal_01x07, Connector_Phoenix_MSTB:PhoenixContact_MSTBA_2,5_7-G_1x07_P5.00mm_Horizontal
- removed the C10 at (103.1, 84.3)
- removed the C18 at (46.9, 85.3)
- removed the J1 at (224.1, 117.7)
- removed the J2 at (159.3, 60.4)
- removed the L2 at (155.6, 87.1)
- removed P3, P4: BeagleBone_Black_Header, Connector_PinHeader_2.54mm:PinHeader_2x23_P2.54mm_Vertical
- removed the R15 at (45.6, 101.2)
- removed the R17 at (73.6, 81.1)
- removed the R42 at (38.1, 101.1)
- removed R65, R66, R67, R68, R69, R70, R71, R72, R73, R74, R75, R76, R77, R78, R79, R80, R81, R82, R83, R84, R85, R86, R87, R88, R89, R90, R91, R94, R95: 10k, Resistor_SMD:R_0603_1608Metric
- added C31: 100n, Capacitor_SMD:C_0603_1608Metric, F.Cu at (17.7, 68.7)
- added C39: 100n, Capacitor_SMD:C_0603_1608Metric, F.Cu at (121.0, 31.6)
- added C44: 100n, Capacitor_SMD:C_0603_1608Metric, F.Cu at (143.9, 10.4)
- added C48: 100n, Capacitor_SMD:C_0603_1608Metric, F.Cu at (254.3, 77.8)
- added C49: 100n, Capacitor_SMD:C_0603_1608Metric, F.Cu at (138.7, 16.0)
- added C50: 100n, Capacitor_SMD:C_0603_1608Metric, F.Cu at (116.9, 38.6)
- added C51: 100n, Capacitor_SMD:C_0603_1608Metric, F.Cu at (121.0, 34.1)
- added C52: 100n, Capacitor_SMD:C_0603_1608Metric, F.Cu at (134.0, 21.0)
- added C53: 100n, Capacitor_SMD:C_0603_1608Metric, F.Cu at (142.7, 13.5)
- added C54: 100n, Capacitor_SMD:C_0603_1608Metric, F.Cu at (108.9, 43.6)
- added C55: 100n, Capacitor_SMD:C_0603_1608Metric, F.Cu at (89.2, 42.9)
- added C56: 100n, Capacitor_SMD:C_0603_1608Metric, F.Cu at (144.9, -0.94)
- added C57: 100n, Capacitor_SMD:C_0603_1608Metric, F.Cu at (130.6, 14.1)
- added C58: 100n, Capacitor_SMD:C_0603_1608Metric, F.Cu at (119.8, 26.5)
- added D1: B340A-13F, Diode_SMD:D_SMA, F.Cu at (106.9, 35.1)
- added D2: SS34, Diode_SMD:D_SMA, F.Cu at (113.7, 27.5)
- added D4: BAT54A, Package_TO_SOT_SMD:SOT-23, F.Cu at (254.1, 98.9)
- added D5: 1N4148, Diode_SMD:D_MiniMELF, F.Cu at (250.9, 78.9)
- added F1: Fuse_3A, Fuse:Fuse_2512_6332Metric, F.Cu at (124.3, 15.3)
- added J10: BeagleBone_Black_Header, Connector_PinHeader_2.54mm:PinHeader_2x23_P2.54mm_Vertical, F.Cu at (265.4, 116.8)
- added J11: BeagleBone_Black_Header, Connector_PinHeader_2.54mm:PinHeader_2x23_P2.54mm_Vertical, F.Cu at (217.1, 116.8)
- added J12: Conn_02x04_Odd_Even, Connector_PinHeader_2.54mm:PinHeader_2x04_P2.54mm_Vertical, B.Cu at (102.5, 89.3)
- added J13: Screw_Terminal_01x04, Connector:Phoenix_1x04_P5.00mm_Horizontal, F.Cu at (153.9, 117.8)
- added J5: Screw_Terminal_01x08, Connector:8pin, F.Cu at (141.6, 60.4)
- added J7: Screw_Terminal_01x08, Connector:8pin, F.Cu at (257.8, 60.4)
- added J8: Screw_Terminal_01x08, Connector:8pin, F.Cu at (186.3, 60.5)
- added L1: 4.7uH, Inductor_SMD:L_12x12mm_H6mm, F.Cu at (159.1, 86.7)
- added PS1: B2424S-1WR2, Module:CONV_B0505S-1WR2, F.Cu at (102.8, 6.41)
- added R31: 4.7k, Resistor_SMD:R_0603_1608Metric, F.Cu at (130.6, 16.6)
- added R39: 10k, Resistor_SMD:R_0603_1608Metric, F.Cu at (37.1, 115.8)
- added R47: 10k, Resistor_SMD:R_0603_1608Metric, F.Cu at (70.3, 115.8)
- added R48: 10k, Resistor_SMD:R_0603_1608Metric, F.Cu at (75.0, 115.8)
- added R49: 10k, Resistor_SMD:R_0603_1608Metric, F.Cu at (79.8, 115.8)
- added REF**: YAAJ_DCDC_StepDown_LM2596, Module:YAAJ_DCDC_StepDown_LM2596, F.Cu at (144.9, 81.5)
- added U13: EL357N-G, Package_SO:OPTO_EL357N-G, F.Cu at (138.2, -1.25)
- added U14: EL357N-G, Package_SO:OPTO_EL357N-G, F.Cu at (108.2, 107.5)
- added U15: EL357N-G, Package_SO:OPTO_EL357N-G, F.Cu at (75.2, 22.1)
- added U16: EL357N-G, Package_SO:OPTO_EL357N-G, F.Cu at (118.3, -1.25)
- added U17: EL357N-G, Package_SO:OPTO_EL357N-G, F.Cu at (128.2, -6.89)
- added U18: EL357N-G, Package_SO:OPTO_EL357N-G, F.Cu at (65.1, 74.2)
- added U19: EL357N-G, Package_SO:OPTO_EL357N-G, F.Cu at (95.1, 24.3)
- added U20: EL357N-G, Package_SO:OPTO_EL357N-G, F.Cu at (95.1, 30.0)
- added U21: EL357N-G, Package_SO:OPTO_EL357N-G, F.Cu at (78.3, 39.0)
- added U22: EL357N-G, Package_SO:OPTO_EL357N-G, F.Cu at (46.2, 74.2)
- added U23: EL357N-G, Package_SO:OPTO_EL357N-G, F.Cu at (41.5, 74.2)
- added U24: EL357N-G, Package_SO:OPTO_EL357N-G, F.Cu at (115.2, 11.1)
- added U25: EL357N-G, Package_SO:OPTO_EL357N-G, F.Cu at (32.0, 74.2)
- added U26: EL357N-G, Package_SO:OPTO_EL357N-G, F.Cu at (27.2, 74.2)
- added U27: EL357N-G, Package_SO:OPTO_EL357N-G, F.Cu at (88.2, 38.8)
- added U27: EL357N-G, Package_SO:OPTO_EL357N-G, F.Cu at (22.5, 74.2)
- added U28: RS485, Module:RS485_moduleTTL, B.Cu at (233.4, 67.0)
- added U29: EL357N-G, Package_SO:OPTO_EL357N-G, F.Cu at (17.8, 74.2)
- added U30: EL357N-G, Package_SO:OPTO_EL357N-G, F.Cu at (18.2, 107.5)
- added U31: EL357N-G, Package_SO:OPTO_EL357N-G, F.Cu at (23.0, 107.5)
- added U32: EL357N-G, Package_SO:OPTO_EL357N-G, F.Cu at (27.7, 107.5)
- added U34: EL357N-G, Package_SO:OPTO_EL357N-G, F.Cu at (32.4, 107.5)
- added U35: EL357N-G, Package_SO:OPTO_EL357N-G, F.Cu at (128.2, -1.25)
- added U36: EL357N-G, Package_SO:OPTO_EL357N-G, F.Cu at (105.0, 24.3)
- added U37: EL357N-G, Package_SO:OPTO_EL357N-G, F.Cu at (124.5, 4.41)
- added U38: EL357N-G, Package_SO:OPTO_EL357N-G, F.Cu at (105.3, 18.7)
- added U39: EL357N-G, Package_SO:OPTO_EL357N-G, F.Cu at (56.0, 107.5)
- added U40: EL357N-G, Package_SO:OPTO_EL357N-G, F.Cu at (98.2, 41.3)
- added U41: EL357N-G, Package_SO:OPTO_EL357N-G, F.Cu at (95.4, 18.7)
- added U42: EL357N-G, Package_SO:OPTO_EL357N-G, F.Cu at (105.3, 13.0)
- added U43: EL357N-G, Package_SO:OPTO_EL357N-G, F.Cu at (75.0, 107.5)
- added U44: EL357N-G, Package_SO:OPTO_EL357N-G, F.Cu at (85.1, 33.1)
- added U45: EL357N-G, Package_SO:OPTO_EL357N-G, F.Cu at (84.5, 107.5)
- added U46: P82B96, Package_SO:SO-8_3.9x4.9mm_P1.27mm, F.Cu at (254.1, 103.9)
- added U47: EL357N-G, Package_SO:OPTO_EL357N-G, F.Cu at (114.6, 5.46)
- added U48: EL357N-G, Package_SO:OPTO_EL357N-G, F.Cu at (85.1, 27.5)
- added U49: EL357N-G, Package_SO:OPTO_EL357N-G, F.Cu at (95.4, 13.0)
- added U50: EL357N-G, Package_SO:OPTO_EL357N-G, F.Cu at (85.1, 21.8)
- added U51: EL357N-G, Package_SO:OPTO_EL357N-G, F.Cu at (75.2, 33.4)
- added U52: EL357N-G, Package_SO:OPTO_EL357N-G, F.Cu at (118.3, -6.89)
- added U53: EL357N-G, Package_SO:OPTO_EL357N-G, F.Cu at (75.2, 27.7)
- added U54: EL357N-G, Package_SO:OPTO_EL357N-G, F.Cu at (125.2, 10.1)
- added U55: EL357N-G, Package_SO:OPTO_EL357N-G, F.Cu at (138.2, -6.89)
- added U56: EL357N-G, Package_SO:OPTO_EL357N-G, F.Cu at (98.2, 35.6)
- BT1: footprint Battery:BatteryHolder_Keystone_103_1x20mm -> Battery:Battery_Panasonic_CR1220-VCN_Vertical_CircularHoles; moved to F.Cu
- C17: value 100n -> 3n3; footprint Capacitor_SMD:C_0603_1608Metric -> Capacitor_SMD:C_0805_2012Metric
- C43: value 100u/50V -> 100n; footprint Capacitor_SMD:CP_Elec_8x10 -> Capacitor_SMD:C_0603_1608Metric
- C47: value 3n3 -> 100n; footprint Capacitor_SMD:C_0805_2012Metric -> Capacitor_SMD:C_0603_1608Metric
- C9: value 100n -> 100uF/50V; footprint Capacitor_SMD:C_0603_1608Metric -> Capacitor_SMD:CP_Elec_8x10
- D2: renamed from D3; value 1N5825 -> SS34
- D3: renamed from D4; value LED_GREEN -> LED_RED
- J9: value Conn_02x13_Odd_Even -> Screw_Terminal_01x08; footprint Connector_PinSocket_2.54mm:PinSocket_2x13_P2.54mm_Vertical -> Connector:8pin; moved to F.Cu
- R16: value 10k -> 1k
- R30: value 10k -> 4.7k
- R45, R46: value 4.7k -> 10k
- R50, R55, R56, R57, R58, R59, R60, R61, R62, R63, R64: moved to F.Cu
- R51, R52: value 10k -> 680R; moved to F.Cu
- R53: value 10k -> 330R; moved to F.Cu
- R54: value 10k -> 4.7k; moved to F.Cu
- SW1: footprint Button_Switch_THT:SW_PUSH_6mm_H8mm -> Button_Switch_THT:SW_PUSH_6mm_H13mm
- U1: value LM2596S-ADJ -> EL357N-G; footprint Package_TO_SOT_SMD:TO-263-5_TabPin3 -> Package_SO:OPTO_EL357N-G
- U10, U11, U12, U2, U3, U4, U5, U6, U7, U8: value PC847 -> EL357N-G; footprint Package_SO:SOP-16_4.55x10.3mm_P1.27mm -> Package_SO:OPTO_EL357N-G
- U9: value PC847 -> LM2596S-ADJ; footprint Package_SO:SOP-16_4.55x10.3mm_P1.27mm -> Package_TO_SOT_SMD:TO-263-5_TabPin3
- Y1: footprint Crystal:Crystal_C38-LF_D3.0mm_L8.0mm_Horizontal_1EP_style1 -> Crystal:Crystal_C26-LF_D2.1mm_L6.5mm_Horizontal; moved to F.Cu
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- renumbered C44 to C10, C48 to C18, D2 to D1, J3 to J1, J5 to J2, J4 to J3, J6 to J4, J7 to J6, L1 to L2, R47 to R15, R48 to R16, R49 to R17, R96 to R42, U13 to U33
Connections:
- ANVDD1 pad 1: P9.32 -> VDD_ADC
- ANVDD1 pad 2: P9.34 -> GND_ADC
- C1 pad 1: P8.18 -> Net-(C1-Pad1)
- C1 pad 2: GND -> P8.46_OUT
- C11 pad 1: P8.38 -> Net-(C11-Pad1)
- C11 pad 2: GND -> P8.42_OUT
- C12 pad 1: P8.31 -> Net-(C12-Pad1)
- C12 pad 2: GND -> P8.41_OUT
- C13 pad 1: P8.16 -> Net-(C13-Pad1)
- C13 pad 2: GND -> P8.40_OUT
- C14 pad 1: P8.09 -> Net-(C14-Pad1)
- C14 pad 2: GND -> P8.39_OUT
- C15 pad 1: P8.23 -> Net-(C15-Pad1)
- C15 pad 2: GND -> P9.21_OUT
- C16 pad 1: P8.44 -> Net-(C16-Pad1)
- C16 pad 2: GND -> P9.22_OUT
- C17 pad 1: P8.37 -> +5V
- C17 pad 2: GND -> Net-(C17-Pad2)
- C19 pad 1: P8.15 -> Net-(C19-Pad1)
- C19 pad 2: GND -> P8.38_OUT
- C2 pad 1: P8.11 -> Net-(C2-Pad1)
- C2 pad 2: GND -> P8.45_OUT
- C20 pad 1: P8.08 -> Net-(C20-Pad1)
- C20 pad 2: GND -> P8.37_OUT
- C21 pad 1: P8.22 -> Net-(C21-Pad1)
- C21 pad 2: GND -> P8.36_OUT
- C22 pad 1: P8.43 -> Net-(C22-Pad1)
- C22 pad 2: GND -> P8.35_OUT
- C23 pad 1: P8.36 -> Net-(C23-Pad1)
- C23 pad 2: GND -> P8.34_OUT
- C24 pad 1: P8.29 -> Net-(C24-Pad1)
- C24 pad 2: GND -> P8.33_OUT
- C25 pad 1: P8.14 -> Net-(C25-Pad1)
- C25 pad 2: GND -> P8.32_OUT
- C26 pad 1: P8.07 -> Net-(C26-Pad1)
- C26 pad 2: GND -> P8.31_OUT
- C27 pad 1: P8.21 -> Net-(C27-Pad1)
- C27 pad 2: GND -> P8.30_OUT
- C28 pad 1: P8.42 -> Net-(C28-Pad1)
- C28 pad 2: GND -> P8.29_OUT
- C29 pad 1: P8.35 -> Net-(C29-Pad1)
- C29 pad 2: GND -> P8.28_OUT
- C3 pad 1: P8.25 -> Net-(C3-Pad1)
- C3 pad 2: GND -> P8.44_OUT
- C30 pad 1: P8.28 -> Net-(C30-Pad1)
- C30 pad 2: GND -> P8.27_OUT
- C32 pad 1: P8.06 -> Net-(C32-Pad1)
- C32 pad 2: GND -> P9.16_OUT
- C33 pad 1: P8.20 -> Net-(C33-Pad1)
- C33 pad 2: GND -> P9.17_OUT
- C34 pad 1: P8.41 -> Net-(C34-Pad1)
- C34 pad 2: GND -> P9.18_OUT
- C35 pad 1: P8.34 -> Net-(C35-Pad1)
- C35 pad 2: GND -> P9.11_OUT
- C36 pad 1: P8.27 -> Net-(C36-Pad1)
- C36 pad 2: GND -> P9.12_OUT
- C37 pad 1: P8.12 -> Net-(C37-Pad1)
- C37 pad 2: GND -> P9.13_OUT
- C38 pad 1: P8.05 -> Net-(C38-Pad1)
- C38 pad 2: GND -> P8.18_OUT
- C4 pad 1: P8.46 -> Net-(C4-Pad1)
- C4 pad 2: GND -> P8.43_OUT
- C40 pad 1: P8.40 -> Net-(C40-Pad1)
- C40 pad 2: GND -> P8.16_OUT
- C41 pad 1: P8.33 -> Net-(C41-Pad1)
- C41 pad 2: GND -> P8.15_OUT
- C42 pad 1: P8.26 -> Net-(C42-Pad1)
- C42 pad 2: GND -> P8.14_OUT
- C43 pad 1: +24V -> Net-(C43-Pad1)
- C43 pad 2: Earth -> P8.12_OUT
- C45 pad 1: P8.04 -> Net-(C45-Pad1)
- C45 pad 2: GND -> P8.10_OUT
- C46 pad 1: P8.03 -> Net-(C46-Pad1)
- C46 pad 2: GND -> P8.09_OUT
- C47 pad 1: +5V -> +3V3
- C47 pad 2: Net-(C47-Pad2) -> GND
- C5 pad 1: P8.39 -> Net-(C5-Pad1)
- C5 pad 2: GND -> P8.08_OUT
- C6 pad 1: P8.32 -> Net-(C6-Pad1)
- C6 pad 2: GND -> P8.07_OUT
- C7 pad 1: P8.17 -> Net-(C7-Pad1)
- C7 pad 2: GND -> P9.14_OUT
- C8 pad 1: P8.10 -> Net-(C8-Pad1)
- C8 pad 2: GND -> P9.15_OUT
- C9 pad 1: P8.24 -> +24V
- C9 pad 2: GND -> Earth
- D2 pad 1: Net-(D3-Pad1) -> Net-(D2-Pad1)
- J1 pad 2: Net-(J3-Pad2) -> P8.39_OUT
- J1 pad 3: Net-(J3-Pad3) -> P8.38_OUT
- J1 pad 4: Net-(J3-Pad4) -> P8.37_OUT
- J1 pad 5: Net-(J3-Pad5) -> P8.36_OUT
- J1 pad 6: Net-(J3-Pad6) -> P8.35_OUT
- J1 pad 7: Net-(J3-Pad7) -> P8.34_OUT
- J1 pad 8: Net-(J3-Pad8) -> P8.33_OUT
- J2 pad 2: Net-(J5-Pad2) -> P9.11_OUT
- J2 pad 3: Net-(J5-Pad3) -> P9.12_OUT
- J2 pad 4: Net-(J5-Pad4) -> P9.13_OUT
- J2 pad 5: Net-(J5-Pad5) -> P9.14_OUT
- J2 pad 6: Net-(J5-Pad6) -> P9.15_OUT
- J2 pad 7: Net-(J5-Pad7) -> P9.16_OUT
- J2 pad 8: Net-(J5-Pad8) -> P8.18_OUT
- J3 pad 2: Net-(J4-Pad2) -> P8.32_OUT
- J3 pad 3: Net-(J4-Pad3) -> P8.31_OUT
- J3 pad 4: Net-(J4-Pad4) -> P8.30_OUT
- J3 pad 5: Net-(J4-Pad5) -> P8.29_OUT
- J3 pad 6: Net-(J4-Pad6) -> P8.28_OUT
- J3 pad 7: Net-(J4-Pad7) -> P8.27_OUT
- J3 pad 8: Net-(J4-Pad8) -> P8.26_OUT
- J4 pad 2: Net-(J6-Pad2) -> P8.17_OUT
- J4 pad 3: Net-(J6-Pad3) -> P8.16_OUT
- J4 pad 4: Net-(J6-Pad4) -> P8.15_OUT
- J4 pad 5: Net-(J6-Pad5) -> P8.14_OUT
- J4 pad 6: Net-(J6-Pad6) -> P8.12_OUT
- J4 pad 7: Net-(J6-Pad7) -> P8.11_OUT
- J4 pad 8: Net-(J6-Pad8) -> P8.10_OUT
- J6 pad 2: Net-(J7-Pad2) -> P8.09_OUT
- J6 pad 3: Net-(J7-Pad3) -> P8.08_OUT
- J6 pad 4: Net-(J7-Pad4) -> P8.07_OUT
- J6 pad 5: Net-(J7-Pad5) -> P9.42_OUT
- J6 pad 6: Net-(J7-Pad6) -> P9.31_OUT
- J6 pad 7: Net-(J7-Pad7) -> P9.30_OUT
- J6 pad 8: Net-(J7-Pad8) -> P9.29_OUT
- J9 pad 1: +24V -> +5V
- J9 pad 2: GND -> +3V3
- J9 pad 3: P9.11 -> GND
- J9 pad 4: P9.42 -> SDA_OUT
- J9 pad 5: P9.12 -> SCL_OUT
- J9 pad 6: P9.31 -> A+
- J9 pad 7: P9.13 -> B-
- J9 pad 8: P9.30 -> GNDD
- R1 pad 1: +3V3 -> Net-(C1-Pad1)
- R1 pad 2: P8.18 -> +24VA
- R10 pad 1: +3V3 -> Net-(C12-Pad1)
- R10 pad 2: P8.45 -> +24VA
- R11 pad 1: +3V3 -> Net-(C13-Pad1)
- R11 pad 2: P8.38 -> +24VA
- R12 pad 1: +3V3 -> Net-(C14-Pad1)
- R12 pad 2: P8.31 -> +24VA
- R13 pad 1: +3V3 -> Net-(C15-Pad1)
- R13 pad 2: P8.16 -> +24VA
- R14 pad 1: +3V3 -> Net-(C16-Pad1)
- R14 pad 2: P8.09 -> +24VA
- R15 pad 2: Net-(C47-Pad2) -> Net-(C17-Pad2)
- R16 pad 1: +3V3 -> Net-(C17-Pad2)
- R16 pad 2: P8.44 -> Earth
- R16 pad 1: Net-(C47-Pad2) -> Net-(C17-Pad2)
- R18 pad 1: +3V3 -> Net-(C19-Pad1)
- R18 pad 2: P8.30 -> +24VA
- R19 pad 1: +3V3 -> Net-(C20-Pad1)
- R19 pad 2: P8.15 -> +24VA
- R2 pad 1: +3V3 -> Net-(C2-Pad1)
- R2 pad 2: P8.11 -> +24VA
- R20 pad 1: +3V3 -> Net-(C21-Pad1)
- R20 pad 2: P8.08 -> +24VA
- R21 pad 1: +3V3 -> Net-(C22-Pad1)
- R21 pad 2: P8.22 -> +24VA
- R22 pad 1: +3V3 -> Net-(C23-Pad1)
- R22 pad 2: P8.43 -> +24VA
- R23 pad 1: +3V3 -> Net-(C24-Pad1)
- R23 pad 2: P8.36 -> +24VA
- R24 pad 1: +3V3 -> Net-(C25-Pad1)
- R24 pad 2: P8.29 -> +24VA
- R25 pad 1: +3V3 -> Net-(C26-Pad1)
- R25 pad 2: P8.14 -> +24VA
- R26 pad 1: +3V3 -> Net-(C27-Pad1)
- R26 pad 2: P8.07 -> +24VA
- R27 pad 1: +3V3 -> Net-(C28-Pad1)
- R27 pad 2: P8.21 -> +24VA
- R28 pad 1: +3V3 -> Net-(C29-Pad1)
- R28 pad 2: P8.42 -> +24VA
- R29 pad 1: +3V3 -> Net-(C30-Pad1)
- R29 pad 2: P8.35 -> +24VA
- R3 pad 1: +3V3 -> Net-(C3-Pad1)
- R3 pad 2: P8.25 -> +24VA
- R30 pad 2: P8.28 -> SCL
- R32 pad 1: +3V3 -> Net-(C31-Pad1)
- R32 pad 2: P8.06 -> +24VA
- R33 pad 1: +3V3 -> Net-(C32-Pad1)
- R33 pad 2: P8.20 -> +24VA
- R34 pad 1: +3V3 -> Net-(C33-Pad1)
- R34 pad 2: P8.41 -> +24VA
- R35 pad 1: +3V3 -> Net-(C34-Pad1)
- R35 pad 2: P8.34 -> +24VA
- R36 pad 2: P8.27 -> SDA
- R37 pad 2: P8.12 -> SCL
- R38 pad 1: +3V3 -> Net-(C35-Pad1)
- R38 pad 2: P8.05 -> +24VA
- R4 pad 1: +3V3 -> Net-(C4-Pad1)
- R4 pad 2: P8.46 -> +24VA
- R40 pad 1: +3V3 -> Net-(C37-Pad1)
- R40 pad 2: P8.40 -> +24VA
- R41 pad 1: +3V3 -> Net-(C38-Pad1)
- R41 pad 2: P8.33 -> +24VA
- R43 pad 1: +3V3 -> Net-(C39-Pad1)
- R43 pad 2: P8.04 -> +24VA
- R44 pad 1: +3V3 -> Net-(C40-Pad1)
- R44 pad 2: P8.03 -> +24VA
- R45 pad 1: +3V3 -> Net-(C41-Pad1)
- R45 pad 2: SCL -> +24VA
- R46 pad 1: +3V3 -> Net-(C42-Pad1)
- R46 pad 2: SDA -> +24VA
- R5 pad 1: +3V3 -> Net-(C5-Pad1)
- R5 pad 2: P8.39 -> +24VA
- R50 pad 1: +24V -> Net-(C46-Pad1)
- R50 pad 2: Net-(R50-Pad2) -> +24VA
- R51 pad 1: +24V -> +3V3
- R51 pad 2: Net-(R51-Pad2) -> SCL_OUT
- R52 pad 1: +24V -> +3V3
- R52 pad 2: Net-(R52-Pad2) -> SDA_OUT
- R53 pad 1: +24V -> Net-(R53-Pad1)
- R53 pad 2: Net-(R53-Pad2) -> GND
- R54 pad 1: +24V -> +3V3
- R54 pad 2: Net-(R54-Pad2) -> P9.41
- R55 pad 1: +24V -> Net-(C49-Pad1)
- R55 pad 2: Net-(R55-Pad2) -> +24VA
- R56 pad 1: +24V -> Net-(C50-Pad1)
- R56 pad 2: Net-(R56-Pad2) -> +24VA
- R57 pad 1: +24V -> Net-(C51-Pad1)
- R57 pad 2: Net-(R57-Pad2) -> +24VA
- R58 pad 1: +24V -> Net-(C52-Pad1)
- R58 pad 2: Net-(R58-Pad2) -> +24VA
- R59 pad 1: +24V -> Net-(C53-Pad1)
- R59 pad 2: Net-(R59-Pad2) -> +24VA
- R6 pad 1: +3V3 -> Net-(C6-Pad1)
- R6 pad 2: P8.32 -> +24VA
- R60 pad 1: +24V -> Net-(C54-Pad1)
- R60 pad 2: Net-(R60-Pad2) -> +24VA
- R61 pad 1: +24V -> Net-(C55-Pad1)
- R61 pad 2: Net-(R61-Pad2) -> +24VA
- R62 pad 1: +24V -> Net-(C56-Pad1)
- R62 pad 2: Net-(R62-Pad2) -> +24VA
- R63 pad 1: +24V -> Net-(C57-Pad1)
- R63 pad 2: Net-(R63-Pad2) -> +24VA
- R64 pad 1: +24V -> Net-(C58-Pad1)
- R64 pad 2: Net-(R64-Pad2) -> +24VA
- R7 pad 1: +3V3 -> Net-(C7-Pad1)
- R7 pad 2: P8.17 -> +24VA
- R8 pad 1: +3V3 -> Net-(C8-Pad1)
- R8 pad 2: P8.10 -> +24VA
- R9 pad 1: +3V3 -> Net-(C11-Pad1)
- R9 pad 2: P8.24 -> +24VA
- SW1 pad 1: GND -> Net-(R53-Pad1)
- U1 pad 1: +24V -> Net-(C1-Pad1)
- U1 pad 2: Net-(D3-Pad1) -> P8.46_OUT
- U1 pad 3: Earth -> GND
- U1 pad 4: Net-(C47-Pad2) -> P8.46
- U10 pad 1: Net-(R82-Pad2) -> Net-(C11-Pad1)
- U10 pad 2: Net-(J6-Pad6) -> P8.42_OUT
- U10 pad 3: Net-(R83-Pad2) -> GND
- U10 pad 4: Net-(J6-Pad7) -> P8.42
- U11 pad 1: Net-(R86-Pad2) -> Net-(C12-Pad1)
- U11 pad 2: Net-(J7-Pad3) -> P8.41_OUT
- U11 pad 3: Net-(R87-Pad2) -> GND
- U11 pad 4: Net-(J7-Pad4) -> P8.41
- U12 pad 1: Net-(R90-Pad2) -> Net-(C13-Pad1)
- U12 pad 2: Net-(J7-Pad7) -> P8.40_OUT
- U12 pad 3: Net-(R91-Pad2) -> GND
- U12 pad 4: Net-(J7-Pad8) -> P8.40
- U2 pad 1: Net-(R50-Pad2) -> Net-(C2-Pad1)
- U2 pad 2: Net-(J2-Pad2) -> P8.45_OUT
- U2 pad 3: Net-(R51-Pad2) -> GND
- U2 pad 4: Net-(J2-Pad3) -> P8.45
- U3 pad 1: Net-(R54-Pad2) -> Net-(C3-Pad1)
- U3 pad 2: Net-(J2-Pad6) -> P8.44_OUT
- U3 pad 3: Net-(R55-Pad2) -> GND
- U3 pad 4: Net-(J2-Pad7) -> P8.44
- U4 pad 1: Net-(R58-Pad2) -> Net-(C4-Pad1)
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Routing:
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- added copper zone on F.Cu, net +24V
- added copper zone on B.Cu, net Earth
- added copper zone on F.Cu, net Earth
- added copper zone on B.Cu, net GNDA
- added copper zone on F.Cu, net GNDA
- added copper zone on F.Cu, net Net-(D2-Pad1)
- removed copper zone on F.Cu, net (none)
- removed copper zone on F.Cu, net Net-(D3-Pad1)
Other:
- board size 231 x 74 mm -> 256 x 74 mm
- board text added: "+5V"
- board text added: "1.Dołożyć Drganie styków na Switch 2. Poprawić poligony GND"
- board text added: "A+"
- board text added: "B-"
- board text added: "GND_RS"
- board text added: "LM2596"
- board text added: "P8.03"
- board text added: "P8.04"
- board text added: "RS485"
- board text added: "RTC CLOCK"
- board text added: "input board v0.2"
- board text removed: "AIN0"
- board text removed: "AIN1"
- board text removed: "AIN2"
- board text removed: "AIN3"
- board text removed: "AIN4"
- board text removed: "AIN5"
- board text removed: "AIN6"
- board text removed: "P8.13"
- board text removed: "P8.19"
- board text removed: "boneIO - input board v0.1 Author - Maciej Krasuski"

Commit message: 03.11.2021
Parts:
- removed the D1 at (106.9, 35.1)
- removed the F1 at (124.3, 15.3)
- removed PS1: B2424S-1WR2, Module:CONV_B0505S-1WR2
- removed U15, U16, U17, U18, U19, U20, U21, U22, U23, U24, U25, U26, U27 (x2), U29, U30, U31, U32, U34, U35, U36, U37, U38, U39, U40, U41, U42, U43, U44, U45, U47, U48, U49, U50, U51, U52, U53, U54, U55, U56: EL357N-G, Package_SO:OPTO_EL357N-G
- added J14: ZW_VCC, Connector_PinHeader_2.54mm:PinHeader_1x03_P2.54mm_Vertical, F.Cu at (18.0, 81.8)
- added J15: ZW_GND, Connector_PinHeader_2.54mm:PinHeader_1x03_P2.54mm_Vertical, F.Cu at (18.0, 97.7)
- added J16: INNY ZASILACZ, Connector:Phoenix_1x02_P5.00mm_Horizontal, F.Cu at (200.7, 64.0)
- added R100: 10k, Resistor_SMD:R_0603_1608Metric, F.Cu at (223.2, 22.9)
- added R101: 10k, Resistor_SMD:R_0603_1608Metric, F.Cu at (215.5, 30.4)
- added R102: 10k, Resistor_SMD:R_0603_1608Metric, F.Cu at (227.2, 18.6)
- added R103: 10k, Resistor_SMD:R_0603_1608Metric, F.Cu at (242.9, 3.54)
- added R104: 10k, Resistor_SMD:R_0603_1608Metric, F.Cu at (235.6, 11.1)
- added R105: 10k, Resistor_SMD:R_0603_1608Metric, F.Cu at (231.6, 16.1)
- added R106: 10k, Resistor_SMD:R_0603_1608Metric, F.Cu at (211.5, 33.0)
- added R107: 10k, Resistor_SMD:R_0603_1608Metric, F.Cu at (207.4, 39.8)
- added R108: 10k, Resistor_SMD:R_0603_1608Metric, F.Cu at (219.5, 27.9)
- added R109: 4,7k, Resistor_SMD:R_0603_1608Metric, F.Cu at (231.2, 21.1)
- added R110: 4,7k, Resistor_SMD:R_0603_1608Metric, F.Cu at (239.6, 11.1)
- added R111: 4,7k, Resistor_SMD:R_0603_1608Metric, F.Cu at (235.6, 16.1)
- added R112: 4,7k, Resistor_SMD:R_0603_1608Metric, F.Cu at (215.5, 35.5)
- added R113: 10k, Resistor_SMD:R_0603_1608Metric, F.Cu at (227.2, 23.6)
- added R114: 10k, Resistor_SMD:R_0603_1608Metric, F.Cu at (223.5, 27.9)
- added R115: 10k, Resistor_SMD:R_0603_1608Metric, F.Cu at (243.6, 8.56)
- added R116: 10k, Resistor_SMD:R_0603_1608Metric, F.Cu at (235.6, 13.6)
- added R65: 10k, Resistor_SMD:R_0603_1608Metric, F.Cu at (238.9, 3.54)
- added R66: 10k, Resistor_SMD:R_0603_1608Metric, F.Cu at (219.5, 30.4)
- added R67: 10k, Resistor_SMD:R_0603_1608Metric, F.Cu at (231.2, 18.6)
- added R68: 10k, Resistor_SMD:R_0603_1608Metric, F.Cu at (231.6, 11.1)
- added R69: 10k, Resistor_SMD:R_0603_1608Metric, F.Cu at (203.4, 37.3)
- added R70: 10k, Resistor_SMD:R_0603_1608Metric, F.Cu at (215.2, 25.4)
- added R71: 10k, Resistor_SMD:R_0603_1608Metric, F.Cu at (235.6, 6.05)
- added R72: 10k, Resistor_SMD:R_0603_1608Metric, F.Cu at (227.6, 13.6)
- added R73: 10k, Resistor_SMD:R_0603_1608Metric, F.Cu at (242.9, -1.48)
- added R74: 10k, Resistor_SMD:R_0603_1608Metric, F.Cu at (211.5, 27.9)
- added R75: 10k, Resistor_SMD:R_0603_1608Metric, F.Cu at (219.2, 22.9)
- added R76: 10k, Resistor_SMD:R_0603_1608Metric, F.Cu at (211.5, 30.4)
- added R77: 4,7k, Resistor_SMD:R_0603_1608Metric, F.Cu at (207.4, 34.8)
- added R78: 4,7k, Resistor_SMD:R_0603_1608Metric, F.Cu at (223.2, 17.9)
- added R79: 4,7k, Resistor_SMD:R_0603_1608Metric, F.Cu at (239.6, 8.56)
- added R80: 4,7k, Resistor_SMD:R_0603_1608Metric, F.Cu at (242.9, 1.03)
- added R81: 4,7k, Resistor_SMD:R_0603_1608Metric, F.Cu at (215.5, 27.9)
- added R82: 4,7k, Resistor_SMD:R_0603_1608Metric, F.Cu at (227.6, 16.1)
- added R83: 4,7k, Resistor_SMD:R_0603_1608Metric, F.Cu at (203.4, 39.8)
- added R84: 4,7k, Resistor_SMD:R_0603_1608Metric, F.Cu at (223.2, 20.4)
- added R85: 4,7k, Resistor_SMD:R_0603_1608Metric, F.Cu at (235.6, 8.56)
- added R86: 4,7k, Resistor_SMD:R_0603_1608Metric, F.Cu at (207.4, 37.3)
- added R87: 4,7k, Resistor_SMD:R_0603_1608Metric, F.Cu at (234.9, 3.54)
- added R88: 4,7k, Resistor_SMD:R_0603_1608Metric, F.Cu at (223.6, 12.9)
- added R89: 4,7k, Resistor_SMD:R_0603_1608Metric, F.Cu at (242.9, -3.99)
- added R90: 4,7k, Resistor_SMD:R_0603_1608Metric, F.Cu at (215.5, 38.0)
- added R91: 4,7k, Resistor_SMD:R_0603_1608Metric, F.Cu at (239.6, 13.6)
- added R92: 4,7k, Resistor_SMD:R_0603_1608Metric, F.Cu at (223.5, 30.4)
- added R93: 10k, Resistor_SMD:R_0603_1608Metric, F.Cu at (235.2, 18.6)
- added R94: 10k, Resistor_SMD:R_0603_1608Metric, F.Cu at (243.6, 11.1)
- added R95: 10k, Resistor_SMD:R_0603_1608Metric, F.Cu at (239.6, 16.1)
- added R96: 10k, Resistor_SMD:R_0603_1608Metric, F.Cu at (211.5, 35.5)
- added R97: 10k, Resistor_SMD:R_0603_1608Metric, F.Cu at (219.2, 25.4)
- added R98: 10k, Resistor_SMD:R_0603_1608Metric, F.Cu at (239.6, 6.05)
- added R99: 10k, Resistor_SMD:R_0603_1608Metric, F.Cu at (219.5, 33.0)
- R1, R10, R11, R12, R13, R14, R18, R19, R20, R21, R22, R40, R41, R43, R44, R45, R46, R47, R48, R49, R5, R50, R55, R56, R57, R58, R59, R6, R60, R7, R8, R9: value 10k -> 4,7k
- U1, U10, U11, U12, U13, U14, U2, U3, U4, U5, U6, U7, U8: value EL357N-G -> TLP290-4; footprint Package_SO:OPTO_EL357N-G -> Package_SO:SOP-16_4.55x10.3mm_P1.27mm
- moved C33 245.2 mm to (243.6, 6.05)
- moved R35 236.8 mm to (234.9, 1.03)
- moved R28 223.0 mm to (238.9, -3.99), turned to 0 degrees
- moved C32 222.9 mm to (223.2, 25.4)
- moved R40 219.0 mm to (226.8, -1.48)
- moved C30 210.2 mm to (227.2, 21.1), turned to 0 degrees
- moved R29 209.4 mm to (223.6, 7.86), turned to 0 degrees
- moved R32 208.1 mm to (219.6, 15.4), turned to 0 degrees
- moved R38 206.2 mm to (215.2, 20.4)
- moved C26 201.2 mm to (230.8, 1.03), turned to 0 degrees
- moved C31 200.9 mm to (215.5, 33.0), turned to 0 degrees
- moved R39 199.7 mm to (211.2, 17.9)
- moved R34 198.8 mm to (203.4, 32.3)
- moved C34 198.5 mm to (211.5, 38.0)
- moved R49 197.7 mm to (238.9, -1.48)
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Connections:
- C1 pad 1: Net-(C1-Pad1) -> P8.46
- C1 pad 2: P8.46_OUT -> GND
- C11 pad 1: Net-(C11-Pad1) -> P8.37
- C11 pad 2: P8.42_OUT -> GND
- C12 pad 1: Net-(C12-Pad1) -> P8.33
- C12 pad 2: P8.41_OUT -> GND
- C13 pad 1: Net-(C13-Pad1) -> P8.40
- C13 pad 2: P8.40_OUT -> GND
- C14 pad 1: Net-(C14-Pad1) -> P8.36
- C14 pad 2: P8.39_OUT -> GND
- C15 pad 1: Net-(C15-Pad1) -> P8.32
- C15 pad 2: P9.21_OUT -> GND
- C16 pad 1: Net-(C16-Pad1) -> P8.39
- C16 pad 2: P9.22_OUT -> GND
- C19 pad 1: Net-(C19-Pad1) -> P8.35
- C19 pad 2: P8.38_OUT -> GND
- C2 pad 1: Net-(C2-Pad1) -> P8.45
- C2 pad 2: P8.45_OUT -> GND
- C20 pad 1: Net-(C20-Pad1) -> P8.31
- C20 pad 2: P8.37_OUT -> GND
- C21 pad 1: Net-(C21-Pad1) -> P8.30
- C21 pad 2: P8.36_OUT -> GND
- C22 pad 1: Net-(C22-Pad1) -> P8.26
- C22 pad 2: P8.35_OUT -> GND
- C23 pad 1: Net-(C23-Pad1) -> P8.15
- C23 pad 2: P8.34_OUT -> GND
- C24 pad 1: Net-(C24-Pad1) -> P8.10
- C24 pad 2: P8.33_OUT -> GND
- C25 pad 1: Net-(C25-Pad1) -> P8.29
- C25 pad 2: P8.32_OUT -> GND
- C26 pad 1: Net-(C26-Pad1) -> P8.18
- C26 pad 2: P8.31_OUT -> GND
- C27 pad 1: Net-(C27-Pad1) -> P8.14
- C27 pad 2: P8.30_OUT -> GND
- C28 pad 1: Net-(C28-Pad1) -> P8.09
- C28 pad 2: P8.29_OUT -> GND
- C29 pad 1: Net-(C29-Pad1) -> P8.28
- C29 pad 2: P8.28_OUT -> GND
- C3 pad 1: Net-(C3-Pad1) -> P8.43
- C3 pad 2: P8.44_OUT -> GND
- C30 pad 1: Net-(C30-Pad1) -> P8.17
- C30 pad 2: P8.27_OUT -> GND
- C31 pad 1: Net-(C31-Pad1) -> P8.12
- C31 pad 2: P8.26_OUT -> GND
- C32 pad 1: Net-(C32-Pad1) -> P8.08
- C32 pad 2: P9.16_OUT -> GND
- C33 pad 1: Net-(C33-Pad1) -> P8.27
- C33 pad 2: P9.17_OUT -> GND
- C34 pad 1: Net-(C34-Pad1) -> P8.16
- C34 pad 2: P9.18_OUT -> GND
- C35 pad 1: Net-(C35-Pad1) -> P8.11
- C35 pad 2: P9.11_OUT -> GND
- C36 pad 1: Net-(C36-Pad1) -> P8.07
- C36 pad 2: P9.12_OUT -> GND
- C37 pad 1: Net-(C37-Pad1) -> P9.11
- C37 pad 2: P9.13_OUT -> GND
- C38 pad 1: Net-(C38-Pad1) -> P9.15
- C38 pad 2: P8.18_OUT -> GND
- C39 pad 1: Net-(C39-Pad1) -> P9.21
- C39 pad 2: P8.17_OUT -> GND
- C4 pad 1: Net-(C4-Pad1) -> P8.44
- C4 pad 2: P8.43_OUT -> GND
- C40 pad 1: Net-(C40-Pad1) -> P9.25
- C40 pad 2: P8.16_OUT -> GND
- C41 pad 1: Net-(C41-Pad1) -> P9.12
- C41 pad 2: P8.15_OUT -> GND
- C42 pad 1: Net-(C42-Pad1) -> P9.16
- C42 pad 2: P8.14_OUT -> GND
- C43 pad 1: Net-(C43-Pad1) -> P9.22
- C43 pad 2: P8.12_OUT -> GND
- C44 pad 1: Net-(C44-Pad1) -> P9.26
- C44 pad 2: P8.11_OUT -> GND
- C45 pad 1: Net-(C45-Pad1) -> P9.13
- C45 pad 2: P8.10_OUT -> GND
- C46 pad 1: Net-(C46-Pad1) -> P9.17
- C46 pad 2: P8.09_OUT -> GND
- C49 pad 1: Net-(C49-Pad1) -> P9.23
- C49 pad 2: P9.27_OUT -> GND
- C5 pad 1: Net-(C5-Pad1) -> P8.42
- C5 pad 2: P8.08_OUT -> GND
- C50 pad 1: Net-(C50-Pad1) -> P9.27
- C50 pad 2: P9.26_OUT -> GND
- C51 pad 1: Net-(C51-Pad1) -> P9.14
- C51 pad 2: P9.25_OUT -> GND
- C52 pad 1: Net-(C52-Pad1) -> P9.18
- C52 pad 2: P9.24_OUT -> GND
- C53 pad 1: Net-(C53-Pad1) -> P9.24
- C53 pad 2: P9.23_OUT -> GND
- C54 pad 1: Net-(C54-Pad1) -> P9.28
- C54 pad 2: P9.42_OUT -> GND
- C55 pad 1: Net-(C55-Pad1) -> P9.29
- C55 pad 2: P9.31_OUT -> GND
- C56 pad 1: Net-(C56-Pad1) -> P9.30
- C56 pad 2: P9.30_OUT -> GND
- C57 pad 1: Net-(C57-Pad1) -> P9.31
- C57 pad 2: P9.29_OUT -> GND
- C58 pad 1: Net-(C58-Pad1) -> P9.42
- C58 pad 2: P9.28_OUT -> GND
- C6 pad 1: Net-(C6-Pad1) -> P8.38
- C6 pad 2: P8.07_OUT -> GND
- C7 pad 1: Net-(C7-Pad1) -> P8.34
- C7 pad 2: P9.14_OUT -> GND
- C8 pad 1: Net-(C8-Pad1) -> P8.41
- C8 pad 2: P9.15_OUT -> GND
- J1 pad 1: GNDA -> VDD
- J13 pad 1: GND -> VDD
- J2 pad 1: GNDA -> VDD
- J3 pad 1: GNDA -> VDD
- J4 pad 1: GNDA -> VDD
- J5 pad 1: GNDA -> VDD
- J6 pad 1: GNDA -> VDD
- J8 pad 1: GND -> VDD
- R1 pad 1: Net-(C1-Pad1) -> Net-(R1-Pad1)
- R1 pad 2: +24VA -> GNDA
- R10 pad 1: Net-(C12-Pad1) -> Net-(R10-Pad1)
- R10 pad 2: +24VA -> GNDA
- R11 pad 1: Net-(C13-Pad1) -> Net-(R11-Pad1)
- R11 pad 2: +24VA -> GNDA
- R12 pad 1: Net-(C14-Pad1) -> Net-(R12-Pad1)
- R12 pad 2: +24VA -> GNDA
- R13 pad 1: Net-(C15-Pad1) -> Net-(R13-Pad1)
- R13 pad 2: +24VA -> GNDA
- R14 pad 1: Net-(C16-Pad1) -> Net-(R14-Pad1)
- R14 pad 2: +24VA -> GNDA
- R18 pad 1: Net-(C19-Pad1) -> Net-(R18-Pad1)
- R18 pad 2: +24VA -> GNDA
- R19 pad 1: Net-(C20-Pad1) -> Net-(R19-Pad1)
- R19 pad 2: +24VA -> GNDA
- R2 pad 1: Net-(C2-Pad1) -> P8.46
- R2 pad 2: +24VA -> +3V3
- R20 pad 1: Net-(C21-Pad1) -> Net-(R20-Pad1)
- R20 pad 2: +24VA -> GNDA
- R21 pad 1: Net-(C22-Pad1) -> Net-(R21-Pad1)
- R21 pad 2: +24VA -> GNDA
- R22 pad 1: Net-(C23-Pad1) -> Net-(R22-Pad1)
- R22 pad 2: +24VA -> GNDA
- R23 pad 1: Net-(C24-Pad1) -> P8.42
- R23 pad 2: +24VA -> +3V3
- R24 pad 1: Net-(C25-Pad1) -> P8.38
- R24 pad 2: +24VA -> +3V3
- R25 pad 1: Net-(C26-Pad1) -> P8.34
- R25 pad 2: +24VA -> +3V3
- R26 pad 1: Net-(C27-Pad1) -> P8.41
- R26 pad 2: +24VA -> +3V3
- R27 pad 1: Net-(C28-Pad1) -> P8.37
- R27 pad 2: +24VA -> +3V3
- R28 pad 1: Net-(C29-Pad1) -> P8.33
- R28 pad 2: +24VA -> +3V3
- R29 pad 1: Net-(C30-Pad1) -> P8.40
- R29 pad 2: +24VA -> +3V3
- R3 pad 1: Net-(C3-Pad1) -> P8.45
- R3 pad 2: +24VA -> +3V3
- R32 pad 1: Net-(C31-Pad1) -> P8.36
- R32 pad 2: +24VA -> +3V3
- R33 pad 1: Net-(C32-Pad1) -> P8.32
- R33 pad 2: +24VA -> +3V3
- R34 pad 1: Net-(C33-Pad1) -> P8.43
- R34 pad 2: +24VA -> +3V3
- R35 pad 1: Net-(C34-Pad1) -> P8.39
- R35 pad 2: +24VA -> +3V3
- R38 pad 1: Net-(C35-Pad1) -> P8.35
- R38 pad 2: +24VA -> +3V3
- R39 pad 1: Net-(C36-Pad1) -> P8.31
- R39 pad 2: +24VA -> +3V3
- R4 pad 1: Net-(C4-Pad1) -> P8.44
- R4 pad 2: +24VA -> +3V3
- R40 pad 1: Net-(C37-Pad1) -> Net-(R40-Pad1)
- R40 pad 2: +24VA -> GNDA
- R41 pad 1: Net-(C38-Pad1) -> Net-(R41-Pad1)
- R41 pad 2: +24VA -> GNDA
- R43 pad 1: Net-(C39-Pad1) -> Net-(R43-Pad1)
- R43 pad 2: +24VA -> GNDA
- R44 pad 1: Net-(C40-Pad1) -> Net-(R44-Pad1)
- R44 pad 2: +24VA -> GNDA
- R45 pad 1: Net-(C41-Pad1) -> Net-(R45-Pad1)
- R45 pad 2: +24VA -> GNDA
- R46 pad 1: Net-(C42-Pad1) -> Net-(R46-Pad1)
- R46 pad 2: +24VA -> GNDA
- R47 pad 1: Net-(C43-Pad1) -> Net-(R47-Pad1)
- R47 pad 2: +24VA -> GNDA
- R48 pad 1: Net-(C44-Pad1) -> Net-(R48-Pad1)
- R48 pad 2: +24VA -> GNDA
- R49 pad 1: Net-(C45-Pad1) -> Net-(R49-Pad1)
- R49 pad 2: +24VA -> GNDA
- R5 pad 1: Net-(C5-Pad1) -> Net-(R5-Pad1)
- R5 pad 2: +24VA -> GNDA
- R50 pad 1: Net-(C46-Pad1) -> Net-(R50-Pad1)
- R50 pad 2: +24VA -> GNDA
- R55 pad 1: Net-(C49-Pad1) -> Net-(R55-Pad1)
- R55 pad 2: +24VA -> GNDA
- R56 pad 1: Net-(C50-Pad1) -> Net-(R56-Pad1)
- R56 pad 2: +24VA -> GNDA
- R57 pad 1: Net-(C51-Pad1) -> Net-(R57-Pad1)
- R57 pad 2: +24VA -> GNDA
- R58 pad 1: Net-(C52-Pad1) -> Net-(R58-Pad1)
- R58 pad 2: +24VA -> GNDA
- R59 pad 1: Net-(C53-Pad1) -> Net-(R59-Pad1)
- R59 pad 2: +24VA -> GNDA
- R6 pad 1: Net-(C6-Pad1) -> Net-(R6-Pad1)
- R6 pad 2: +24VA -> GNDA
- R60 pad 1: Net-(C54-Pad1) -> Net-(R60-Pad1)
- R60 pad 2: +24VA -> GNDA
- R61 pad 1: Net-(C55-Pad1) -> P8.30
- R61 pad 2: +24VA -> +3V3
- R62 pad 1: Net-(C56-Pad1) -> P8.26
- R62 pad 2: +24VA -> +3V3
- R63 pad 1: Net-(C57-Pad1) -> P8.15
- R63 pad 2: +24VA -> +3V3
- R64 pad 1: Net-(C58-Pad1) -> P8.10
- R64 pad 2: +24VA -> +3V3
- R7 pad 1: Net-(C7-Pad1) -> Net-(R7-Pad1)
- R7 pad 2: +24VA -> GNDA
- R8 pad 1: Net-(C8-Pad1) -> Net-(R8-Pad1)
- R8 pad 2: +24VA -> GNDA
- R9 pad 1: Net-(C11-Pad1) -> Net-(R9-Pad1)
- R9 pad 2: +24VA -> GNDA
- U1 pad 1: Net-(C1-Pad1) -> P8.43_OUT
- U1 pad 2: P8.46_OUT -> Net-(R1-Pad1)
- U1 pad 3: GND -> P8.44_OUT
- U1 pad 4: P8.46 -> Net-(R5-Pad1)
- U10 pad 1: Net-(C11-Pad1) -> P9.11_OUT
- U10 pad 2: P8.42_OUT -> Net-(R77-Pad1)
- U10 pad 3: GND -> P9.12_OUT
- U10 pad 4: P8.42 -> Net-(R78-Pad1)
- U11 pad 1: Net-(C12-Pad1) -> P9.15_OUT
- U11 pad 2: P8.41_OUT -> Net-(R81-Pad1)
- U11 pad 3: GND -> P9.16_OUT
- U11 pad 4: P8.41 -> Net-(R82-Pad1)
- U12 pad 1: Net-(C13-Pad1) -> P9.21_OUT
- U12 pad 2: P8.40_OUT -> Net-(R85-Pad1)
- U12 pad 3: GND -> P9.22_OUT
- U12 pad 4: P8.40 -> Net-(R86-Pad1)
- U13 pad 1: Net-(C14-Pad1) -> P9.25_OUT
- U13 pad 2: P8.39_OUT -> Net-(R89-Pad1)
- U13 pad 3: GND -> P9.26_OUT
- U13 pad 4: P8.39 -> Net-(R90-Pad1)
- U14 pad 1: Net-(C15-Pad1) -> P9.29_OUT
- U14 pad 2: P9.21_OUT -> Net-(R109-Pad1)
- U14 pad 3: GND -> P9.30_OUT
- U14 pad 4: P9.21 -> Net-(R110-Pad1)
- U2 pad 1: Net-(C2-Pad1) -> P8.42_OUT
- U2 pad 2: P8.45_OUT -> Net-(R8-Pad1)
- U2 pad 3: GND -> P8.41_OUT
- U2 pad 4: P8.45 -> Net-(R9-Pad1)
- U3 pad 1: Net-(C3-Pad1) -> P8.38_OUT
- U3 pad 2: P8.44_OUT -> Net-(R12-Pad1)
- U3 pad 3: GND -> P8.37_OUT
- U3 pad 4: P8.44 -> Net-(R13-Pad1)
- U4 pad 1: Net-(C4-Pad1) -> P8.34_OUT
- U4 pad 2: P8.43_OUT -> Net-(R19-Pad1)
- U4 pad 3: GND -> P8.33_OUT
- U4 pad 4: P8.43 -> Net-(R20-Pad1)
- U5 pad 1: Net-(C5-Pad1) -> P8.30_OUT
- U5 pad 2: P8.08_OUT -> Net-(R40-Pad1)
- U5 pad 3: GND -> P8.29_OUT
- U5 pad 4: P8.08 -> Net-(R41-Pad1)
- U6 pad 1: Net-(C6-Pad1) -> P8.26_OUT
- U6 pad 2: P8.07_OUT -> Net-(R45-Pad1)
- U6 pad 3: GND -> P8.18_OUT
- U6 pad 4: P8.07 -> Net-(R46-Pad1)
- U7 pad 1: Net-(C7-Pad1) -> P8.15_OUT
- U7 pad 2: P9.14_OUT -> Net-(R49-Pad1)
- U7 pad 3: GND -> P8.14_OUT
- U7 pad 4: P9.14 -> Net-(R50-Pad1)
- U8 pad 1: Net-(C8-Pad1) -> P8.10_OUT
- U8 pad 2: P9.15_OUT -> Net-(R57-Pad1)
- U8 pad 3: GND -> P8.09_OUT
- U8 pad 4: P9.15 -> Net-(R58-Pad1)
Routing:
- removed copper zone on B.Cu, net GND
- removed copper zone on F.Cu, net GND
- removed copper zone on B.Cu, net GNDA
- removed copper zone on F.Cu, net GNDA
Other:
- outline, holes or cut-outs redrawn
- board text removed: "+1.8V"
- board text removed: "AGND"
- board text removed: "P8.27"
- board text removed: "P8.28"
- board text removed: "P8.29"
- board text removed: "P8.30"
- board text removed: "P8.31"
- board text removed: "P8.32"
- board text removed: "P8.33"
- board text removed: "P8.34"
- board text removed: "P8.35"
- board text removed: "P8.36"
- board text removed: "P8.37"
- board text removed: "P8.38"
- board text removed: "P8.39"
- board text removed: "P8.40"
- board text removed: "P8.41"
- board text removed: "P8.42"
- board text removed: "P8.43"
- board text removed: "P8.44"
- board text removed: "P8.45"
- board text removed: "P8.46"
