File: Circuit/boneIO - input board/boneIO_input board_v0.2.kicad_pcb (KiCad board)
At the start: 2 copper layers, 256 x 74 mm, 225 parts, among them J1 Screw_Terminal_01x08, J10 BeagleBone_Black_Header, J11 BeagleBone_Black_Header, J12 Conn_02x04_Odd_Even, J13 Screw_Terminal_01x04, J14 ZW_VCC, J15 ZW_GND, J16 INNY ZASILACZ, J2 Screw_Terminal_01x08, J3 Screw_Terminal_01x08, J4 Screw_Terminal_01x08, J5 Screw_Terminal_01x08, J6 Screw_Terminal_01x08, J7 Screw_Terminal_01x08, J8 Screw_Terminal_01x08, J9 Screw_Terminal_01x08, SW1 SW_Push, U1 TLP290-4, U10 TLP290-4, U11 TLP290-4, U12 TLP290-4, U13 TLP290-4, U14 TLP290-4, U2 TLP290-4, U28 RS485, U3 TLP290-4, U33 DS1307Z+, U4 TLP290-4, U46 P82B96, U5 TLP290-4, U6 TLP290-4, U7 TLP290-4, U8 TLP290-4, U9 LM2596S-ADJ, Y1 32,788 MHz

Commit message: 04.11.2021
Parts:
- removed the D2 at (174.6, 81.7)
- removed the R16 at (157.7, 99.4)
- added G***: LOGO, Symbol:boneIO_LOGO_srednie, F.Cu at (123.6, 91.0)
- moved R73 243.5 mm to (15.6, 86.0), turned to 270 degrees
- moved C33 240.5 mm to (15.6, 82.5), turned to 90 degrees
- moved R65 232.7 mm to (21.2, 86.0), turned to 270 degrees
- moved R61 231.0 mm to (24.0, 86.0), turned to 270 degrees
- moved R82 229.9 mm to (18.4, 111.5), turned to 270 degrees
- moved R44 223.4 mm to (15.3, 69.3), turned to 90 degrees
- moved R41 222.2 mm to (21.1, 69.3), turned to 90 degrees
- moved R47 219.7 mm to (38.9, 111.6), turned to 270 degrees
- moved R49 219.1 mm to (51.2, 111.6), turned to 270 degrees
- moved R84 219.1 mm to (24.0, 111.6), turned to 270 degrees
- moved R81 216.6 mm to (15.7, 111.5), turned to 270 degrees
- moved R40 214.9 mm to (23.9, 69.3), turned to 90 degrees
- moved R45 208.1 mm to (33.3, 111.6), turned to 270 degrees
- moved C30 208.1 mm to (422.6, 92.7)
- moved C36 208.1 mm to (378.8, 103.2)
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Connections:
- C1 pad 1: P8.46 -> P8.45
- C11 pad 1: P8.37 -> P8.36
- C12 pad 1: P8.33 -> P8.32
- C13 pad 1: P8.40 -> P8.39
- C14 pad 1: P8.36 -> P8.35
- C15 pad 1: P8.32 -> P8.31
- C16 pad 1: P8.39 -> P8.38
- C19 pad 1: P8.35 -> P8.34
- C2 pad 1: P8.45 -> P8.44
- C20 pad 1: P8.31 -> P8.30
- C21 pad 1: P8.30 -> P8.29
- C22 pad 1: P8.26 -> P9.15
- C23 pad 1: P8.15 -> P8.16
- C24 pad 1: P8.10 -> P8.11
- C25 pad 1: P8.29 -> P8.28
- C26 pad 1: P8.18 -> P9.16
- C27 pad 1: P8.14 -> P8.15
- C28 pad 1: P8.09 -> P8.10
- C29 pad 1: P8.28 -> P8.27
- C3 pad 1: P8.43 -> P8.42
- C30 pad 1: P8.17 -> P8.18
- C31 pad 1: P8.12 -> P8.14
- C32 pad 1: P8.08 -> P8.09
- C33 pad 1: P8.27 -> P8.26
- C34 pad 1: P8.16 -> P8.17
- C35 pad 1: P8.11 -> P8.12
- C36 pad 1: P8.07 -> P8.08
- C37 pad 1: P9.11 -> P9.28
- C38 pad 1: P9.15 -> P9.11
- C39 pad 1: P9.21 -> P9.29
- C4 pad 1: P8.44 -> P8.43
- C40 pad 1: P9.25 -> P9.24
- C41 pad 1: P9.12 -> P9.27
- C42 pad 1: P9.16 -> P9.12
- C43 pad 1: P9.22 -> P9.18
- C44 pad 1: P9.26 -> P9.23
- C45 pad 1: P9.13 -> P9.26
- C46 pad 1: P9.17 -> P9.13
- C49 pad 1: P9.23 -> P9.21
- C5 pad 1: P8.42 -> P8.41
- C50 pad 1: P9.27 -> P9.17
- C51 pad 1: P9.14 -> P9.25
- C52 pad 1: P9.18 -> P9.14
- C53 pad 1: P9.24 -> P9.22
- C54 pad 1: P9.28 -> P9.46
- C55 pad 1: P9.29 -> P8.07
- C56 pad 1: P9.30 -> P9.42
- C58 pad 1: P9.42 -> P9.30
- C6 pad 1: P8.38 -> P8.37
- C7 pad 1: P8.34 -> P8.33
- C8 pad 1: P8.41 -> P8.40
- J15 pad 3: GNDD -> GND1
- J16 pad 1: GNDD -> GND1
- R100 pad 1: P9.26 -> P9.23
- R101 pad 1: P9.13 -> P9.26
- R102 pad 1: P9.17 -> P9.13
- R103 pad 1: P9.23 -> P9.21
- R104 pad 1: P9.27 -> P9.17
- R105 pad 1: P9.14 -> P9.25
- R106 pad 1: P9.18 -> P9.14
- R107 pad 1: P9.24 -> P9.22
- R108 pad 1: P9.28 -> P9.46
- R113 pad 1: P9.29 -> P8.07
- R114 pad 1: P9.30 -> P9.42
- R116 pad 1: P9.42 -> P9.30
- R2 pad 1: P8.46 -> P8.45
- R23 pad 1: P8.42 -> P8.41
- R24 pad 1: P8.38 -> P8.37
- R25 pad 1: P8.34 -> P8.33
- R26 pad 1: P8.41 -> P8.40
- R27 pad 1: P8.37 -> P8.36
- R28 pad 1: P8.33 -> P8.32
- R29 pad 1: P8.40 -> P8.39
- R3 pad 1: P8.45 -> P8.44
- R32 pad 1: P8.36 -> P8.35
- R33 pad 1: P8.32 -> P8.31
- R34 pad 1: P8.43 -> P8.42
- R35 pad 1: P8.39 -> P8.38
- R38 pad 1: P8.35 -> P8.34
- R39 pad 1: P8.31 -> P8.30
- R4 pad 1: P8.44 -> P8.43
- R61 pad 1: P8.30 -> P8.29
- R62 pad 1: P8.26 -> P9.15
- R63 pad 1: P8.15 -> P8.16
- R64 pad 1: P8.10 -> P8.11
- R65 pad 1: P8.29 -> P8.28
- R66 pad 1: P8.18 -> P9.16
- R67 pad 1: P8.14 -> P8.15
- R68 pad 1: P8.09 -> P8.10
- R69 pad 1: P8.28 -> P8.27
- R70 pad 1: P8.17 -> P8.18
- R71 pad 1: P8.12 -> P8.14
- R72 pad 1: P8.08 -> P8.09
- R73 pad 1: P8.27 -> P8.26
- R74 pad 1: P8.16 -> P8.17
- R75 pad 1: P8.11 -> P8.12
- R76 pad 1: P8.07 -> P8.08
- R93 pad 1: P9.11 -> P9.28
- R94 pad 1: P9.15 -> P9.11
- R95 pad 1: P9.21 -> P9.29
- R96 pad 1: P9.25 -> P9.24
- R97 pad 1: P9.12 -> P9.27
- R98 pad 1: P9.16 -> P9.12
- R99 pad 1: P9.22 -> P9.18
- U1 pad 1: P8.43_OUT -> P8.45_OUT
- U1 pad 10: P8.43 -> P8.42
- U1 pad 12: P8.44 -> P8.43
- U1 pad 14: P8.45 -> P8.44
- U1 pad 16: P8.46 -> P8.45
- U1 pad 5: P8.45_OUT -> P8.43_OUT
- U1 pad 7: P8.46_OUT -> P8.42_OUT
- U10 pad 1: P9.11_OUT -> P9.28_OUT
- U10 pad 10: P9.14 -> P9.25
- U10 pad 12: P9.13 -> P9.26
- U10 pad 14: P9.12 -> P9.27
- U10 pad 16: P9.11 -> P9.28
- U10 pad 3: P9.12_OUT -> P9.27_OUT
- U10 pad 5: P9.13_OUT -> P9.26_OUT
- U10 pad 7: P9.14_OUT -> P9.25_OUT
- U11 pad 1: P9.15_OUT -> P9.11_OUT
- U11 pad 10: P9.18 -> P9.14
- U11 pad 12: P9.17 -> P9.13
- U11 pad 14: P9.16 -> P9.12
- U11 pad 16: P9.15 -> P9.11
- U11 pad 3: P9.16_OUT -> P9.12_OUT
- U11 pad 5: P9.17_OUT -> P9.13_OUT
- U11 pad 7: P9.18_OUT -> P9.14_OUT
- U12 pad 1: P9.21_OUT -> P9.29_OUT
- U12 pad 10: P9.24 -> P9.22
- U12 pad 12: P9.23 -> P9.21
- U12 pad 14: P9.22 -> P9.18
- U12 pad 16: P9.21 -> P9.29
- U12 pad 3: P9.22_OUT -> P9.18_OUT
- U12 pad 5: P9.23_OUT -> P9.21_OUT
- U12 pad 7: P9.24_OUT -> P9.22_OUT
- U13 pad 1: P9.25_OUT -> P9.24_OUT
- U13 pad 10: P9.28 -> P9.46
- U13 pad 12: P9.27 -> P9.17
- U13 pad 14: P9.26 -> P9.23
- U13 pad 16: P9.25 -> P9.24
- U13 pad 3: P9.26_OUT -> P9.23_OUT
- U13 pad 5: P9.27_OUT -> P9.17_OUT
- U13 pad 7: P9.28_OUT -> P8.46_OUT
- U14 pad 1: P9.29_OUT -> P8.07_OUT
- U14 pad 10: P9.42 -> P9.30
- U14 pad 14: P9.30 -> P9.42
- U14 pad 16: P9.29 -> P8.07
- U14 pad 3: P9.30_OUT -> P9.42_OUT
- U14 pad 7: P9.42_OUT -> P9.30_OUT
- U2 pad 1: P8.42_OUT -> P8.41_OUT
- U2 pad 10: P8.39 -> P8.38
- U2 pad 12: P8.40 -> P8.39
- U2 pad 14: P8.41 -> P8.40
- U2 pad 16: P8.42 -> P8.41
- U2 pad 3: P8.41_OUT -> P8.40_OUT
- U2 pad 5: P8.40_OUT -> P8.39_OUT
- U2 pad 7: P8.39_OUT -> P8.38_OUT
- U3 pad 1: P8.38_OUT -> P8.37_OUT
- U3 pad 10: P8.35 -> P8.34
- U3 pad 12: P8.36 -> P8.35
- U3 pad 14: P8.37 -> P8.36
- U3 pad 16: P8.38 -> P8.37
- U3 pad 3: P8.37_OUT -> P8.36_OUT
- U3 pad 5: P8.36_OUT -> P8.35_OUT
- U3 pad 7: P8.35_OUT -> P8.34_OUT
- U4 pad 1: P8.34_OUT -> P8.33_OUT
- U4 pad 10: P8.31 -> P8.30
- U4 pad 12: P8.32 -> P8.31
- U4 pad 14: P8.33 -> P8.32
- U4 pad 16: P8.34 -> P8.33
- U4 pad 3: P8.33_OUT -> P8.32_OUT
- U4 pad 5: P8.32_OUT -> P8.31_OUT
- U4 pad 7: P8.31_OUT -> P8.30_OUT
- U5 pad 1: P8.30_OUT -> P8.29_OUT
- U5 pad 10: P8.27 -> P8.26
- U5 pad 12: P8.28 -> P8.27
- U5 pad 14: P8.29 -> P8.28
- U5 pad 16: P8.30 -> P8.29
- U5 pad 3: P8.29_OUT -> P8.28_OUT
- U5 pad 5: P8.28_OUT -> P8.27_OUT
- U5 pad 7: P8.27_OUT -> P8.26_OUT
- U6 pad 1: P8.26_OUT -> P9.15_OUT
- U6 pad 10: P8.16 -> P8.17
- U6 pad 12: P8.17 -> P8.18
- U6 pad 14: P8.18 -> P9.16
- U6 pad 16: P8.26 -> P9.15
- U6 pad 3: P8.18_OUT -> P9.16_OUT
- U6 pad 5: P8.17_OUT -> P8.18_OUT
- U6 pad 7: P8.16_OUT -> P8.17_OUT
- U7 pad 1: P8.15_OUT -> P8.16_OUT
- U7 pad 10: P8.11 -> P8.12
- U7 pad 12: P8.12 -> P8.14
- U7 pad 14: P8.14 -> P8.15
- U7 pad 16: P8.15 -> P8.16
- U7 pad 3: P8.14_OUT -> P8.15_OUT
- U7 pad 5: P8.12_OUT -> P8.14_OUT
- U7 pad 7: P8.11_OUT -> P8.12_OUT
- U8 pad 1: P8.10_OUT -> P8.11_OUT
- U8 pad 10: P8.07 -> P8.08
- U8 pad 12: P8.08 -> P8.09
- U8 pad 14: P8.09 -> P8.10
- U8 pad 16: P8.10 -> P8.11
- U8 pad 3: P8.09_OUT -> P8.10_OUT
- U8 pad 5: P8.08_OUT -> P8.09_OUT
- U8 pad 7: P8.07_OUT -> P8.08_OUT
Routing:
- net VDD: track 0.00 -> 427.8 mm
- net Earth: track 0.00 -> 54.4 mm, vias 0 -> 66
- net P8.41_OUT: track 0.00 -> 38.5 mm
- net P8.44_OUT: track 0.00 -> 37.0 mm
- net P8.40_OUT: track 0.00 -> 36.1 mm
- net P8.43_OUT: track 0.00 -> 35.9 mm
- net +24V: track 0.00 -> 35.3 mm
- net P8.42_OUT: track 0.00 -> 33.7 mm
- net P8.37_OUT: track 0.00 -> 27.2 mm
- net P8.36_OUT: track 0.00 -> 25.4 mm
- net P8.39_OUT: track 0.00 -> 25.2 mm
- net P8.33_OUT: track 0.00 -> 25.1 mm
- net P8.35_OUT: track 0.00 -> 22.9 mm
- net P8.38_OUT: track 0.00 -> 22.4 mm
- net P8.34_OUT: track 0.00 -> 20.9 mm
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Other:
- board text added: "I2C"
- board text added: "input board BBB v0.2"
- board text removed: "1.Dołożyć Drganie styków na Switch 2. Poprawić poligony GND"
- board text removed: "P8.03"
- board text removed: "P8.04"
- board text removed: "P8.05"
- board text removed: "P8.06"
- board text removed: "P8.07"
- board text removed: "P8.08"
- board text removed: "P8.09"
- board text removed: "P8.10"
- board text removed: "P8.11"
- board text removed: "P8.12"
- board text removed: "P8.14"
- board text removed: "P8.15"
- board text removed: "P8.16"
- board text removed: "P8.17"
- board text removed: "P8.18"
- board text removed: "P8.20"
- board text removed: "P8.21"
- board text removed: "P8.22"
- board text removed: "P8.23"
- board text removed: "P8.24"
- board text removed: "P8.25"
- board text removed: "P8.26"
- board text removed: "input board v0.2"

Commit message: Update boneIO_input board_v0.2.kicad_pcb
zmiany 05/11
Parts:
- moved R28 402.6 mm to (32.2, 87.8), turned to 270 degrees
- moved R35 381.6 mm to (49.0, 87.9), turned to 270 degrees
- moved R39 380.0 mm to (26.6, 87.9), turned to 270 degrees
- moved R32 374.4 mm to (40.5, 87.9), turned to 270 degrees
- moved R23 373.3 mm to (57.4, 87.9), turned to 270 degrees
- moved R38 372.8 mm to (37.8, 87.9), turned to 270 degrees
- moved R26 371.9 mm to (54.5, 87.9), turned to 270 degrees
- moved C19 369.2 mm to (37.8, 84.4), turned to 90 degrees
- moved R29 367.3 mm to (51.8, 87.9), turned to 270 degrees
- moved R33 366.0 mm to (29.4, 87.9), turned to 270 degrees
- moved C11 359.3 mm to (43.3, 84.4), turned to 90 degrees
- moved C6 356.9 mm to (46.1, 84.4), turned to 90 degrees
- moved R104 356.7 mm to (74.3, 88.0), turned to 270 degrees
- moved R24 356.6 mm to (46.1, 87.9), turned to 270 degrees
- moved C54 351.0 mm to (71.4, 84.5), turned to 90 degrees
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Routing:
- net P8.41_OUT: track 38.5 -> 0.00 mm
- net P8.44_OUT: track 37.0 -> 0.00 mm
- net P8.43_OUT: track 35.9 -> 0.00 mm
- net P8.40_OUT: track 36.1 -> 0.22 mm
- net P8.42_OUT: track 33.7 -> 0.00 mm
- net P8.37_OUT: track 27.2 -> 0.00 mm
- net P8.36_OUT: track 25.4 -> 0.00 mm
- net P8.39_OUT: track 25.2 -> 0.00 mm
- net P8.33_OUT: track 25.1 -> 0.00 mm
- net P8.35_OUT: track 22.9 -> 0.00 mm
- net P8.38_OUT: track 22.4 -> 0.00 mm
- net P8.34_OUT: track 20.9 -> 0.00 mm
- net P8.32_OUT: track 14.4 -> 0.00 mm
- net P8.29_OUT: track 13.3 -> 0.00 mm
- net P8.31_OUT: track 11.8 -> 0.00 mm
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
Commit message: 06/11/21
Parts:
- moved R89 419.9 mm to (19.2, 92.6), turned to 90 degrees
- moved R94 413.3 mm to (22.0, 92.6), turned to 90 degrees
- moved R99 397.8 mm to (24.8, 92.6), turned to 90 degrees
- moved C27 393.8 mm to (33.1, 96.1), turned to 270 degrees
- moved C40 388.1 mm to (19.2, 96.2), turned to 270 degrees
- moved C31 386.7 mm to (35.9, 96.1), turned to 270 degrees
- moved R64 384.2 mm to (47.1, 92.6), turned to 90 degrees
- moved R60 382.3 mm to (44.4, 92.6), turned to 90 degrees
- moved R59 381.9 mm to (33.1, 92.6), turned to 90 degrees
- moved R103 379.5 mm to (27.6, 92.6), turned to 90 degrees
- moved C48 378.5 mm to (24.8, 96.2), turned to 270 degrees
- moved C44 376.5 mm to (22.0, 96.2), turned to 270 degrees
- moved R63 374.7 mm to (35.9, 92.6), turned to 90 degrees
- moved R57 374.5 mm to (52.7, 92.6), turned to 90 degrees
- moved R56 373.0 mm to (41.6, 92.6), turned to 90 degrees
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- renumbered C47 to C1, C11 to C10, C12 to C11, C4 to C12, C3 to C16, C16 to C17, C19 to C18, C20 to C19, C9 to C2, C17 to C20, C18 to C21, C21 to C22, C22 to C23, C23 to C24, C24 to C25, C25 to C26, C26 to C27, C27 to C28, C28 to C29, C10 to C3, C29 to C30, C30 to C31, C31 to C32, C32 to C33, C33 to C34, C34 to C35, C35 to C36, C36 to C37, C48 to C38, C37 to C39, C1 to C4, C38 to C40, C39 to C41, C40 to C42, C41 to C43, C42 to C44, C43 to C45, C44 to C46, C45 to C47, C46 to C48, C2 to C8, C8 to C9, D4 to D2, D2 to D3, D3 to D4, J12 to J1, J13 to J10, J7 to J11, J10 to J12, J14 to J13, J15 to J14, J11 to J15, J9 to J2, J1 to J3, J2 to J4, J3 to J5, J4 to J6, J5 to J7, J6 to J8, J8 to J9, R13 to R10, R103 to R100, R104 to R101, R105 to R102, R106 to R103, R107 to R104, R108 to R105, R36 to R106, R37 to R107, R109 to R108, R110 to R109, R14 to R11, R111 to R110, R112 to R111, R42 to R112, R18 to R12, R19 to R13, R20 to R14, R21 to R15, R22 to R16, R51 to R17, R2 to R18, R23 to R19, R5 to R2, R24 to R20, R25 to R21, R3 to R22, R26 to R23, R27 to R24, R28 to R25, R52 to R26, R4 to R27, R29 to R28, R32 to R29, R6 to R3, R33 to R30, R34 to R31, R35 to R32, R38 to R33, R39 to R34, R15 to R35, R16 to R36, R17 to R37, R40 to R38, R41 to R39, R7 to R4, R43 to R40, R44 to R41, R45 to R42, R46 to R43, R47 to R44, R48 to R45, R49 to R46, R50 to R47, R55 to R48, R56 to R49, R8 to R5, R57 to R50, R58 to R51, R59 to R52, R60 to R53, R61 to R54, R62 to R55, R63 to R56, R64 to R57, R65 to R58, R66 to R59, R9 to R6, R67 to R60, R68 to R61, R69 to R62, R70 to R63, R71 to R64, R72 to R65, R73 to R66, R74 to R67, R75 to R68, R76 to R69, R10 to R7, R53 to R70, R54 to R71, R77 to R72, R78 to R73, R79 to R74, R80 to R75, R81 to R76, R82 to R77, R83 to R78, R84 to R79, R11 to R8, R85 to R80, R86 to R81, R87 to R82, R88 to R83, R89 to R84, R90 to R85, R91 to R86, R92 to R87, R93 to R88, R94 to R89, R12 to R9, R95 to R90, R96 to R91, R30 to R92, R97 to R93, R98 to R94, R99 to R95, R100 to R96, R31 to R97, R101 to R98, R102 to R99, U46 to U1, U7 to U10, U8 to U11, U10 to U12, U11 to U13, U12 to U14, U13 to U15, U33 to U16, U14 to U17, U1 to U2, U2 to U3, U3 to U4, U4 to U5, U9 to U6, U28 to U7, U5 to U8, U6 to U9
Routing:
- net +5V: track 0.00 -> 169.5 mm
- net +3V3: track 0.00 -> 142.1 mm
- net P9.22_OUT: track 0.00 -> 58.2 mm, vias 0 -> 1
- net P9.21_OUT: track 0.00 -> 56.3 mm, vias 0 -> 1
- net P9.18_OUT: track 0.00 -> 53.8 mm, vias 0 -> 1
- net P9.28_OUT: track 0.00 -> 52.6 mm, vias 0 -> 1
- net P9.24_OUT: track 0.00 -> 51.4 mm, vias 0 -> 1
- net P9.27_OUT: track 0.00 -> 51.0 mm, vias 0 -> 1
- net P9.26_OUT: track 0.00 -> 49.0 mm, vias 0 -> 1
- net P9.23_OUT: track 0.00 -> 48.3 mm, vias 0 -> 1
- net P9.30_OUT: track 0.00 -> 47.4 mm, vias 0 -> 1
- net P9.17_OUT: track 0.00 -> 46.6 mm, vias 0 -> 1
- net P9.25_OUT: track 0.00 -> 46.6 mm, vias 0 -> 1
- net P9.31_OUT: track 0.00 -> 45.7 mm, vias 0 -> 1
- net P8.08_OUT: track 0.00 -> 45.6 mm, vias 0 -> 1
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
Commit message: a
Routing:
- net P8.11: track 1.95 -> 23.1 mm, vias 0 -> 2
- net P8.09: track 1.95 -> 23.1 mm, vias 0 -> 2
- net P8.10: track 1.95 -> 22.8 mm, vias 0 -> 2
- net P8.08: track 1.95 -> 21.8 mm, vias 0 -> 2
- net P8.12: track 1.92 -> 15.9 mm, vias 0 -> 2
- net P8.14: track 1.92 -> 15.8 mm, vias 0 -> 2
- net P8.16: track 1.94 -> 15.4 mm, vias 0 -> 2
- net P8.15: track 1.92 -> 15.2 mm, vias 0 -> 2
- net P9.14: track 1.92 -> 11.0 mm, vias 0 -> 2
- net P9.13: track 1.92 -> 11.0 mm, vias 0 -> 2
- net P9.12: track 1.92 -> 10.8 mm, vias 0 -> 2
- net P9.11: track 1.95 -> 10.7 mm, vias 0 -> 2
- net P9.15: track 1.91 -> 10.3 mm, vias 0 -> 2
- net P9.16: track 1.90 -> 10.1 mm, vias 0 -> 2
- net P8.18: track 1.90 -> 10.0 mm, vias 0 -> 2
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