File: Circuit/boneIO - input board/boneIO_input board_v0.3.kicad_pcb (KiCad board)
At the start: 2 copper layers, 256 x 74 mm, 263 parts, among them J1 Screw_Terminal_01x08, J10 Screw_Terminal_01x08, J11 Screw_Terminal_01x08, J12 ZW_VCC, J13 ZW_GND, J14 INNY ZASILACZ, J15 BeagleBone_Black_Header, J16 BeagleBone_Black_Header, J2 Screw_Terminal_01x08, J3 Screw_Terminal_01x08, J4 Screw_Terminal_01x08, J5 Screw_Terminal_01x08, J6 Screw_Terminal_01x08, J7 Screw_Terminal_01x08, J8 Screw_Terminal_01x04, J9 Conn_02x04_Odd_Even, SW1 SW_Push, U1 P82B96, U10 LM2596S-ADJ, U11 RS485, U12 PC817X2NIP0F, U13 PC817X2NIP0F, U14 PC817X2NIP0F, U15 PC817X2NIP0F, U16 PC817X2NIP0F, U17 PC817X2NIP0F, U18 PC817X2NIP0F, U19 PC817X2NIP0F, U2 PC817X2NIP0F, U20 PC817X2NIP0F, U21 PC817X2NIP0F, U22 PC817X2NIP0F, U23 PC817X2NIP0F, U24 PC817X2NIP0F, U25 PC817X2NIP0F, U26 PC817X2NIP0F, U27 PC817X2NIP0F, U28 PC817X2NIP0F, U29 PC817X2NIP0F, U3 PC817X2NIP0F, U30 PC817X2NIP0F, U31 PC817X2NIP0F, U32 PC817X2NIP0F, U33 PC817X2NIP0F, U34 PC817X2NIP0F, U35 PC817X2NIP0F, U36 DS1307Z+, U37 PC817X2NIP0F, U38 PC817X2NIP0F, U39 PC817X2NIP0F, U4 PC817X2NIP0F, U40 PC817X2NIP0F, U41 PC817X2NIP0F, U42 PC817X2NIP0F, U43 PC817X2NIP0F, U44 PC817X2NIP0F, U45 PC817X2NIP0F, U46 PC817X2NIP0F, U47 PC817X2NIP0F, U48 PC817X2NIP0F, U49 PC817X2NIP0F, U5 PC817X2NIP0F, U50 PC817X2NIP0F, U51 PC817X2NIP0F, U52 PC817X2NIP0F, U53 PC817X2NIP0F, U54 PC817X2NIP0F, U55 PC817X2NIP0F, U56 PC817X2NIP0F, U6 PC817X2NIP0F, U7 PC817X2NIP0F, U8 PC817X2NIP0F, U9 PC817X2NIP0F, Y1 32,788 MHz

Commit message: update PCB
Parts:
- moved U56 39.5 mm to (136.0, 99.6)
- moved C58 39.5 mm to (137.6, 91.2)
- moved R112 39.5 mm to (135.2, 106.5)
- moved R116 39.5 mm to (134.7, 91.2)
- moved C36 5.66 mm to (98.0, 91.2)
- moved C57 5.66 mm to (126.3, 91.2)
- moved R111 5.66 mm to (124.1, 106.4)
- moved R114 5.66 mm to (117.7, 91.2)
- moved R115 5.66 mm to (123.4, 91.2)
- moved R63 5.66 mm to (95.9, 106.5)
- moved R64 5.66 mm to (101.6, 106.5)
- moved R65 5.66 mm to (107.0, 106.4)
- moved U35 5.66 mm to (107.7, 99.6)
- moved C37 5.66 mm to (103.6, 91.2)
- moved C38 5.66 mm to (109.3, 91.2)
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Connections:
- C42 pad 1: P9,25 -> P9.25
- J6 pad 7: P9.30_OUT -> P9.29_OUT
- J6 pad 8: P9.29_OUT -> P9.30_OUT
- R88 pad 1: P9,25 -> P9.25
- REF** pad 1: (no net) -> Earth
- REF** pad 2: (no net) -> +5V
- REF** pad 4: (no net) -> Earth
- U40 pad 4: P9,25 -> P9.25
Routing:
- net +3V3: track 0.00 -> 666.0 mm
- net +5V: track 0.00 -> 215.6 mm
- net P8.08: track 6.31 -> 156.7 mm, vias 0 -> 2
- net VDD_ADC: track 0.00 -> 150.3 mm
- net P8.09: track 6.25 -> 153.8 mm, vias 0 -> 2
- net GND_ADC: track 0.00 -> 145.1 mm
- net P8.10: track 6.23 -> 145.1 mm, vias 0 -> 2
- net P8.11: track 6.22 -> 143.3 mm, vias 0 -> 2
- net P8.12: track 6.25 -> 134.8 mm, vias 0 -> 2
- net P9.41: track 0.00 -> 55.9 mm, vias 0 -> 1
- net P9.33: track 0.00 -> 45.8 mm
- net P9.36: track 0.00 -> 38.0 mm
- net TX: track 0.00 -> 35.9 mm
- net Earth: track 0.00 -> 34.9 mm, vias 0 -> 1
- net P9.35: track 0.00 -> 33.4 mm
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- added copper zone on B.Cu, net Earth
- removed copper zone on B.Cu, net (none)

Commit message: update PCB 08/11/21
Parts:
- moved R81 161.3 mm to (176.7, 60.1), turned to 180 degrees
- moved U41 156.4 mm to (175.9, 67.0), turned to 270 degrees
- moved R89 156.2 mm to (177.1, 75.4), turned to 270 degrees
- moved C43 150.6 mm to (174.3, 75.4), turned to 270 degrees
- moved R82 150.5 mm to (171.0, 60.1), turned to 180 degrees
- moved U42 145.3 mm to (170.2, 67.0), turned to 270 degrees
- moved R90 145.0 mm to (171.5, 75.4), turned to 270 degrees
- moved R83 139.7 mm to (165.3, 60.1), turned to 180 degrees
- moved C44 139.3 mm to (168.6, 75.4), turned to 270 degrees
- moved U43 134.3 mm to (164.6, 67.0), turned to 270 degrees
- moved R91 133.7 mm to (165.8, 75.4), turned to 270 degrees
- moved R84 129.0 mm to (159.6, 60.1), turned to 180 degrees
- moved C45 128.1 mm to (163.0, 75.4), turned to 270 degrees
- moved U44 123.4 mm to (158.9, 67.0), turned to 270 degrees
- moved R92 122.6 mm to (160.2, 75.4), turned to 270 degrees
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Connections:
- C41 pad 1: P9.26 -> P8.19
- C51 pad 1: P9.24 -> P8.13
- C55 pad 1: P9.07 -> P8.07
- J1 pad 2: P8.39_OUT -> P9.29_OUT
- J1 pad 3: P8.38_OUT -> P9.30_OUT
- J1 pad 4: P8.37_OUT -> P9.31_OUT
- J1 pad 5: P8.36_OUT -> P9.42_OUT
- J1 pad 6: P8.35_OUT -> P8.46_OUT
- J1 pad 7: P8.34_OUT -> P8.45_OUT
- J1 pad 8: P8.33_OUT -> P8.44_OUT
- J11 pad 8: Net-(J11-Pad8) -> GND
- J2 pad 2: P9.11_OUT -> P8.36_OUT
- J2 pad 3: P9.12_OUT -> P8.35_OUT
- J2 pad 4: P9.13_OUT -> P8.34_OUT
- J2 pad 5: P9.14_OUT -> P8.33_OUT
- J2 pad 6: P9.15_OUT -> P8.32_OUT
- J2 pad 7: P9.16_OUT -> P8.31_OUT
- J2 pad 8: P8.18_OUT -> P8.30_OUT
- J3 pad 2: P8.32_OUT -> P8.43_OUT
- J3 pad 3: P8.31_OUT -> P8.42_OUT
- J3 pad 4: P8.30_OUT -> P8.41_OUT
- J3 pad 5: P8.29_OUT -> P8.40_OUT
- J3 pad 6: P8.28_OUT -> P8.39_OUT
- J3 pad 7: P8.27_OUT -> P8.38_OUT
- J3 pad 8: P8.26_OUT -> P8.37_OUT
- J4 pad 2: P8.17_OUT -> P8.29_OUT
- J4 pad 3: P8.16_OUT -> P8.28_OUT
- J4 pad 4: P8.15_OUT -> P8.27_OUT
- J4 pad 5: P8.14_OUT -> P8.26_OUT
- J4 pad 6: P8.12_OUT -> P8.19_OUT
- J4 pad 7: P8.11_OUT -> P8.18_OUT
- J4 pad 8: P8.10_OUT -> P8.17_OUT
- J5 pad 2: P8.46_OUT -> P9.18_OUT
- J5 pad 3: P8.45_OUT -> P9.21_OUT
- J5 pad 4: P8.44_OUT -> P9.22_OUT
- J5 pad 5: P8.43_OUT -> P9.23_OUT
- J5 pad 6: P8.42_OUT -> P9.25_OUT
- J5 pad 7: P8.41_OUT -> P9.27_OUT
- J5 pad 8: P8.40_OUT -> P9.28_OUT
- J6 pad 2: P8.09_OUT -> P8.16_OUT
- J6 pad 3: P8.08_OUT -> P8.15_OUT
- J6 pad 4: P8.07_OUT -> P8.14_OUT
- J6 pad 5: P9.42_OUT -> P8.13_OUT
- J6 pad 6: P9.31_OUT -> P8.12_OUT
- J6 pad 7: P9.29_OUT -> P8.11_OUT
- J6 pad 8: P9.30_OUT -> P8.10_OUT
- J7 pad 2: P9.28_OUT -> P9.11_OUT
- J7 pad 3: P9.27_OUT -> P9.12_OUT
- J7 pad 4: P9.26_OUT -> P9.13_OUT
- J7 pad 5: P9.25_OUT -> P9.14_OUT
- J7 pad 6: P9.24_OUT -> P9.15_OUT
- J7 pad 7: P9.23_OUT -> P9.16_OUT
- J8 pad 2: P9.18_OUT -> P8.09_OUT
- J8 pad 3: P9.21_OUT -> P8.08_OUT
- J8 pad 4: P9.22_OUT -> P8.07_OUT
- R105 pad 1: P9.24 -> P8.13
- R113 pad 1: P9.07 -> P8.07
- R87 pad 1: P9.26 -> P8.19
- U26 pad 2: P8.18_OUT -> P8.14_OUT
- U27 pad 2: P8.17_OUT -> P8.15_OUT
- U29 pad 2: P8.15_OUT -> P8.18_OUT
- U30 pad 2: P8.14_OUT -> P8.17_OUT
- U31 pad 2: P8.12_OUT -> P8.08_OUT
- U32 pad 2: P8.11_OUT -> P8.09_OUT
- U34 pad 2: P8.09_OUT -> P8.11_OUT
- U35 pad 2: P8.08_OUT -> P8.12_OUT
- U39 pad 2: P9.26_OUT -> P8.19_OUT
- U39 pad 4: P9.26 -> P8.19
- U49 pad 2: P9.24_OUT -> P8.13_OUT
- U49 pad 4: P9.24 -> P8.13
- U53 pad 4: P9.07 -> P8.07
Routing:
- net P9.11: track 288.3 -> 6.21 mm, vias 1 -> 0
- net P9.12: track 284.2 -> 6.21 mm, vias 1 -> 0
- net P9.13: track 282.2 -> 6.21 mm, vias 1 -> 0
- net P9.14: track 276.2 -> 6.17 mm, vias 1 -> 0
- net P9.15: track 276.4 -> 6.64 mm, vias 1 -> 0
- net P9.16: track 271.0 -> 6.62 mm, vias 1 -> 0
- net P8.14: track 209.1 -> 6.25 mm, vias 1 -> 0
- net P8.27: track 208.1 -> 6.16 mm, vias 1 -> 0
- net P8.15: track 207.5 -> 6.83 mm, vias 1 -> 0
- net P8.26: track 205.9 -> 6.18 mm, vias 1 -> 0
- net P8.16: track 199.1 -> 6.19 mm, vias 1 -> 0
- net P8.28: track 198.9 -> 6.00 mm, vias 1 -> 0
- net P8.18: track 196.4 -> 6.19 mm, vias 1 -> 0
- net P8.29: track 195.4 -> 6.18 mm, vias 1 -> 0
- net P8.17: track 194.9 -> 6.17 mm, vias 1 -> 0
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- added copper zone on B.Cu, net GND
- added copper zone on F.Cu, net GND

Commit message: PCB board to be checked
Parts:
- renumbered VDD1 to +24V
Connections:
- REF** pad 3: (no net) -> +24V
Routing:
- net P8.36: track 6.18 -> 246.0 mm, vias 0 -> 2
- net P8.35: track 6.23 -> 243.6 mm, vias 0 -> 2
- net P9.42: track 6.30 -> 242.4 mm, vias 0 -> 2
- net P8.34: track 6.33 -> 235.3 mm, vias 0 -> 2
- net P8.33: track 6.08 -> 231.2 mm, vias 0 -> 2
- net P9.31: track 6.25 -> 227.9 mm, vias 0 -> 1
- net P8.32: track 6.21 -> 221.9 mm, vias 0 -> 2
- net P8.31: track 6.23 -> 219.0 mm, vias 0 -> 2
- net P9.30: track 6.25 -> 214.2 mm, vias 0 -> 1
- net P8.37: track 6.82 -> 211.8 mm, vias 0 -> 2
- net P8.30: track 6.13 -> 208.5 mm, vias 0 -> 2
- net P9.29: track 6.25 -> 208.2 mm, vias 0 -> 1
- net P8.29: track 6.18 -> 207.6 mm, vias 0 -> 2
- net P8.38: track 6.44 -> 204.6 mm, vias 0 -> 2
- net P8.39: track 6.09 -> 202.7 mm, vias 0 -> 2
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Other:
- board text added: "+12-48V"
- board text added: "GNDA"

Commit message: update PCB
Parts:
- moved J15 2.13 mm to (272.6, 107.1)
- moved J16 2.13 mm to (224.3, 107.2)
- moved SW1 1.02 mm to (258.3, 81.1)
- moved R64 0.48 mm to (129.5, 106.5)
- moved R63 0.39 mm to (135.1, 106.5)
- moved I2C1 0.38 mm to (232.5, 69.4)
- moved R62 0.35 mm to (140.7, 106.5)
- moved R100 0.34 mm to (74.9, 60.1)
- moved R97 0.32 mm to (118.2, 106.5)
- moved R61 0.31 mm to (146.4, 106.5)
- moved R46 0.29 mm to (112.6, 106.5)
- moved R93 0.28 mm to (97.5, 60.1)
- moved R47 0.27 mm to (106.9, 106.5)
- moved R60 0.27 mm to (95.6, 106.5)
- moved R43 0.22 mm to (78.7, 106.5)
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Routing:
- net P8.14: track 140.3 -> 199.5 mm
- net P9.18: track 154.1 -> 201.3 mm
- net P8.13: track 156.7 -> 193.1 mm
- net P8.07: track 104.2 -> 134.5 mm
- net P8.43: track 184.5 -> 200.6 mm
- net P8.15: track 149.8 -> 157.8 mm
- net Earth: track 54.6 -> 61.5 mm, vias 105 -> 121
- net P8.45: track 176.2 -> 182.2 mm
- net P8.46: track 168.4 -> 173.1 mm
- net P8.40: track 194.9 -> 198.6 mm
- net P9.36: track 38.0 -> 35.0 mm
- net P9.39: track 12.4 -> 9.44 mm
- net P9.27: track 189.5 -> 186.8 mm
- net SCL: track 237.1 -> 239.6 mm
- net VDD_ADC: track 146.8 -> 149.2 mm
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
Commit message: update
zmiany w rozmieszczeniu BBB i dodane Gerbery, BOM i P&P
Parts:
- added JP1: 5V, Jumper:SolderJumper-2_P1.3mm_Open_Pad1.0x1.5mm, F.Cu at (169.2, 94.9)
- D1: value B340A-13F -> SS34
- R29: value 1k -> 1.2k
- moved J13 6.65 mm to (210.3, 63.0), turned to 270 degrees
- moved J12 6.35 mm to (201.7, 63.0)
- moved J15 1.46 mm to (273.1, 105.8)
- moved J16 1.46 mm to (224.8, 105.8)
- moved R29 1.29 mm to (164.9, 95.4)
- moved J10 0.54 mm to (229.9, 113.7)
- moved J11 0.43 mm to (265.4, 52.9)
- renumbered +24V to VDD1
Connections:
- J11 pad 8: GND -> Net-(J11-Pad8)
Routing:
- net P9.28: track 192.3 -> 223.2 mm
- net P9.25: track 187.1 -> 180.0 mm
- net GNDA: track 31.8 -> 38.5 mm
- net P8.14: track 199.5 -> 193.2 mm
- net P8.18: track 163.2 -> 169.4 mm
- net P9.12: track 147.7 -> 142.2 mm
- net SCL: track 239.6 -> 244.8 mm
- net P9.13: track 151.8 -> 147.0 mm
- net P9.11: track 149.1 -> 144.4 mm
- net +48V: track 5.58 -> 10.0 mm
- net SDA: track 223.3 -> 227.8 mm
- net P8.30: track 209.7 -> 214.1 mm
- net P8.31: track 220.1 -> 224.3 mm
- net P9.14: track 150.0 -> 145.9 mm
- net P9.42: track 243.7 -> 247.8 mm
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Other:
- board text added: "+48V"
- board text removed: "+12-48V"
