File: Circuit/boneIO - input board/boneIO_input board.sch (KiCad schematic (older format))
At the start: 262 parts, among them J1 Screw_Terminal_01x08, J10 Screw_Terminal_01x08, J11 Screw_Terminal_01x08, J12 ZW_VCC, J13 ZW_GND, J14 INNY ZASILACZ, J15 BeagleBone_Black_Header, J16 BeagleBone_Black_Header, J2 Screw_Terminal_01x08, J3 Screw_Terminal_01x08, J4 Screw_Terminal_01x08, J5 Screw_Terminal_01x08, J6 Screw_Terminal_01x08, J7 Screw_Terminal_01x08, J8 Screw_Terminal_01x04, J9 Conn_02x04_Odd_Even, SW1 SW_Push, U1 P82B96, U10 LM2596S-ADJ, U11 RS485, U12 PC817X2NIP0F, U13 PC817X2NIP0F, U14 PC817X2NIP0F, U15 PC817X2NIP0F, U16 PC817X2NIP0F, U17 PC817X2NIP0F, U18 PC817X2NIP0F, U19 PC817X2NIP0F, U2 PC817X2NIP0F, U20 PC817X2NIP0F, U21 PC817X2NIP0F, U22 PC817X2NIP0F, U23 PC817X2NIP0F, U24 PC817X2NIP0F, U25 PC817X2NIP0F, U26 PC817X2NIP0F, U27 PC817X2NIP0F, U28 PC817X2NIP0F, U29 PC817X2NIP0F, U3 PC817X2NIP0F, U30 PC817X2NIP0F, U31 PC817X2NIP0F, U32 PC817X2NIP0F, U33 PC817X2NIP0F, U34 PC817X2NIP0F, U35 PC817X2NIP0F, U36 DS1307Z+, U37 PC817X2NIP0F, U38 PC817X2NIP0F, U39 PC817X2NIP0F, U4 PC817X2NIP0F, U40 PC817X2NIP0F, U41 PC817X2NIP0F, U42 PC817X2NIP0F, U43 PC817X2NIP0F, U44 PC817X2NIP0F, U45 PC817X2NIP0F, U46 PC817X2NIP0F, U47 PC817X2NIP0F, U48 PC817X2NIP0F, U49 PC817X2NIP0F, U5 PC817X2NIP0F, U50 PC817X2NIP0F, U51 PC817X2NIP0F, U52 PC817X2NIP0F, U53 PC817X2NIP0F, U54 PC817X2NIP0F, U55 PC817X2NIP0F, U56 PC817X2NIP0F, U6 PC817X2NIP0F, U7 PC817X2NIP0F, U8 PC817X2NIP0F, U9 PC817X2NIP0F, Y1 32,788 MHz

Commit message: renaming and cleaning files
Parts:
- J15, J16: symbol boneIO_input-board_v0.3-rescue:BeagleBone_Black_Header-Connector_Generic -> boneIO_input-board-rescue:BeagleBone_Black_Header-Connector_Generic-boneIO_input-board_v0.3-rescue-boneIO_input-board-r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
- U11: symbol boneIO_input-board_v0.3-rescue:RS485-RF_Module -> boneIO_input-board-rescue:RS485-RF_Module-boneIO_input-board_v0.3-rescue-boneIO_input-board-rescue
Changed lines of the file:
@@
 P8.07_OUT
 $Comp
-L boneIO_input-board_v0.3-rescue:RS485-RF_Module U11
+L boneIO_input-board-rescue:RS485-RF_Module-boneIO_input-board_v0.3-rescue-boneIO_input-board-rescue U11
 U 1 1 6187A9D0
 P 28250 9450
@@
 P8.39_OUT
 $Comp
-L boneIO_input-board_v0.3-rescue:BeagleBone_Black_Header-Connector_Generic J15
+L boneIO_input-board-rescue:BeagleBone_Black_Header-Connector_Generic-boneIO_input-board_v0.3-rescue-boneIO_input-board-rescue J15
 U 1 1 64765995
 P 27000 6200
@@
 $EndComp
 $Comp
-L boneIO_input-board_v0.3-rescue:BeagleBone_Black_Header-Connector_Generic J16
+L boneIO_input-board-rescue:BeagleBone_Black_Header-Connector_Generic-boneIO_input-board_v0.3-rescue-boneIO_input-board-rescue J16
 U 1 1 643393F0
 P 29000 6200

Commit message: fixed PCB errors and added descriptions on the schematic
Other:
- moved on the sheet: ANVDD1, BT1, C1, C10, C11, C12, C13, C14, C15, C16, C17, C18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

Commit message: cleanup to finish 0.2
Parts:
- BT1: footprint Battery:Battery_Panasonic_CR1220-VCN_Vertical_CircularHoles -> boneIO:Battery_Panasonic_CR1220-VCN_Vertical_CircularHoles
- J15, J16: symbol boneIO_input-board-rescue:BeagleBone_Black_Header-Connector_Generic-boneIO_input-board_v0.3-rescue-boneIO_input-board-r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 -> boneIO:BeagleBone_Black_Header-Connector_Generic-boneIO_input-board_v0.3-rescue-boneIO_input-board-rescue
- U11: symbol boneIO_input-board-rescue:RS485-RF_Module-boneIO_input-board_v0.3-rescue-boneIO_input-board-rescue -> boneIO:RS485-RF_Module-boneIO_input-board_v0.3-rescue-boneIO_input-board-rescue
Changed lines of the file:
@@
 F 0 "BT1" V 15895 5150 50  0000 C CNN
 F 1 "Battery" V 15804 5150 50  0000 C CNN
-F 2 "Battery:Battery_Panasonic_CR1220-VCN_Vertical_CircularHoles" V 15650 5210 50  0001 C CNN
+F 2 "boneIO:Battery_Panasonic_CR1220-VCN_Vertical_CircularHoles" V 15650 5210 50  0001 C CNN
 F 3 "~" V 15650 5210 50  0001 C CNN
 	1    15650 5150
@@
 P8.07_OUT
 $Comp
-L boneIO_input-board-rescue:RS485-RF_Module-boneIO_input-board_v0.3-rescue-boneIO_input-board-rescue U11
+L boneIO:RS485-RF_Module-boneIO_input-board_v0.3-rescue-boneIO_input-board-rescue U11
 U 1 1 6187A9D0
 P 28300 9450
@@
 P8.39_OUT
 $Comp
-L boneIO_input-board-rescue:BeagleBone_Black_Header-Connector_Generic-boneIO_input-board_v0.3-rescue-boneIO_input-board-rescue J15
+L boneIO:BeagleBone_Black_Header-Connector_Generic-boneIO_input-board_v0.3-rescue-boneIO_input-board-rescue J15
 U 1 1 64765995
 P 27050 6200
@@
 $EndComp
 $Comp
-L boneIO_input-board-rescue:BeagleBone_Black_Header-Connector_Generic-boneIO_input-board_v0.3-rescue-boneIO_input-board-rescue J16
+L boneIO:BeagleBone_Black_Header-Connector_Generic-boneIO_input-board_v0.3-rescue-boneIO_input-board-rescue J16
 U 1 1 643393F0
 P 29050 6200
