File: Circuit/boneIO - ssr board/boneIO - ssr board.sch (KiCad schematic (older format))
At the start: 55 parts, among them J1 Screw_Terminal_01x04, J10 Screw_Terminal_01x04, J11 Screw_Terminal_01x04, J2 Screw_Terminal_01x04, J3 Conn_02x13_Odd_Even, J4 Screw_Terminal_01x04, J5 Screw_Terminal_01x04, J6 Screw_Terminal_01x04, J7 Screw_Terminal_01x04, J8 Screw_Terminal_01x04, J9 Screw_Terminal_01x04, U1 MCP9808_MSOP, U2 ULN2803A, U3 ULN2803A, U4 ULN2803A, U5 ULN2803A

Commit message: Finished schema for SSR board
Parts:
- removed R1, R2, R3, R4, R5, R6: 0k, Resistor_SMD:R_0603_1608Metric, symbol boneIO---ssr-board-rescue:R-Device
- added C1, C?: 100nF, symbol Device:C
- added K1, K2, K3, K? (x27): HF46F, HF46F, symbol HF46F:HF46F
- added R? (x9): 10k, Resistor_SMD:R_0603_1608Metric, symbol boneIO---ssr-board-rescue:R-Device
- added SW1, SW2, SW3: SW_DIP_x03, symbol Switch:SW_DIP_x03
- added U6, U7: MCP23017_SS, Package_SO:SSOP-28_5.3x10.2mm_P0.65mm, symbol Interface_Expansion:MCP23017_SS
- renumbered J11 to J10, J3 to J11, J4 to J3, J5 to J4, J6 to J5, J7 to J6, J8 to J7, J9 to J8, J10 to J9
Connections:
- net +24V: now also K1.1, K2.1, K3.1, K?.1, K?.1, K?.1, K?.1, K?.1, K?.1, K?.1, K?.1, K?.1, K?.1, K?.1, K?.1, K?.1, K?.1, K?.1, K?.1, K?.1, K?.1, K?.1, K?.1, K?.1, K?.1, K?.1, K?.1, K?.1, K?.1, K?.1
- net +3V3: now also C1.2, C?.2, SW1.1, SW1.2, SW1.3, SW2.1, SW2.2, SW2.3, SW3.1, SW3.2, SW3.3, U6.9 (VDD), U7.9 (VDD)
- net GND: now also C1.1, C?.1, R?.2, R?.2, R?.2, R?.2, R?.2, R?.2, R?.2, R?.2, R?.2, U6.10 (VSS), U7.10 (VSS)
- net RELAY1: now also K1.2
- net RELAY10: now also K?.2
- net RELAY11: now also K?.2
- net RELAY12: now also K?.2
- net RELAY13: now also K?.2
- net RELAY14: now also K?.2
- net RELAY15: now also K?.2
- net RELAY16: now also K?.2
- net RELAY17: now also K?.2
- net RELAY18: now also K?.2
- net RELAY19: now also K?.2
- net RELAY2: now also K2.2
- net RELAY20: now also K?.2
- net RELAY21: now also K?.2
- net RELAY22: now also K?.2
- net RELAY23: now also K?.2
- net RELAY24: now also K?.2
- net RELAY25: now also K?.2
- net RELAY26: now also K?.2
- net RELAY27: now also K?.2
- net RELAY28: now also K?.2
- net RELAY29: now also K?.2
- net RELAY3: now also K3.2
- net RELAY30: now also K?.2
- net RELAY4: now also K?.2
- net RELAY5: now also K?.2
- net RELAY6: now also K?.2
- net RELAY7: now also K?.2
- net RELAY8: now also K?.2
- net RELAY9: now also K?.2
- net SCL: now also U6.12 (SCK), U7.12 (SCK)
- net SDA: now also U6.13 (SDA), U7.13 (SDA)
- net at U1.5 (A2): now also R?.1, SW3.4
- net at U1.6 (A1): now also R?.1, SW3.5
- net at U1.7 (A0): now also R?.1, SW3.6
- net at J1.1 (Pin_1): now also K1.3, K2.3, K3.3
- net at J1.2 (Pin_2): now also K1.4
- net at J1.3 (Pin_3): now also K2.4
- net at J1.4 (Pin_4): now also K3.4
- net at J2.1 (Pin_1): now also K?.3, K?.3, K?.3
- net at J2.2 (Pin_2): now also K?.4
- net at J2.3 (Pin_3): now also K?.4
- net at J2.4 (Pin_4): now also K?.4
- net at J3.1 (Pin_1): now also K?.3, K?.3, K?.3
- net at J3.2 (Pin_2): now also K?.4
- net at J3.3 (Pin_3): now also K?.4
- net at J3.4 (Pin_4): now also K?.4
- net at J4.1 (Pin_1): now also K?.3, K?.3, K?.3
- net at J4.2 (Pin_2): now also K?.4
- net at J4.3 (Pin_3): now also K?.4
- net at J4.4 (Pin_4): now also K?.4
- net at J5.1 (Pin_1): now also K?.3, K?.3, K?.3
- net at J5.2 (Pin_2): now also K?.4
- net at J5.3 (Pin_3): now also K?.4
- net at J5.4 (Pin_4): now also K?.4
- net at J6.1 (Pin_1): now also K?.4
- net at J6.2 (Pin_2): now also K?.4
- net at J6.3 (Pin_3): now also K?.4
- net at J6.4 (Pin_4): now also K?.3, K?.3, K?.3
- net at J8.1 (Pin_1): now also K?.3, K?.3, K?.3
- net at J8.2 (Pin_2): now also K?.4
- net at J8.3 (Pin_3): now also K?.4
- net at J8.4 (Pin_4): now also K?.4
- net at J7.1 (Pin_1): now also K?.3, K?.3, K?.3
- net at J7.2 (Pin_2): now also K?.4
- net at J7.3 (Pin_3): now also K?.4
- net at J7.4 (Pin_4): now also K?.4
- net at J9.1 (Pin_1): now also K?.4
- net at J9.2 (Pin_2): now also K?.4
- net at J9.3 (Pin_3): now also K?.4
- net at J9.4 (Pin_4): now also K?.3, K?.3, K?.3
- net at J10.1 (Pin_1): now also K?.4
- net at J10.2 (Pin_2): now also K?.4
- net at J10.3 (Pin_3): now also K?.4
- net at J10.4 (Pin_4): now also K?.3, K?.3, K?.3
- net K1: no longer names the net of R31.1, U2.1 (I1)
- net K1: now also U6.1 (GPB0)
- net K10: no longer names the net of R30.1, U3.2 (I2)
- net K10: now also U6.22 (GPA1)
- net K11: no longer names the net of R20.1, U3.3 (I3)
- net K11: now also U6.23 (GPA2)
- net K12: no longer names the net of R18.1, U3.4 (I4)
- net K12: now also U6.24 (GPA3)
- net K13: no longer names the net of R16.1, U3.5 (I5)
- net K13: now also U6.25 (GPA4)
- net K14: no longer names the net of R14.1, U3.6 (I6)
- net K14: now also U6.26 (GPA5)
- net K15: no longer names the net of R12.1, U3.7 (I7)
- net K15: now also U6.27 (GPA6)
- net K16: no longer names the net of R29.1, U4.1 (I1)
- net K16: now also U7.1 (GPB0)
- net K17: no longer names the net of R28.1, U4.2 (I2)
- net K17: now also U7.2 (GPB1)
- net K18: no longer names the net of R27.1, U4.3 (I3)
- net K18: now also U7.3 (GPB2)
- net K19: no longer names the net of R26.1, U4.4 (I4)
- net K19: now also U7.4 (GPB3)
- net K2: no longer names the net of R21.1, U2.2 (I2)
- net K2: now also U6.2 (GPB1)
- net K20: no longer names the net of R25.1, U4.5 (I5)
- net K20: now also U7.5 (GPB4)
- net K21: no longer names the net of R24.1, U4.6 (I6)
- net K21: now also U7.6 (GPB5)
- net K22: no longer names the net of R23.1, U4.7 (I7)
- net K22: now also U7.7 (GPB6)
- net K23: no longer names the net of R22.1, U4.8 (I8)
- net K23: now also U7.8 (GPB7)
- net K24: no longer names the net of R39.1, U5.1 (I1)
- net K24: now also U7.21 (GPA0)
- net K25: no longer names the net of R38.1, U5.2 (I2)
- net K25: now also U7.22 (GPA1)
- net K26: no longer names the net of R37.1, U5.3 (I3)
- net K26: now also U7.23 (GPA2)
- net K27: no longer names the net of R36.1, U5.4 (I4)
- net K27: now also U7.24 (GPA3)
- net K28: no longer names the net of R35.1, U5.5 (I5)
- net K28: now also U7.25 (GPA4)
- net K29: no longer names the net of R34.1, U5.6 (I6)
- net K29: now also U7.26 (GPA5)
- net K3: no longer names the net of R19.1, U2.3 (I3)
- net K3: now also U6.3 (GPB2)
- net K30: no longer names the net of R33.1, U5.7 (I7)
- net K30: now also U7.27 (GPA6)
- net K4: no longer names the net of R17.1, U2.4 (I4)
- net K4: now also U6.4 (GPB3)
- net K5: no longer names the net of R15.1, U2.5 (I5)
- net K5: now also U6.5 (GPB4)
- net K6: no longer names the net of R13.1, U2.6 (I6)
- net K6: now also U6.6 (GPB5)
- net K7: no longer names the net of R11.1, U2.7 (I7)
- net K7: now also U6.7 (GPB6)
- net K8: no longer names the net of R10.1, U2.8 (I8)
- net K8: now also U6.8 (GPB7)
- net K9: no longer names the net of R32.1, U3.1 (I1)
- net K9: now also U6.21 (GPA0)
- new net: R?.1, SW1.4, U6.15 (A0)
- new net: R?.1, SW1.5, U6.16 (A1)
- new net: R?.1, SW1.6, U6.17 (A2)
- new net: R?.1, SW2.4, U7.15 (A0)
- new net: R?.1, SW2.5, U7.16 (A1)
- new net: R?.1, SW2.6, U7.17 (A2)
Other:
- note added: "MCP23017 and ULN2803A"
- note removed: "ULN2803A"
- moved on the sheet: J1, J11, J2, R10, R11, R12, R13, R14, R15, R16, R17, R18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

Commit message: Schema updates
- removed pull down resistors between mcp and uln
- added numbers for resistors and capacitors
Parts:
- removed R10, R11, R12, R13, R14, R15, R16, R17, R18, R19, R20, R21, R22, R23, R24, R25, R26, R27, R28, R29, R30, R31, R32, R33, R34, R35, R36, R37, R38, R39: 10k, Resistor_SMD:R_0603_1608Metric, symbol boneIO---ssr-board-rescue:R-Device
- gave numbers to parts that had none: 10

Commit message: Finished
Niestety przekombinowaliśmy z tymi ssr'ami i wyszła nam płytka ze zwykłymi przekaźnikami 5A - 30 sztuk. Niestety ssr'y nie zmieściły się na wysokość. Płytka w całości obsługiwana po i2c do zastosowania w module rozszerzeń lub w boneIO bezpośrednio.
Parts:
- added R13, R14: 0, Resistor_SMD:R_0603_1608Metric, symbol Device:R
- C1, C2: footprint (none) -> Capacitor_SMD:C_0603_1608Metric
- K1, K2, K3: footprint HF46F -> HF46F:HF46F
- K10, K11, K12, K13, K14, K15, K16, K17, K18, K19, K20, K21, K22, K23, K24, K25, K26, K27, K28, K29, K30, K4, K5, K6, K7, K8, K9: renamed from K?; footprint HF46F -> HF46F:HF46F
- SW1, SW2, SW3: footprint (none) -> Button_Switch_SMD:SW_DIP_SPSTx03_Slide_KingTek_DSHP03TJ_W5.25mm_P1.27mm_JPin
Connections:
- net RELAY1: now also U2.15 (O4); no longer U2.18 (O1)
- net RELAY10: now also U4.17 (O2); no longer U3.17 (O2)
- net RELAY11: now also U4.18 (O1); no longer U3.16 (O3)
- net RELAY12: now also U5.14 (O5); no longer U3.15 (O4)
- net RELAY13: now also U5.13 (O6); no longer U3.14 (O5)
- net RELAY14: now also U5.12 (O7); no longer U3.13 (O6)
- net RELAY15: now also U5.11 (O8); no longer U3.12 (O7)
- net RELAY16: now also U2.11 (O8); no longer U4.18 (O1)
- net RELAY17: now also U2.12 (O7); no longer U4.17 (O2)
- net RELAY18: now also U2.13 (O6); no longer U4.16 (O3)
- net RELAY19: now also U2.14 (O5); no longer U4.15 (O4)
- net RELAY2: now also U2.16 (O3); no longer U2.17 (O2)
- net RELAY20: now also U3.18 (O1); no longer U4.14 (O5)
- net RELAY21: now also U3.17 (O2); no longer U4.13 (O6)
- net RELAY22: now also U3.16 (O3); no longer U4.12 (O7)
- net RELAY24: now also U4.12 (O7); no longer U5.18 (O1)
- net RELAY25: now also U4.13 (O6); no longer U5.17 (O2)
- net RELAY26: now also U4.14 (O5); no longer U5.16 (O3)
- net RELAY27: now also U5.18 (O1); no longer U5.15 (O4)
- net RELAY28: now also U5.17 (O2); no longer U5.14 (O5)
- net RELAY29: now also U5.16 (O3); no longer U5.13 (O6)
- net RELAY3: now also U2.17 (O2); no longer U2.16 (O3)
- net RELAY30: now also U5.15 (O4); no longer U5.12 (O7)
- net RELAY4: now also U2.18 (O1); no longer U2.15 (O4)
- net RELAY5: now also U3.15 (O4); no longer U2.14 (O5)
- net RELAY6: now also U3.14 (O5); no longer U2.13 (O6)
- net RELAY7: now also U3.13 (O6); no longer U2.12 (O7)
- net RELAY8: now also U4.15 (O4); no longer U2.11 (O8)
- net RELAY9: now also U4.16 (O3); no longer U3.18 (O1)
- net at K16.3, K17.3, K18.3: now also J6.1 (Pin_1); no longer J6.4 (Pin_4)
- net at K16.4: now also J6.4 (Pin_4); no longer J6.3 (Pin_3)
- net at K17.4: now also J6.3 (Pin_3); no longer J6.2 (Pin_2)
- net at K18.4: now also J6.2 (Pin_2); no longer J6.1 (Pin_1)
- net at K25.3, K26.3, K27.3: now also J9.1 (Pin_1); no longer J9.4 (Pin_4)
- net at K25.4: now also J9.4 (Pin_4); no longer J9.3 (Pin_3)
- net at K26.4: now also J9.3 (Pin_3); no longer J9.2 (Pin_2)
- net at K27.4: now also J9.2 (Pin_2); no longer J9.1 (Pin_1)
- net at K28.3, K29.3, K30.3: now also J10.1 (Pin_1); no longer J10.4 (Pin_4)
- net at K28.4: now also J10.4 (Pin_4); no longer J10.3 (Pin_3)
- net at K29.4: now also J10.3 (Pin_3); no longer J10.2 (Pin_2)
- net at K30.4: now also J10.2 (Pin_2); no longer J10.1 (Pin_1)
- net at K22.4: now also J8.4 (Pin_4); no longer J8.2 (Pin_2)
- net at K24.4: now also J8.2 (Pin_2); no longer J8.4 (Pin_4)
- net at K19.4: now also J7.4 (Pin_4); no longer J7.2 (Pin_2)
- net at K21.4: now also J7.2 (Pin_2); no longer J7.4 (Pin_4)
- net at U3.11 (O8): now also R14.1
- net MCP.1: now reaches J11.3 (Pin_3)
- net MCP.1: now also R13.1
- net MCP.2: now reaches J11.4 (Pin_4)
- net MCP.2: now also R14.2
- new net: R13.2, U3.12 (O7)
Other:
- moved on the sheet: K19, K21, K22, K24
