File: Circuit/boneIO - relay board/boneIO - relay board.kicad_pcb (KiCad board)
At the start: 2 copper layers, 197 x 102 mm, 66 parts, among them J1 Screw_Terminal_01x04, J10 Screw_Terminal_01x04, J11 Screw_Terminal_01x04, J12 Screw_Terminal_01x04, J13 Screw_Terminal_01x04, J2 Screw_Terminal_01x04, J3 Conn_02x04_Odd_Even, J4 Screw_Terminal_01x04, J5 Screw_Terminal_01x04, J6 Screw_Terminal_01x04, J7 Screw_Terminal_01x04, J8 Screw_Terminal_01x04, J9 Screw_Terminal_01x04, K1 RM85-2011-35-1005, K10 RM85-2011-35-1005, K11 RM85-2011-35-1005, K12 RM85-2011-35-1005, K13 RM85-2011-35-1005, K14 RM85-2011-35-1005, K15 RM85-2011-35-1005, K16 RM85-2011-35-1005, K17 RM85-2011-35-1005, K18 RM85-2011-35-1005, K19 RM85-2011-35-1005, K2 RM85-2011-35-1005, K20 RM85-2011-35-1005, K21 RM85-2011-35-1005, K22 RM85-2011-35-1005, K23 RM85-2011-35-1005, K24 RM85-2011-35-1005, K3 RM85-2011-35-1005, K4 RM85-2011-35-1005, K5 RM85-2011-35-1005, K6 RM85-2011-35-1005, K7 RM85-2011-35-1005, K8 RM85-2011-35-1005, K9 RM85-2011-35-1005, SW1 SW_DIP_x03, SW2 SW_DIP_x03, SW3 SW_DIP_x03, U1 MCP9808_MSOP, U2 MCP23017_SS, U3 MCP23017_SS, U4 ULN2803A, U5 ULN2803A, U6 ULN2803A

Commit message: Wersja z dnia 02.11.2021
Parts:
- added JP1: Jumper_3_Open, Jumper:SolderJumper-3_P1.3mm_Open_RoundedPad1.0x1.5mm, B.Cu at (379.4, 320.1)
- added R14: 4.7k, Resistor_SMD:R_0603_1608Metric, F.Cu at (404.7, 317.9)
- moved R7 55.0 mm to (350.0, 312.4), turned to 180 degrees
Connections:
- C4 pad 1: +24V -> VCC
- C5 pad 1: +24V -> VCC
- C6 pad 1: +24V -> VCC
- K1 pad A2: +24V -> VCC
- K10 pad A2: +24V -> VCC
- K11 pad A2: +24V -> VCC
- K12 pad A2: +24V -> VCC
- K13 pad A2: +24V -> VCC
- K14 pad A2: +24V -> VCC
- K15 pad A2: +24V -> VCC
- K16 pad A2: +24V -> VCC
- K17 pad A2: +24V -> VCC
- K18 pad A2: +24V -> VCC
- K19 pad A2: +24V -> VCC
- K2 pad A2: +24V -> VCC
- K20 pad A2: +24V -> VCC
- K21 pad A2: +24V -> VCC
- K22 pad A2: +24V -> VCC
- K23 pad A2: +24V -> VCC
- K24 pad A2: +24V -> VCC
- K3 pad A2: +24V -> VCC
- K4 pad A2: +24V -> VCC
- K5 pad A2: +24V -> VCC
- K6 pad A2: +24V -> VCC
- K7 pad A2: +24V -> VCC
- K8 pad A2: +24V -> VCC
- K9 pad A2: +24V -> VCC
- R7 pad 2: RESET_MCP -> Net-(R7-Pad2)
- U2 pad 18: RESET_MCP -> Net-(R7-Pad2)
- U3 pad 18: RESET_MCP -> Net-(R14-Pad2)
- U4 pad 10: +24V -> VCC
- U5 pad 10: +24V -> VCC
- U6 pad 10: +24V -> VCC
Routing:
- net +24V: track 542.3 -> 4.40 mm
- net VCC: track 0.00 -> 537.3 mm
- net RESET_MCP: track 84.4 -> 0.00 mm, vias 2 -> 0
- net Net-(R7-Pad2): track 0.00 -> 10.9 mm
- net Net-(R14-Pad2): track 0.00 -> 8.02 mm
- net +3V3: track 203.7 -> 209.4 mm, vias 10 -> 12
- net +5V: track 0.00 -> 4.42 mm
- net K13: track 26.7 -> 30.6 mm
- net K15: track 29.8 -> 31.5 mm
- net Net-(R10-Pad1): track 17.5 -> 19.0 mm
- net Net-(R9-Pad1): track 15.2 -> 16.5 mm
- net K14: track 28.2 -> 29.3 mm
- net K22: track 99.4 -> 98.8 mm
- net GND: vias 92 -> 105

Commit message: Gotowa PCB board relay v0.2
Parts:
- JP1: value Jumper_3_Open -> SolderJumper_3_Bridged12; footprint Jumper:SolderJumper-3_P1.3mm_Open_RoundedPad1.0x1.5mm -> Jumper:SolderJumper-3_P1.3mm_Bridged12_RoundedPad1.0x1.5mm
- moved R2 64.9 mm to (389.5, 317.8)
- moved R5 59.3 mm to (392.3, 317.8)
- moved R6 1.17 mm to (457.2, 317.6)
- moved JP1 0.05 mm to (379.4, 320.2)
Routing:
- net Net-(J12-Pad1): track 24.2 -> 48.5 mm
- net Net-(J7-Pad3): track 24.2 -> 48.5 mm
- net Net-(J7-Pad1): track 24.2 -> 48.5 mm
- net Net-(J5-Pad1): track 24.2 -> 48.5 mm
- net Net-(J4-Pad3): track 24.2 -> 48.5 mm
- net Net-(J4-Pad1): track 24.2 -> 48.5 mm
- net Net-(J9-Pad1): track 24.2 -> 48.5 mm
- net Net-(J9-Pad3): track 24.2 -> 48.5 mm
- net Net-(J8-Pad3): track 24.2 -> 48.5 mm
- net Net-(J6-Pad3): track 24.2 -> 48.5 mm
- net Net-(J2-Pad3): track 24.2 -> 48.5 mm
- net Net-(J2-Pad1): track 24.2 -> 48.5 mm
- net Net-(J12-Pad3): track 24.2 -> 48.5 mm
- net Net-(J11-Pad1): track 24.2 -> 48.5 mm
- net Net-(J10-Pad3): track 24.2 -> 48.5 mm
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