File: Circuit/boneIO - relay board/boneIO - relay board.sch (KiCad schematic (older format))
At the start: 47 parts, among them J1 Screw_Terminal_01x04, J10 Screw_Terminal_01x04, J11 Screw_Terminal_01x04, J12 Conn_02x13_Odd_Even, J2 Screw_Terminal_01x04, J3 Screw_Terminal_01x04, J4 Screw_Terminal_01x04, J5 Screw_Terminal_01x04, J6 Screw_Terminal_01x04, J7 POWER RELAY, J8 Screw_Terminal_01x04, J9 Screw_Terminal_01x04, K1 RM85-2011-35-1005, K10 RM85-2011-35-1005, K11 RM85-2011-35-1005, K12 RM85-2011-35-1005, K13 RM85-2011-35-1005, K14 RM85-2011-35-1005, K15 RM85-2011-35-1005, K16 RM85-2011-35-1005, K17 RM85-2011-35-1005, K18 RM85-2011-35-1005, K19 RM85-2011-35-1005, K2 RM85-2011-35-1005, K20 RM85-2011-35-1005, K3 RM85-2011-35-1005, K4 RM85-2011-35-1005, K5 RM85-2011-35-1005, K6 RM85-2011-35-1005, K7 RM85-2011-35-1005, K8 RM85-2011-35-1005, K9 RM85-2011-35-1005, U1 ULN2803A, U2 ULN2803A, U3 ULN2803A, U4 MCP9808_MSOP

Commit message: Circuit Repo Cleanup
Parts:
- removed J7: POWER RELAY, Connector_PinHeader_2.54mm:PinHeader_1x03_P2.54mm_Vertical, symbol Connector:Screw_Terminal_01x03
- added C1: 100n, Capacitor_SMD:C_0603_1608Metric, symbol Device:C
- added C2, C3, C4: 4.7uF/50V, Capacitor_SMD:C_1206_3216Metric, symbol Device:C
- added R10, R11, R12, R13, R14, R15, R16, R17, R18, R19, R20, R21, R22, R23, R24, R25, R26, R27, R28, R29: 10k, Resistor_SMD:R_0603_1608Metric, symbol Device:R
- K1, K10, K11, K12, K17, K18, K19, K2, K20, K3, K4, K5, K6, K7, K8, K9: symbol boneIO---relay-board-rescue:RM85-2011-35-1005-MK-boneIO---relay-board-rescue -> boneIO---relay-board-rescue:RM85-2011-35-1005-MK
- K13: renamed from K16; symbol boneIO---relay-board-rescue:RM85-2011-35-1005-MK-boneIO---relay-board-rescue -> boneIO---relay-board-rescue:RM85-2011-35-1005-MK
- K14: renamed from K15; symbol boneIO---relay-board-rescue:RM85-2011-35-1005-MK-boneIO---relay-board-rescue -> boneIO---relay-board-rescue:RM85-2011-35-1005-MK
- K15: renamed from K14; symbol boneIO---relay-board-rescue:RM85-2011-35-1005-MK-boneIO---relay-board-rescue -> boneIO---relay-board-rescue:RM85-2011-35-1005-MK
- K16: renamed from K13; symbol boneIO---relay-board-rescue:RM85-2011-35-1005-MK-boneIO---relay-board-rescue -> boneIO---relay-board-rescue:RM85-2011-35-1005-MK
- U1: renamed from U4; symbol boneIO---relay-board-rescue:MCP9808_MSOP-Sensor_Temperature-boneIO---relay-board-rescue -> Sensor_Temperature:MCP9808_MSOP
- renumbered J12 to J3, J3 to J4, J4 to J5, J5 to J6, J6 to J7, U1 to U2, U2 to U3, U3 to U4
Connections:
- net labels removed: +5V, VCC
- wire segments 339 -> 401
Other:
- note added: "OPTIONAL"
- note removed: "POWER JUMPER\n\n"
- moved on the sheet: R1, R2, R3, R4, R5, R6, R7, R8, R9, U2, U3, U4

Commit message: Repo Sync for new people
Parts:
- removed C1: 100n, Capacitor_SMD:C_0603_1608Metric, symbol Device:C
- removed C2, C3, C4: 4.7uF/50V, Capacitor_SMD:C_1206_3216Metric, symbol Device:C
Connections:
- wire segments 401 -> 393
Other:
- note removed: "OPTIONAL"
- moved on the sheet: R1, R2, R3, R4, R5, R6, R7, R8, R9

Commit message: Wykonana PCB RELAY RM85_v0.2
Parts:
- removed H1, H2: MountingHole, MountingHole:MountingHole_4.3mm_M4, symbol Mechanical:MountingHole
- removed J3: Conn_02x13_Odd_Even, Connector_PinHeader_2.54mm:PinHeader_2x13_P2.54mm_Vertical, symbol Connector_Generic:Conn_02x13_Odd_Even
- removed R1, R3, R5: 0k, Resistor_SMD:R_0603_1608Metric, symbol Device:R
- removed R14, R15, R16, R17, R18, R19, R20, R21, R22, R23, R24, R25, R26, R27, R28, R29: 10k, Resistor_SMD:R_0603_1608Metric, symbol Device:R
- added C1, C2, C3, C4, C5, C6: 100n, Capacitor_SMD:C_0603_1608Metric, symbol Device:C
- added J12, J13: Screw_Terminal_01x04, Connector_Phoenix_GMSTB:PhoenixContact_GMSTBA_2,5_4-G_1x04_P7.50mm_Horizontal, symbol Connector:Screw_Terminal_01x04
- added J3: Conn_02x04_Odd_Even, Connector_PinSocket_2.54mm:PinSocket_2x04_P2.54mm_Vertical, symbol Connector_Generic:Conn_02x04_Odd_Even
- added K21, K22, K23, K24: RM85-2011-35-1005, boneIO - RM85:RM852011351005_1, symbol boneIO---relay-board-rescue:RM85-2011-35-1005-MK-boneIO---relay-board-rescue
- added R7: 4.7k, Resistor_SMD:R_0603_1608Metric, symbol Device:R
- added R8, R9: 0k, Resistor_SMD:R_0603_1608Metric, symbol Device:R
- added SW1, SW2, SW3: SW_DIP_x03, Button_Switch_SMD:SW_DIP_SPSTx03_Slide_KingTek_DSHP03TJ_W5.25mm_P1.27mm_JPin, symbol Switch:SW_DIP_x03
- added U2, U3: MCP23017_SS, Package_SO:SSOP-28_5.3x10.2mm_P0.65mm, symbol Interface_Expansion:MCP23017_SS
- K1, K10, K11, K12, K13, K14, K15, K16, K17, K18, K19, K2, K20, K3, K4, K5, K6, K7, K8, K9: footprint RM85-2011-35-1005:RM852011351005 -> boneIO - RM85:RM852011351005_1; symbol boneIO---relay-board-rescue:RM85-2011-35-1005-MK -> boneIO---relay-board-rescue:RM85-2011-35-1005-MK-boneIO---relay-board-rescue
- R10, R11, R12, R13: value 10k -> 0k
- U1: symbol Sensor_Temperature:MCP9808_MSOP -> boneIO---relay-board-rescue:MCP9808_MSOP-Sensor_Temperature-boneIO---relay-board-rescue
- renumbered R2 to R1, R7 to R2, R4 to R3, R6 to R4, R8 to R5, R9 to R6, U2 to U4, U3 to U5, U4 to U6
Connections:
- net labels added: +3.3V, +5V, K21, K22, K23, K24, RELAY21, RELAY22, RELAY23, RELAY24, RESET_MCP
- wire segments 393 -> 477
- no-connect marks 80 -> 52
Other:
- moved on the sheet: J1, J10, J11, J2, J4, J5, J6, J7, J8, J9, R1, R2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

Commit message: 01.11.2021
Connections:
- net +3V3: now also J3.6 (Pin_6); no longer J3.8 (Pin_8)
- net GND: now also J3.5 (Pin_5); no longer J3.7 (Pin_7)
- net SCL: now also J3.8 (Pin_8); no longer J3.6 (Pin_6)
- net SDA: now also J3.7 (Pin_7); no longer J3.5 (Pin_5)
Changed lines of the file:
@@
 	8900 3950 8300 3950
 Wire Wire Line
-	9150 3600 9150 4150
-Wire Wire Line
-	9150 4150 8300 4150
-Wire Wire Line
-	7550 4350 7550 4150
+	9150 3600 9150 4050
+Wire Wire Line
+	9150 4050 8300 4050
 Wire Wire Line
 	7550 3850 7800 3850
@@
 	7550 3950 7550 3850
 Wire Wire Line
-	7800 4150 7550 4150
-Connection ~ 7550 4150
-Wire Wire Line
-	7550 4150 7550 3950
-Text GLabel 8300 4050 2    50   Input ~ 0
+	7800 4050 7550 4050
+Text GLabel 8300 4150 2    50   Input ~ 0
 SCL
-Text GLabel 7800 4050 0    50   Input ~ 0
+Text GLabel 7800 4150 0    50   Input ~ 0
 SDA
 $Comp
@@
 Text GLabel 10500 -1850 0    50   Input ~ 0
 RESET_MCP
+Wire Wire Line
+	7550 3950 7550 4050
+Connection ~ 7550 4050
+Wire Wire Line
+	7550 4050 7550 4350
 $EndSCHEMATC

Commit message: Wersja z dnia 02.11.2021
Parts:
- added JP1: Jumper_3_Open, Jumper:SolderJumper-3_P1.3mm_Open_RoundedPad1.0x1.5mm, symbol Jumper:Jumper_3_Open
- added R14: 4.7k, Resistor_SMD:R_0603_1608Metric, symbol Device:R
Connections:
- net +24V: now also JP1.1 (A); no longer C4.1, C5.1, C6.1, K1.A2 (COIL_2), K10.A2 (COIL_2), K11.A2 (COIL_2), K12.A2 (COIL_2), K13.A2 (COIL_2), K14.A2 (COIL_2), K15.A2 (COIL_2), K16.A2 (COIL_2), K17.A2 (COIL_2), K18.A2 (COIL_2), K19.A2 (COIL_2), K2.A2 (COIL_2), K20.A2 (COIL_2), K21.A2 (COIL_2), K22.A2 (COIL_2), K23.A2 (COIL_2), K24.A2 (COIL_2), K3.A2 (COIL_2), K4.A2 (COIL_2), K5.A2 (COIL_2), K6.A2 (COIL_2), K7.A2 (COIL_2), K8.A2 (COIL_2), K9.A2 (COIL_2), U4.10 (COM), U5.10 (COM), U6.10 (COM)
- net +3V3: now also R14.1
- net +5V: now also JP1.3 (B)
- net RESET_MCP: no longer names the net of R7.2, U2.18 (~RESET~)
- net RESET_MCP: no longer U3.18 (~RESET~)
- new net: R14.2, U3.18 (~RESET~)
- new net VCC: C4.1, C5.1, C6.1, JP1.2 (C), K1.A2 (COIL_2), K10.A2 (COIL_2), K11.A2 (COIL_2), K12.A2 (COIL_2), K13.A2 (COIL_2), K14.A2 (COIL_2), K15.A2 (COIL_2), K16.A2 (COIL_2), K17.A2 (COIL_2), K18.A2 (COIL_2), K19.A2 (COIL_2), K2.A2 (COIL_2), K20.A2 (COIL_2), K21.A2 (COIL_2), K22.A2 (COIL_2), K23.A2 (COIL_2), K24.A2 (COIL_2), K3.A2 (COIL_2), K4.A2 (COIL_2), K5.A2 (COIL_2), K6.A2 (COIL_2), K7.A2 (COIL_2), K8.A2 (COIL_2), K9.A2 (COIL_2), U4.10 (COM), U5.10 (COM), U6.10 (COM)
Other:
- moved on the sheet: J3

Commit message: Gotowa PCB board relay v0.2
Parts:
- removed JP1: Jumper_3_Open, Jumper:SolderJumper-3_P1.3mm_Open_RoundedPad1.0x1.5mm, symbol Jumper:Jumper_3_Open
- added JP1: SolderJumper_3_Bridged12, Jumper:SolderJumper-3_P1.3mm_Bridged12_RoundedPad1.0x1.5mm, symbol Jumper:SolderJumper_3_Bridged12
Connections:
- net +24V: now also JP1.1 (A)
- net +5V: now also JP1.3 (B)
- net SCL: now also R5.2; no longer R2.2
- net SDA: now also R2.2; no longer R5.2
- net VCC: now also JP1.2 (C)
Other:
- note added: "MCP23017"
- note added: "boneIO - relay board v0.2"
- moved on the sheet: C1, C2, C3, C4, C5, C6, J3, R1, R10, R11, R12, R13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

Commit message: Wersja Poprawiona
Parts:
- added J14: Conn_02x04_Odd_Even, Connector_PinHeader_2.54mm:PinHeader_2x04_P2.54mm_Vertical, symbol Connector_Generic:Conn_02x04_Odd_Even
- R1, R10, R11, R12, R13, R3, R4, R8, R9: value 0k -> 10k
Connections:
- net +24V: now also J3.1 (Pin_1), J14.1 (Pin_1); no longer J3.2 (Pin_2)
- net +3V3: now also J3.5 (Pin_5), J14.5 (Pin_5); no longer J3.6 (Pin_6)
- net +5V: now also J3.3 (Pin_3), J14.3 (Pin_3); no longer J3.4 (Pin_4)
- net GND: now also J3.2 (Pin_2), J3.4 (Pin_4), J3.6 (Pin_6), J14.2 (Pin_2), J14.4 (Pin_4), J14.6 (Pin_6); no longer J3.1 (Pin_1), J3.3 (Pin_3), J3.5 (Pin_5)
- net SCL: now also J3.7 (Pin_7), J14.7 (Pin_7); no longer J3.8 (Pin_8)
- net SDA: now also J3.8 (Pin_8), J14.8 (Pin_8); no longer J3.7 (Pin_7)
Changed lines of the file:
@@
 P 2150 4750
 F 0 "R1" H 2220 4796 50  0000 L CNN
-F 1 "0k" H 2220 4705 50  0000 L CNN
+F 1 "10k" H 2220 4705 50  0000 L CNN
 F 2 "Resistor_SMD:R_0603_1608Metric" V 2080 4750 50  0001 C CNN
 F 3 "~" H 2150 4750 50  0001 C CNN
@@
 P 2350 4750
 F 0 "R3" H 2420 4796 50  0000 L CNN
-F 1 "0k" H 2420 4705 50  0000 L CNN
+F 1 "10k" H 2420 4705 50  0000 L CNN
 F 2 "Resistor_SMD:R_0603_1608Metric" V 2280 4750 50  0001 C CNN
 F 3 "~" H 2350 4750 50  0001 C CNN
@@
 P 2550 4750
 F 0 "R4" H 2620 4796 50  0000 L CNN
-F 1 "0k" H 2620 4705 50  0000 L CNN
+F 1 "10k" H 2620 4705 50  0000 L CNN
 F 2 "Resistor_SMD:R_0603_1608Metric" V 2480 4750 50  0001 C CNN
 F 3 "~" H 2550 4750 50  0001 C CNN
@@
 P 16750 5000
 F 0 "R8" H 16820 5046 50  0000 L CNN
-F 1 "0k" H 16820 4955 50  0000 L CNN
+F 1 "10k" H 16820 4955 50  0000 L CNN
 F 2 "Resistor_SMD:R_0603_1608Metric" V 16680 5000 50  0001 C CNN
 F 3 "~" H 16750 5000 50  0001 C CNN
@@
 P 16950 5000
 F 0 "R9" H 17020 5046 50  0000 L CNN
-F 1 "0k" H 17020 4955 50  0000 L CNN
+F 1 "10k" H 17020 4955 50  0000 L CNN
 F 2 "Resistor_SMD:R_0603_1608Metric" V 16880 5000 50  0001 C CNN
 F 3 "~" H 16950 5000 50  0001 C CNN
@@
 P 17150 5000
 F 0 "R10" H 17220 5046 50  0000 L CNN
-F 1 "0k" H 17220 4955 50  0000 L CNN
+F 1 "10k" H 17220 4955 50  0000 L CNN
 F 2 "Resistor_SMD:R_0603_1608Metric" V 17080 5000 50  0001 C CNN
 F 3 "~" H 17150 5000 50  0001 C CNN
@@
 P 20300 5000
 F 0 "R11" H 20370 5046 50  0000 L CNN
-F 1 "0k" H 20370 4955 50  0000 L CNN
+F 1 "10k" H 20370 4955 50  0000 L CNN
 F 2 "Resistor_SMD:R_0603_1608Metric" V 20230 5000 50  0001 C CNN
 F 3 "~" H 20300 5000 50  0001 C CNN
@@
 P 20500 5000
 F 0 "R12" H 20570 5046 50  0000 L CNN
-F 1 "0k" H 20570 4955 50  0000 L CNN
+F 1 "10k" H 20570 4955 50  0000 L CNN
 F 2 "Resistor_SMD:R_0603_1608Metric" V 20430 5000 50  0001 C CNN
 F 3 "~" H 20500 5000 50  0001 C CNN
@@
 P 20700 5000
 F 0 "R13" H 20770 5046 50  0000 L CNN
-F 1 "0k" H 20770 4955 50  0000 L CNN
+F 1 "10k" H 20770 4955 50  0000 L CNN
 F 2 "Resistor_SMD:R_0603_1608Metric" V 20630 5000 50  0001 C CNN
 F 3 "~" H 20700 5000 50  0001 C CNN
@@
 $EndComp
 Wire Wire Line
-	5900 3450 5900 3750
-Connection ~ 5900 3450
-Wire Wire Line
-	5900 3350 5900 3450
+	6900 3450 6900 3750
+Connection ~ 6900 3450
+Wire Wire Line
+	6900 3350 6900 3450
+Text GLabel 6650 3550 2    50   Input ~ 0
+SDA
 Text GLabel 6150 3550 0    50   Input ~ 0
-SDA
-Text GLabel 6650 3550 2    50   Input ~ 0
 SCL
 Wire Wire Line
-	6150 3450 5900 3450
-Wire Wire Line
-	5900 3350 5900 3250
-Connection ~ 5900 3350
-Wire Wire Line
-	6150 3350 5900 3350
-Wire Wire Line
-	5900 3250 6150 3250
-Wire Wire Line
-	7500 3450 6650 3450
-Wire Wire Line
-	7500 3000 7500 3450
-Wire Wire Line
-	7250 3350 6650 3350
-Wire Wire Line
-	7250 3000 7250 3350
-Wire Wire Line
-	7000 3250 6650 3250
-Wire Wire Line
-	7000 3000 7000 3250
+	6650 3450 6900 3450
+Wire Wire Line
+	6900 3350 6900 3250
+Connection ~ 6900 3350
+Wire Wire Line
+	6650 3350 6900 3350
+Wire Wire Line
+	6900 3250 6650 3250
+Wire Wire Line
+	5300 3450 6150 3450
+Wire Wire Line
+	5300 3000 5300 3450
+Wire Wire Line
+	5550 3350 6150 3350
+Wire Wire Line
+	5550 3000 5550 3350
+Wire Wire Line
+	5800 3250 6150 3250
+Wire Wire Line
+	5800 3000 5800 3250
 $Comp
 L power:GND #PWR026
 U 1 1 61B786DB
-P 5900 3750
-F 0 "#PWR026" H 5900 3500 50  0001 C CNN
-F 1 "GND" H 5905 3577 50  0000 C CNN
-F 2 "" H 5900 3750 50  0001 C CNN
-F 3 "" H 5900 3750 50  0001 C CNN
-	1    5900 3750
-	-1   0    0    -1
+P 6900 3750
+F 0 "#PWR026" H 6900 3500 50  0001 C CNN
+F 1 "GND" H 6905 3577 50  0000 C CNN
+F 2 "" H 6900 3750 50  0001 C CNN
+F 3 "" H 6900 3750 50  0001 C CNN
+	1    6900 3750
+	1    0    0    -1
 $EndComp
 $Comp
 L power:+5V #PWR031
 U 1 1 61B7750C
-P 7250 3000
-F 0 "#PWR031" H 7250 2850 50  0001 C CNN
-F 1 "+5V" H 7265 3173 50  0000 C CNN
-F 2 "" H 7250 3000 50  0001 C CNN
-F 3 "" H 7250 3000 50  0001 C CNN
-	1    7250 3000
-	-1   0    0    -1
+P 5550 3000
+F 0 "#PWR031" H 5550 2850 50  0001 C CNN
+F 1 "+5V" H 5565 3173 50  0000 C CNN
+F 2 "" H 5550 3000 50  0001 C CNN
+F 3 "" H 5550 3000 50  0001 C CNN
+	1    5550 3000
+	1    0    0    -1
 $EndComp
 $Comp
 L power:+24V #PWR029
 U 1 1 61B0C600
-P 7000 3000
-F 0 "#PWR029" H 7000 2850 50  0001 C CNN
-F 1 "+24V" H 7015 3173 50  0000 C CNN
-F 2 "" H 7000 3000 50  0001 C CNN
-F 3 "" H 7000 3000 50  0001 C CNN
-	1    7000 3000
-	-1   0    0    -1
+P 5800 3000
+F 0 "#PWR029" H 5800 2850 50  0001 C CNN
+F 1 "+24V" H 5815 3173 50  0000 C CNN
+F 2 "" H 5800 3000 50  0001 C CNN
+F 3 "" H 5800 3000 50  0001 C CNN
+	1    5800 3000
+	1    0    0    -1
 $EndComp
 $Comp
 L power:+3V3 #PWR032
 U 1 1 61B0C5FA
-P 7500 3000
-F 0 "#PWR032" H 7500 2850 50  0001 C CNN
-F 1 "+3V3" H 7515 3173 50  0000 C CNN
-F 2 "" H 7500 3000 50  0001 C CNN
-F 3 "" H 7500 3000 50  0001 C CNN
-	1    7500 3000
-	-1   0    0    -1
+P 5300 3000
+F 0 "#PWR032" H 5300 2850 50  0001 C CNN
+F 1 "+3V3" H 5315 3173 50  0000 C CNN
+F 2 "" H 5300 3000 50  0001 C CNN
+F 3 "" H 5300 3000 50  0001 C CNN
+	1    5300 3000
+	1    0    0    -1
 $EndComp
 $Comp
@@
 Text Notes 9600 1250 0    197  ~ 39
 boneIO - relay board v0.2
+Wire Wire Line
+	6750 100  6750 400
+Connection ~ 6750 100
+Wire Wire Line
+	6750 0    6750 100
+Text GLabel 6500 200  2    50   Input ~ 0
+SDA
+Text GLabel 6000 200  0    50   Input ~ 0
+SCL
+Wire Wire Line
+	6500 100  6750 100
+Wire Wire Line
+	6750 0    6750 -100
+Connection ~ 6750 0
+Wire Wire Line
+	6500 0    6750 0
+Wire Wire Line
+	6750 -100 6500 -100
+Wire Wire Line
+	5150 100  6000 100
+Wire Wire Line
+	5150 -350 5150 100
+Wire Wire Line
+	5400 0    6000 0
+Wire Wire Line
+	5400 -350 5400 0
+Wire Wire Line
+	5650 -100 6000 -100
+Wire Wire Line
+	5650 -350 5650 -100
+$Comp
+L power:GND #PWR0132
+U 1 1 61859DEA
+P 6750 400
+F 0 "#PWR0132" H 6750 150 50  0001 C CNN
+F 1 "GND" H 6755 227 50  0000 C CNN
+F 2 "" H 6750 400 50  0001 C CNN
+F 3 "" H 6750 400 50  0001 C CNN
+	1    6750 400
+	1    0    0    -1
+$EndComp
+$Comp
+L power:+5V #PWR0133
+U 1 1 61859DF0
+P 5400 -350
+F 0 "#PWR0133" H 5400 -500 50  0001 C CNN
+F 1 "+5V" H 5415 -177 50  0000 C CNN
+F 2 "" H 5400 -350 50  0001 C CNN
+F 3 "" H 5400 -350 50  0001 C CNN
+	1    5400 -350
+	1    0    0    -1
+$EndComp
+$Comp
+L power:+24V #PWR0134
+U 1 1 61859DF6
+P 5650 -350
+F 0 "#PWR0134" H 5650 -500 50  0001 C CNN
+F 1 "+24V" H 5665 -177 50  0000 C CNN
+F 2 "" H 5650 -350 50  0001 C CNN
+F 3 "" H 5650 -350 50  0001 C CNN
+	1    5650 -350
+	1    0    0    -1
+$EndComp
+$Comp
+L power:+3V3 #PWR0135
+U 1 1 61859DFC
+P 5150 -350
+F 0 "#PWR0135" H 5150 -500 50  0001 C CNN
+F 1 "+3V3" H 5165 -177 50  0000 C CNN
+F 2 "" H 5150 -350 50  0001 C CNN
+F 3 "" H 5150 -350 50  0001 C CNN
+	1    5150 -350
+	1    0    0    -1
+$EndComp
+$Comp
+L Connector_Generic:Conn_02x04_Odd_Even J14
+U 1 1 61859E02
+P 6200 0
+F 0 "J14" H 6250 317 50  0000 C CNN
+F 1 "Conn_02x04_Odd_Even" H 6250 226 50  0000 C CNN
+F 2 "Connector_PinHeader_2.54mm:PinHeader_2x04_P2.54mm_Vertical" H 6200 0   50  0001 C CNN
+F 3 "~" H 6200 0   50  0001 C CNN
+	1    6200 0
+	1    0    0    -1
+$EndComp
 $EndSCHEMATC

Commit message: Zmiana Nazwy PCB
Parts:
- removed J14: Conn_02x04_Odd_Even, Connector_PinHeader_2.54mm:PinHeader_2x04_P2.54mm_Vertical, symbol Connector_Generic:Conn_02x04_Odd_Even
Other:
- note added: "boneIO - relay board 24x16A v0.2"
- note removed: "boneIO - relay board v0.2"
Changed lines of the file:
@@
 Text Notes 18650 2300 0    197  ~ 39
 MCP23017
-Text Notes 9600 1250 0    197  ~ 39
-boneIO - relay board v0.2
-Wire Wire Line
-	6750 100  6750 400
-Connection ~ 6750 100
-Wire Wire Line
-	6750 0    6750 100
-Text GLabel 6500 200  2    50   Input ~ 0
-SDA
-Text GLabel 6000 200  0    50   Input ~ 0
-SCL
-Wire Wire Line
-	6500 100  6750 100
-Wire Wire Line
-	6750 0    6750 -100
-Connection ~ 6750 0
-Wire Wire Line
-	6500 0    6750 0
-Wire Wire Line
-	6750 -100 6500 -100
-Wire Wire Line
-	5150 100  6000 100
-Wire Wire Line
-	5150 -350 5150 100
-Wire Wire Line
-	5400 0    6000 0
-Wire Wire Line
-	5400 -350 5400 0
-Wire Wire Line
-	5650 -100 6000 -100
-Wire Wire Line
-	5650 -350 5650 -100
-$Comp
-L power:GND #PWR0132
-U 1 1 61859DEA
-P 6750 400
-F 0 "#PWR0132" H 6750 150 50  0001 C CNN
-F 1 "GND" H 6755 227 50  0000 C CNN
-F 2 "" H 6750 400 50  0001 C CNN
-F 3 "" H 6750 400 50  0001 C CNN
-	1    6750 400
-	1    0    0    -1
-$EndComp
-$Comp
-L power:+5V #PWR0133
-U 1 1 61859DF0
-P 5400 -350
-F 0 "#PWR0133" H 5400 -500 50  0001 C CNN
-F 1 "+5V" H 5415 -177 50  0000 C CNN
-F 2 "" H 5400 -350 50  0001 C CNN
-F 3 "" H 5400 -350 50  0001 C CNN
-	1    5400 -350
-	1    0    0    -1
-$EndComp
-$Comp
-L power:+24V #PWR0134
-U 1 1 61859DF6
-P 5650 -350
-F 0 "#PWR0134" H 5650 -500 50  0001 C CNN
-F 1 "+24V" H 5665 -177 50  0000 C CNN
-F 2 "" H 5650 -350 50  0001 C CNN
-F 3 "" H 5650 -350 50  0001 C CNN
-	1    5650 -350
-	1    0    0    -1
-$EndComp
-$Comp
-L power:+3V3 #PWR0135
-U 1 1 61859DFC
-P 5150 -350
-F 0 "#PWR0135" H 5150 -500 50  0001 C CNN
-F 1 "+3V3" H 5165 -177 50  0000 C CNN
-F 2 "" H 5150 -350 50  0001 C CNN
-F 3 "" H 5150 -350 50  0001 C CNN
-	1    5150 -350
-	1    0    0    -1
-$EndComp
-$Comp
-L Connector_Generic:Conn_02x04_Odd_Even J14
-U 1 1 61859E02
-P 6200 0
-F 0 "J14" H 6250 317 50  0000 C CNN
-F 1 "Conn_02x04_Odd_Even" H 6250 226 50  0000 C CNN
-F 2 "Connector_PinHeader_2.54mm:PinHeader_2x04_P2.54mm_Vertical" H 6200 0   50  0001 C CNN
-F 3 "~" H 6200 0   50  0001 C CNN
-	1    6200 0
-	1    0    0    -1
-$EndComp
+Text Notes 8400 1200 0    197  ~ 39
+boneIO - relay board 24x16A v0.2
 $EndSCHEMATC
