File: Circuit/boneIO - relay board/boneIO - relay board.sch (KiCad schematic (older format))
At the start: 67 parts, among them J1 Screw_Terminal_01x04, J10 Screw_Terminal_01x04, J11 Screw_Terminal_01x04, J12 Screw_Terminal_01x04, J13 Screw_Terminal_01x04, J2 Screw_Terminal_01x04, J3 Conn_02x04_Odd_Even, J4 Screw_Terminal_01x04, J5 Screw_Terminal_01x04, J6 Screw_Terminal_01x04, J7 Screw_Terminal_01x04, J8 Screw_Terminal_01x04, J9 Screw_Terminal_01x04, K1 RM85-2011-35-1005, K10 RM85-2011-35-1005, K11 RM85-2011-35-1005, K12 RM85-2011-35-1005, K13 RM85-2011-35-1005, K14 RM85-2011-35-1005, K15 RM85-2011-35-1005, K16 RM85-2011-35-1005, K17 RM85-2011-35-1005, K18 RM85-2011-35-1005, K19 RM85-2011-35-1005, K2 RM85-2011-35-1005, K20 RM85-2011-35-1005, K21 RM85-2011-35-1005, K22 RM85-2011-35-1005, K23 RM85-2011-35-1005, K24 RM85-2011-35-1005, K3 RM85-2011-35-1005, K4 RM85-2011-35-1005, K5 RM85-2011-35-1005, K6 RM85-2011-35-1005, K7 RM85-2011-35-1005, K8 RM85-2011-35-1005, K9 RM85-2011-35-1005, SW1 SW_DIP_x03, SW2 SW_DIP_x03, SW3 SW_DIP_x03, U1 MCP9808_MSOP, U2 MCP23017_SS, U3 MCP23017_SS, U4 ULN2803A, U5 ULN2803A, U6 ULN2803A

Commit message: 05.11.2021
Connections:
- net at R1.1, U1.7 (A0): now also SW1.6; no longer SW1.4
- net at R4.1, U1.5 (A2): now also SW1.4; no longer SW1.6
Changed lines of the file:
@@
 L Switch:SW_DIP_x03 SW1
 U 1 1 619BF441
-P 1650 4250
-F 0 "SW1" H 1650 4717 50  0000 C CNN
-F 1 "SW_DIP_x03" H 1650 4626 50  0000 C CNN
-F 2 "Button_Switch_SMD:SW_DIP_SPSTx03_Slide_KingTek_DSHP03TJ_W5.25mm_P1.27mm_JPin" H 1650 4250 50  0001 C CNN
-F 3 "~" H 1650 4250 50  0001 C CNN
-	1    1650 4250
-	1    0    0    1
+P 1650 4450
+F 0 "SW1" H 1650 4917 50  0000 C CNN
+F 1 "SW_DIP_x03" H 1650 4826 50  0000 C CNN
+F 2 "Button_Switch_SMD:SW_DIP_SPSTx03_Slide_KingTek_DSHP03TJ_W5.25mm_P1.27mm_JPin" H 1650 4450 50  0001 C CNN
+F 3 "~" H 1650 4450 50  0001 C CNN
+	1    1650 4450
+	1    0    0    -1
 $EndComp
 Wire Wire Line
