File: Circuit/boneIOs- input board esp/boneIOs- input board esp.sch (KiCad schematic (older format))
At the start: 49 parts, among them J1 Screw_Terminal_01x08, J12 Conn_02x04_Odd_Even, J2 Screw_Terminal_01x08, J3 Screw_Terminal_01x08, J4 Screw_Terminal_01x08, J5 Screw_Terminal_01x08, J6 Screw_Terminal_01x08, J7 Screw_Terminal_01x08, J9 Screw_Terminal_01x08, U1 EL357N-G, U28 RS485, U46 P82B96, U9 LM2596S-ADJ

Commit message: 01.11.2021a
Parts:
- removed ANVDD1: Screw_Terminal_01x02, Connector:Phoenix_1x02_P5.00mm_Horizontal, symbol Connector:Screw_Terminal_01x02
- added C2, C3, C?: 100n, Capacitor_SMD:C_0603_1608Metric, symbol Device:C
- added R10, R11, R12, R13, R8, R9, R? (x3): 10k, Resistor_SMD:R_0603_1608Metric, symbol Device:R
- added R7, R? (x2): 4.7k, Resistor_SMD:R_0603_1608Metric, symbol Device:R
- added SW2, SW3, SW?: SW_DIP_x03, Button_Switch_SMD:SW_DIP_SPSTx03_Slide_KingTek_DSHP03TJ_W5.25mm_P1.27mm_JPin, symbol Switch:SW_DIP_x03
- added U2, U3, U?: MCP23017_SS, Package_SO:SSOP-28_5.3x10.2mm_P0.65mm, symbol Interface_Expansion:MCP23017_SS
Connections:
- net +3V3: now also C2.1, C3.1, C?.1, R7.1, R?.1, R?.1, SW2.4, SW2.5, SW2.6, SW3.4, SW3.5, SW3.6, SW?.4, SW?.5, SW?.6, U2.9 (VDD), U3.9 (VDD), U?.9 (VDD)
- net GND: now also C2.2, C3.2, C?.2, R10.2, R11.2, R12.2, R13.2, R8.2, R9.2, R?.2, R?.2, R?.2, U2.10 (VSS), U3.10 (VSS), U?.10 (VSS)
- net SCL: now also U2.12 (SCK), U3.12 (SCK), U?.12 (SCK)
- net SDA: now also U2.13 (SDA), U3.13 (SDA), U?.13 (SDA)
- new net: R?.1, SW?.3, U?.15 (A0)
- new net: R?.1, SW?.2, U?.16 (A1)
- new net: R?.1, SW?.1, U?.17 (A2)
- new net: R10.1, SW2.3, U2.15 (A0)
- new net: R9.1, SW2.2, U2.16 (A1)
- new net: R8.1, SW2.1, U2.17 (A2)
- new net: R13.1, SW3.3, U3.15 (A0)
- new net: R12.1, SW3.2, U3.16 (A1)
- new net: R11.1, SW3.1, U3.17 (A2)
- new net RESET_MCP: R7.2, R?.2, R?.2, U2.18 (~RESET~), U3.18 (~RESET~), U?.18 (~RESET~)
- new net in_1: U2.1 (GPB0)
- new net in_10: U2.22 (GPA1)
- new net in_11: U2.23 (GPA2)
- new net in_12: U2.24 (GPA3)
- new net in_13: U2.25 (GPA4)
- new net in_14: U2.26 (GPA5)
- new net in_15: U2.27 (GPA6)
- new net in_16: U2.28 (GPA7)
- new net in_17: U3.1 (GPB0)
- new net in_18: U3.2 (GPB1)
- new net in_19: U3.3 (GPB2)
- new net in_2: U2.2 (GPB1)
- new net in_20: U3.4 (GPB3)
- new net in_21: U3.5 (GPB4)
- new net in_22: U3.6 (GPB5)
- new net in_23: U3.7 (GPB6)
- new net in_24: U3.8 (GPB7)
- new net in_25: U3.21 (GPA0)
- new net in_26: U3.22 (GPA1)
- new net in_27: U3.23 (GPA2)
- new net in_28: U3.24 (GPA3)
- new net in_29: U3.25 (GPA4)
- new net in_3: U2.3 (GPB2)
- new net in_30: U3.26 (GPA5)
- new net in_31: U3.27 (GPA6)
- new net in_32: U3.28 (GPA7)
- new net in_33: U?.1 (GPB0)
- new net in_34: U?.2 (GPB1)
- new net in_35: U?.3 (GPB2)
- new net in_36: U?.4 (GPB3)
- new net in_37: U?.5 (GPB4)
- new net in_38: U?.6 (GPB5)
- new net in_39: U?.7 (GPB6)
- new net in_4: U2.4 (GPB3)
- new net in_40: U?.8 (GPB7)
- new net in_41: U?.21 (GPA0)
- new net in_42: U?.22 (GPA1)
- new net in_43: U?.23 (GPA2)
- new net in_44: U?.24 (GPA3)
- new net in_45: U?.25 (GPA4)
- new net in_46: U?.26 (GPA5)
- new net in_47: U?.27 (GPA6)
- new net in_48: U?.28 (GPA7)
- new net in_5: U2.5 (GPB4)
- new net in_6: U2.6 (GPB5)
- new net in_7: U2.7 (GPB6)
- new net in_8: U2.8 (GPB7)
- new net in_9: U2.21 (GPA0)
- no-connect marks 1 -> 7
Other:
- moved on the sheet: C1, C10, C17, C18, C47, C9, C?, D1, D2, D3, D4, F1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

Commit message: Gotowa PCB board relay v0.2
Parts:
- added C? (x53): 100n, Capacitor_SMD:C_0603_1608Metric, symbol Device:C
- added J?: UART, symbol Connector:Screw_Terminal_01x06
- added J?: Screw_Terminal_01x08, Connector:8pin, symbol Connector:Screw_Terminal_01x08
- added PWN: Screw_Terminal_01x02, Connector:Phoenix_1x02_P5.00mm_Horizontal, symbol Connector:Screw_Terminal_01x02
- added Q? (x2): BC817, Package_TO_SOT_SMD:SOT-23, symbol Transistor_BJT:BC817
- added R? (x2): 10k, symbol Device:R
- added R? (x60): 10k, Resistor_SMD:R_0603_1608Metric, symbol Device:R
- added R? (x2): 1k, Resistor_SMD:R_0603_1608Metric, symbol Device:R
- added U? (x53): EL357N-G, Package_SO:OPTO_EL357N-G, symbol Isolator:PC817
- added U?: BTS3410G, symbol Oscillator:BTS3410G
- I2C1: value Conn_01x04 -> OLED
- J7: value Screw_Terminal_01x08 -> GPIO_OUT
Connections:
- net P8.03_OUT is gone; now on net in_42: J6.8 (Pin_8)
- net P8.04_OUT is gone; now on net in_41: J6.7 (Pin_7)
- net P8.05_OUT is gone; now on net in_40: J6.6 (Pin_6)
- net P8.06_OUT is gone; now on net in_39: J6.5 (Pin_5)
- net P8.07_OUT is gone; now on net in_38: J6.4 (Pin_4)
- net P8.08_OUT is gone; now on net in_37: J6.3 (Pin_3)
- net P8.09_OUT is gone; now on net in_36: J6.2 (Pin_2)
- net P8.10_OUT is gone; now on net in_28: J4.8 (Pin_8)
- net P8.11_OUT is gone; now on net in_27: J4.7 (Pin_7)
- net P8.12_OUT is gone; now on net in_26: J4.6 (Pin_6)
- net P8.14_OUT is gone; now on net in_25: J4.5 (Pin_5)
- net P8.15_OUT is gone; now on net in_24: J4.4 (Pin_4)
- net P8.16_OUT is gone; now on net in_23: J4.3 (Pin_3)
- net P8.17_OUT is gone; now on net in_22: J4.2 (Pin_2)
- net P8.26_OUT is gone; now on net in_21: J3.8 (Pin_8)
- net P8.27_OUT is gone; now on net in_20: J3.7 (Pin_7)
- net P8.28_OUT is gone; now on net in_19: J3.6 (Pin_6)
- net P8.29_OUT is gone; now on net in_18: J3.5 (Pin_5)
- net P8.30_OUT is gone; now on net in_17: J3.4 (Pin_4)
- net P8.31_OUT is gone; now on net in_16: J3.3 (Pin_3)
- net P8.32_OUT is gone; now on net in_15: J3.2 (Pin_2)
- net P8.40_OUT is gone; now on net in_35: J5.8 (Pin_8)
- net P8.41_OUT is gone; now on net in_34: J5.7 (Pin_7)
- net P8.42_OUT is gone; now on net in_33: J5.6 (Pin_6)
- net P8.43_OUT is gone; now on net in_32: J5.5 (Pin_5)
- net P8.44_OUT is gone; now on net in_31: J5.4 (Pin_4)
- net P8.45_OUT is gone; now on net in_30: J5.3 (Pin_3)
- net P8.46 is gone; now on net S0-1: U1.4
- net P9.39 is gone; now on net GND: J7.1 (Pin_1)
- net P9.40 is gone; now on net S0-1_OUT: J7.2 (Pin_2)
- net +24VA: now also R?.2, R?.2, R?.2, R?.2, R?.2, R?.2, R?.2, R?.2, R?.2, R?.2, R?.2, R?.2, R?.2, R?.2, R?.2, R?.2, R?.2, R?.2, R?.2, R?.2, R?.2, R?.2, R?.2, R?.2, R?.2, R?.2, R?.2, R?.2, R?.2, R?.2, R?.2, R?.2, R?.2, R?.2, R?.2, R?.2, R?.2, R?.2, R?.2, R?.2, R?.2, R?.2, R?.2, R?.2, R?.2, R?.2, R?.2, R?.2, R?.2, R?.2, R?.2, R?.2, R?.2
- net +3V3: now also J?.2 (Pin_2), R?.2, R?.2, R?.2, R?.2, R?.2, R?.2, R?.2
- net GND: now also J?.1 (Pin_1), U?.1 (S1), U?.3, U?.3, U?.3, U?.3, U?.3, U?.3, U?.3, U?.3, U?.3, U?.3, U?.3, U?.3, U?.3, U?.3, U?.3, U?.3, U?.3, U?.3, U?.3, U?.3, U?.3, U?.3, U?.3, U?.3, U?.3, U?.3, U?.3, U?.3, U?.3, U?.3, U?.3, U?.3, U?.3, U?.3, U?.3, U?.3, U?.3, U?.3, U?.3, U?.3, U?.3, U?.3, U?.3, U?.3, U?.3, U?.3, U?.3, U?.3, U?.3, U?.3, U?.3, U?.3, U?.3, U?.3 (S2)
- net GNDA: now also J?.1 (Pin_1)
- net GPIO0: now also Q?.3 (C)
- net PWM1: now also R?.1
- net PWM2: now also R?.1
- net RST_32: now also Q?.3 (C)
- net RX: now also J?.5 (Pin_5)
- net S0-1: now also R?.1
- net S0-2: now also R?.1, U?.4
- net S0-3: now also R?.1, U?.4
- net S0-4: now also R?.1, U?.4
- net TX: now also J?.6 (Pin_6)
- net in_1: now also U?.4
- net in_10: now also U?.4
- net in_11: now also U?.4
- net in_12: now also U?.4
- net in_13: now also U?.4
- net in_14: now also U?.4
- net in_15: now also U?.4
- net in_16: now also U?.4
- net in_17: now also U?.4
- net in_18: now also U?.4
- net in_19: now also U?.4
- net in_2: now also U?.4
- net in_20: now also U?.4
- net in_21: now also U?.4
- net in_22: now also U?.4
- net in_23: now also U?.4
- net in_24: now also U?.4
- net in_25: now also U?.4
- net in_26: now also U?.4
- net in_27: now also U?.4
- net in_28: now also U?.4
- net in_29: now also J5.2 (Pin_2), U?.4
- net in_3: now also U?.4
- net in_30: now also U?.4
- net in_31: now also U?.4
- net in_32: now also U?.4
- net in_33: now also U?.4
- net in_35: now also U?.4
- net in_36: now also U?.4
- net in_37: now also U?.4
- net in_38: now also U?.4
- net in_39: now also U?.4
- net in_4: now also U?.4
- net in_40: now also U?.4
- net in_41: now also U?.4
- net in_42: now also U?.4
- net in_43: now also J?.2 (Pin_2), U?.4
- net in_44: now also J?.3 (Pin_3), U?.4
- net in_45: now also J?.4 (Pin_4), U?.4
- net in_46: now also J?.5 (Pin_5), U?.4
- net in_47: now also J?.6 (Pin_6), U?.4
- net in_48: now also J?.7 (Pin_7), U?.4
- net in_5: now also U?.4
- net in_6: now also U?.4
- net in_7: now also U?.4
- net in_8: now also U?.4
- net in_9: now also U?.4
- net S0-5: now reaches U?.14 (IO12)
- net S0-5: now also R?.1, U?.4
- net S0-6: now reaches U?.6 (IO34)
- net S0-6: now also R?.1, U?.4
- net S0-7: now reaches U?.7 (IO35)
- net S0-7: now also R?.1, U?.4
- net S0-7_OUT: now reaches J7.8 (Pin_8)
- net S0-7_OUT: now also C?.2, U?.2
- net P8.18_OUT: no longer names the net of J2.8 (Pin_8)
- net P8.20_OUT: no longer names the net of J2.7 (Pin_7)
- net P8.21_OUT: no longer names the net of J2.6 (Pin_6)
- net P8.22_OUT: no longer names the net of J2.5 (Pin_5)
- net P8.23_OUT: no longer names the net of J2.4 (Pin_4)
- net P8.24_OUT: no longer names the net of J2.3 (Pin_3)
- net P8.25_OUT: no longer names the net of J2.2 (Pin_2)
- net P8.33_OUT renamed in_7_OUT
- net in_7_OUT: now also C?.2, U?.2
- net P8.34_OUT renamed in_6_OUT
- net in_6_OUT: now also C?.2, U?.2
- net P8.35_OUT renamed in_5_OUT
- net in_5_OUT: now also C?.2, U?.2
- net P8.36_OUT renamed in_4_OUT
- net in_4_OUT: now also C?.2, U?.2
- net P8.37_OUT renamed in_3_OUT
- net in_3_OUT: now also C?.2, U?.2
- net P8.38_OUT renamed in_2_OUT
- net in_2_OUT: now also C?.2, U?.2
- net P8.39_OUT renamed in_1_OUT
- net in_1_OUT: now also C?.2, U?.2
- net P8.46_OUT renamed S0-1_OUT
- net S0-1_OUT: no longer J5.2 (Pin_2)
- net P9.33 renamed S0-6_OUT
- net S0-6_OUT: now also C?.2, U?.2
- net P9.35 renamed S0-4_OUT
- net S0-4_OUT: now also C?.2, U?.2
- net P9.36 renamed S0-5_OUT
- net S0-5_OUT: now also C?.2, U?.2
- net P9.37 renamed S0-2_OUT
- net S0-2_OUT: now also C?.2, U?.2
- net P9.38 renamed S0-3_OUT
- net S0-3_OUT: now also C?.2, U?.2
- removed net RESET_MCP: R7.2, R?.2, R?.2, U2.18 (~RESET~), U3.18 (~RESET~), U?.18 (~RESET~)
- new net: R?.2, U?.18 (~RESET~)
- new net: R?.2, U3.18 (~RESET~)
- new net: Q?.1 (B), R?.1 (x2)
- new net: R7.2, U2.18 (~RESET~)
- new net: C?.1, R?.1, U?.1 (x53)
- new net: R?.2, U?.2 (IN1)
- new net: R?.2, U?.4 (IN2)
- new net: PWN.2 (Pin_2), U?.5 (D2), U?.6 (D2)
- new net: PWN.1 (Pin_1), U?.7 (D1), U?.8 (D1)
- new net DTR: J?.3 (Pin_3), Q?.2 (E), R?.2
- new net RTS: J?.4 (Pin_4), Q?.2 (E), R?.2
- new net in_10_OUT: C?.2, U?.2
- new net in_11_OUT: C?.2, U?.2
- new net in_12_OUT: C?.2, U?.2
- new net in_13_OUT: C?.2, U?.2
- new net in_14_OUT: C?.2, U?.2
- new net in_15_OUT: C?.2, U?.2
- new net in_16_OUT: C?.2, U?.2
- new net in_17_OUT: C?.2, U?.2
- new net in_18_OUT: C?.2, U?.2
- new net in_19_OUT: C?.2, U?.2
- new net in_20_OUT: C?.2, U?.2
- new net in_21_OUT: C?.2, U?.2
- new net in_22_OUT: C?.2, U?.2
- new net in_23_OUT: C?.2, U?.2
- new net in_24_OUT: C?.2, U?.2
- new net in_25_OUT: C?.2, U?.2
- new net in_26_OUT: C?.2, U?.2
- new net in_27_OUT: C?.2, U?.2
- new net in_28_OUT: C?.2, U?.2
- new net in_29_OUT: C?.2, U?.2
- new net in_30_OUT: C?.2, U?.2
- new net in_31_OUT: C?.2, U?.2
- new net in_32_OUT: C?.2, U?.2
- new net in_33_OUT: C?.2, U?.2
- new net in_34_OUT: C?.2, U?.2
- new net in_36_OUT: C?.2, U?.2
- new net in_37_OUT: C?.2, U?.2
- new net in_38_OUT: C?.2, U?.2
- new net in_39_OUT: C?.2, U?.2
- new net in_40_OUT: C?.2, U?.2
- new net in_41_OUT: C?.2, U?.2
- new net in_42_OUT: C?.2, U?.2
- new net in_43_OUT: C?.2, U?.2
- new net in_44_OUT: C?.2, U?.2
- new net in_45_OUT: C?.2, U?.2
- new net in_46_OUT: C?.2, U?.2
- new net in_47_OUT: C?.2, U?.2
- new net in_48_OUT: C?.2, U?.2
- new net in_8_OUT: C?.2, U?.2
- new net in_9_OUT: C?.2, U?.2
- no-connect marks 7 -> 6
Other:
- moved on the sheet: C1, C10, C17, C18, C2, C3, C47, C9, C?, D1, D2, D3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
